File: OpenEFI(STM32F) rev1/v2.brd (EAGLE design)
At the start: 160 x 100 mm, 133 parts, among them IC1 4050N, IC10 LM358D, IC11 74HC595D, IC12 74HC595D, IC2 LM358D, IC3 4067D, IC5 4050N, IC6 74HC164D, IC7 4051D, IC8 24AA08SN, IC9 LM358D, P1 39-30-06?, Q1 MJD122, Q10 MJD122, Q11 MJD122, Q13 MJD122, Q15 MJD122, Q16 MJD122, Q17 MJD122, Q2 BC548, Q3 MJD122, Q5 MJD122, Q7 MJD122, Q9 MJD122, U1 ATMEGA328P-AU

Commit message: Creacion de V2 del PCB para SMT32F
Parts:
- removed IC1: 4050N, 40xx:DIL16
- removed IC6: 74HC164D, 74xx-us:SO14
- removed IC7: 4051D, 40xx:SO16
- moved SJ1 270.9 mm to (130.5, 77.1)
- moved DISPLAY 239.0 mm to (143.5, 82.5), turned to 90 degrees
- moved PROG 222.5 mm to (112.4, 82.5), turned to 90 degrees
- moved D23 215.4 mm to (83.8, 88.9), turned to 90 degrees
- moved U1 210.9 mm to (96.4, 51.1)
- moved C3 199.4 mm to (69.4, 67.5), turned to 90 degrees
- moved D22 195.1 mm to (71.1, 88.9), turned to 270 degrees
- moved R6 186.9 mm to (34.3, 49.9), turned to 180 degrees
- moved D21 183.7 mm to (67.3, 88.9), turned to 90 degrees
- moved R17 181.3 mm to (41.9, 78.1), turned to 90 degrees
- moved R12 180.6 mm to (68.5, 93.5), turned to 180 degrees
- moved C10 177.8 mm to (59.0, 67.7)
- moved R14 174.2 mm to (55.1, 96.5), turned to 180 degrees
- moved U$2 172.9 mm to (129.5, 73.7), turned to 270 degrees
- moved Q17 172.8 mm to (94.0, 88.9)
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Connections:
- removed net VDD: IC3.24, IC5.1
- removed net VSS: IC3.12, IC5.8
- net 5V: now also IC3.24; no longer IC6.14, IC7.16
- net 5V1: now also LED1.A, LED2.A, LED3.A, LED4.A, LED5.A; no longer R10.1, R11.1, R12.1, R14.1, R9.1
- net ACC: now also IC5.1, X2.50; no longer IC1.1
- net GND: now also IC3.12, IC5.8; no longer IC1.8, IC6.7, IC7.7, IC7.8
- net IAC_A: now also X2.14
- net IAC_B: now also X2.31
- net IAC_C: now also X2.48
- net IAC_D: now also X2.15
- net L1: now also R9.1; no longer LED1.K
- net L2: now also R10.1; no longer LED2.K
- net L3: now also R11.1; no longer LED3.K
- net L4: now also R12.1; no longer LED4.K
- net L5: now also R14.1; no longer LED5.K
- net N$12: now also LED1.K; no longer LED1.A
- net N$13: now also LED2.K; no longer LED2.A
- net N$15: now also LED3.K; no longer LED3.A
- net N$16: now also LED4.K; no longer LED4.A
- net N$17: now also LED5.K; no longer LED5.A
- net RL1IN: now also X2.17
- net RL2IN: now also X2.33
- net RL3IN: now also X2.16
- net RL4IN: now also X2.49
- net RL5IN: now also X2.32
- net TPSM_A: now also X2.30
- net TPSM_B: now also X2.47
Routing:
- net ACC: track 0.00 -> 169.1 mm, vias 0 -> 5
- net 5V1: track 0.00 -> 151.6 mm, vias 0 -> 1
- net RL5IN: track 0.00 -> 103.0 mm, vias 0 -> 2
- net RL4IN: track 0.00 -> 88.3 mm, vias 0 -> 1
- net RL3IN: track 0.00 -> 66.3 mm, vias 0 -> 1
- net RL1: track 0.00 -> 61.8 mm
- net RL2IN: track 0.00 -> 55.3 mm, vias 0 -> 1
- net RL2: track 0.00 -> 51.8 mm
- net RL3: track 0.00 -> 36.8 mm
- net 5V: track 0.00 -> 36.0 mm
- net N$33: track 0.00 -> 34.0 mm
- net N$30: track 0.00 -> 32.6 mm
- net N$38: track 0.00 -> 29.1 mm
- net N$27: track 0.00 -> 29.1 mm
- net N$39: track 0.00 -> 29.1 mm
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Other:
- board size 160 x 100 mm -> 149.8 x 100 mm

Commit message: cambios menores
Parts:
- removed IC10: LM358D, linear:SO08
- removed X1: (no value), con-subd:F37HP
- moved SV1 277.9 mm to (132.9, 14.1)
- moved SV2 276.7 mm to (132.8, 38.5)
- moved R30 245.7 mm to (141.0, 32.3), turned to 180 degrees
- moved R29 245.3 mm to (145.6, 27.6), turned to 270 degrees
- moved IC9 242.5 mm to (139.1, 27.2)
- moved C19 235.6 mm to (143.2, 27.6), turned to 270 degrees
- moved IC2 230.2 mm to (144.0, 61.3)
- moved C1 229.0 mm to (121.7, 13.3), turned to 270 degrees
- moved R27 228.1 mm to (135.9, 19.5), turned to 180 degrees
- moved R28 228.0 mm to (132.8, 26.8), flipped to the bottom, turned to 90 degrees
- moved R3 224.1 mm to (126.6, 14.6), turned to 270 degrees
- moved C17 222.3 mm to (130.8, 20.7), turned to 90 degrees
- moved R26 220.5 mm to (135.9, 21.6), turned to 180 degrees
- moved C16 219.6 mm to (142.1, 21.3)
- moved C18 218.1 mm to (140.0, 34.8), turned to 180 degrees
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Connections:
- removed net AIRIN: X1.5
- removed net AUX6: IC3.16
- removed net MAPIN: X1.8
- removed net TEMPIN: X1.3
- removed net TPSIN: X1.2
- removed net TPSIN2: X1.9
- net 5V: no longer IC10.8, X1.20, X1.21, X1.22, X1.24, X1.25, X1.27, X1.29
- net ACC: no longer X1.1, X1.10, X1.19, X1.35
- net AOUT0: now also IC3.2; no longer IC3.9
- net AOUT1: now also IC3.3; no longer IC3.8
- net AOUT2: now also IC3.4; no longer IC3.7
- net AOUT3: now also IC3.5; no longer IC3.6
- net AOUT4: now also IC3.6; no longer IC3.5
- net AOUT5: now also IC3.7; no longer IC3.4
- net AOUT6: now also IC3.8; no longer IC3.3
- net AOUT7: now also IC3.9; no longer IC3.2
- net AUX1: now also IC3.20; no longer IC3.21
- net AUX2: now also IC3.19; no longer IC3.20
- net AUX3: now also IC3.18; no longer IC3.19
- net AUX4: now also IC3.17; no longer IC3.18
- net AUX5: now also IC3.16; no longer IC3.17
- net CKPIN: no longer X1.4
- net GNC/GLP_MODE: no longer X1.30
- net GND: no longer IC10.4, X1.15, X1.23, X1.26, X1.28, X1.34
- net IAC_A: no longer X1.13
- net IAC_B: no longer X1.32
- net IAC_C: no longer X1.14
- net IAC_D: no longer X1.33
- net LAMB0: no longer X1.7
- net LAMB1: no longer X1.6
- net LAMB1OUT: now also IC9.7; no longer IC10.1
- net LED1: no longer X1.11
- net N$1: now also IC9.5; no longer IC10.3
- net N$37: now also IC9.6; no longer IC10.2
- net RL1IN: no longer X1.36
- net RL2IN: no longer X1.18
- net RL3IN: no longer X1.17
- net RL4IN: no longer X1.37
- net RL5IN: no longer X1.16
- net TPSM_A: no longer X1.12
- net TPSM_B: no longer X1.31
- net VBAT: now also IC3.21
Routing:
- net 5V: track 36.0 -> 132.7 mm, vias 0 -> 1
- net N$2: track 0.00 -> 87.2 mm, vias 0 -> 1
- net ECN2: track 0.00 -> 74.4 mm
- net N$3: track 0.00 -> 69.1 mm, vias 0 -> 1
- net ECN1: track 0.00 -> 61.1 mm
- net INY3: track 0.00 -> 52.5 mm
- net INY4: track 0.00 -> 47.9 mm
- net N$6: track 0.00 -> 44.2 mm
- net INY2: track 0.00 -> 41.8 mm
- net AOUT3: track 5.15 -> 45.5 mm
- net AOUT2: track 5.11 -> 43.6 mm
- net AOUT0: track 5.71 -> 43.7 mm
- net AOUT1: track 5.82 -> 43.6 mm
- net N$9: track 0.00 -> 36.6 mm, vias 0 -> 1
- net N$33: track 34.0 -> 0.00 mm, vias 0 -> 1
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- added copper zone on layer 1, net GND
Other:
- outline, holes or cut-outs redrawn

Commit message: Avances en I/O en rev1
Parts:
- moved Q4 5.35 mm to (104.8, 77.4)
- moved D2 3.34 mm to (117.0, 9.75)
- moved C1 3.00 mm to (120.3, 10.7)
Connections:
- net N$18 renamed N$18_P
- net N$20 renamed N$20_N
- net AIN0: now also X2.13
- net AIN1: now also X2.29
- net AIN4: now also X2.12
Routing:
- net PWM: track 0.00 -> 96.7 mm, vias 0 -> 4
- net 5V: track 132.7 -> 215.8 mm, vias 1 -> 3
- net AIN6: track 11.2 -> 74.8 mm
- net AIN7: track 10.7 -> 71.2 mm
- net AIN5: track 10.9 -> 65.9 mm
- net AIN4: track 10.9 -> 64.7 mm
- net N$5: track 0.00 -> 50.9 mm, vias 0 -> 1
- net AIN2: track 10.7 -> 43.2 mm
- net AIN3: track 10.1 -> 42.0 mm
- net AIN1: track 10.3 -> 41.9 mm
- net 3V3: track 0.00 -> 29.8 mm
- net MOSI: track 0.00 -> 29.3 mm, vias 0 -> 1
- net MISO: track 0.00 -> 28.9 mm, vias 0 -> 2
- net SCK2: track 0.00 -> 27.5 mm, vias 0 -> 3
- net SS: track 0.00 -> 26.0 mm, vias 0 -> 1
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- added copper zone on layer 16, net GND

Commit message: init v3
Parts:
- removed 1K-1%, 3K-1%: 520, rcl:0204/7
- removed C10, C3: (no value), rcl:E3,5-8
- removed D21, D22, D23, D32, D33: S1M, diode:SMA
- removed IC4: (no value), linear:TO263-5
- removed IC5: 4050N, 40xx:DIL16
- removed L1: 68uH, inductor-neosid:SD12-680
- removed Q17: MJD122, MJD122:DPAK
- removed U1: ATMEGA328P-AU, atmega328:QFP80P900X900X120-32N
- added D11: 1N4148DO35-7, diode:DO35-7
- added D25: BZY97, diode:F126Z12
- added F2: (no value), fuse:TE5
- added J1, J2: 1053141206, 1053141206:MOLEX_1053141206
- added P3: 39-30-04?, con-molex-mini-fit:39-30-?04?
- added Q12, Q19, Q22, Q25: BC558A, transistor-pnp:TO92-EBC
- added Q14, Q20, Q23, Q6: IRLZ44Z, transistor-power:TO220BH
- added Q18, Q21, Q24, Q8: BC548, transistor-npn:TO92-EBC
- added Q26: BD139, transistor-power:TO126AV
- added R15, R51: 1k, rcl:0204/5
- added R31, R32, R33, R34, R43, R44, R45, R46, R47, R48, R49, R50: (no value), rcl:0207/10
- added X1, X3: (no value), con-subd:F15HP
- D1, D16, D4, D6, D7: value 1N4004 -> BZY97; device diode:DO41-10 -> diode:F126Z12
- D12, D13, D14, D15, D20: value S1M -> 1N4446; device diode:SMA -> diode:DO35-10
- D18: value 1N4004 -> 1N4148DO35-7; device diode:DO41-10 -> diode:DO35-7
- D9: value Ss54 -> 1N4446; device s1x_10:DO214AC -> diode:DO35-10
- Q1, Q7: value MJD122 -> IRLZ44Z; device MJD122:DPAK -> transistor-power:TO220BH
- Q10, Q15, Q16, Q9: value MJD122 -> BD139; device MJD122:DPAK -> transistor-power:TO126AV
- Q11, Q3: value MJD122 -> BC548; device MJD122:DPAK -> transistor-npn:TO92-EBC
- Q13, Q5: value MJD122 -> BC558A; device MJD122:DPAK -> transistor-pnp:TO92-EBC
- Q4: value (none) -> BD139; device special:QS -> transistor-power:TO126AV
- X2: value (none) -> MINI-USB_4P-85-32004-10X; device con-subd:F50HP -> con-cypressindustries:85-32004-10X
- moved Q10 141.0 mm to (165.7, 16.8)
- moved D13 113.0 mm to (86.5, -3.56), turned to 0 degrees
- moved D20 103.8 mm to (101.8, -3.59), turned to 0 degrees
- moved D12 95.0 mm to (56.9, -3.36), turned to 0 degrees
- moved D15 94.7 mm to (71.3, -3.53), turned to 0 degrees
- moved Q9 94.6 mm to (56.7, -1.20), turned to 180 degrees
- moved Q4 93.3 mm to (40.1, 10.2), turned to 0 degrees
- moved D14 92.4 mm to (42.3, -3.42), turned to 0 degrees
- moved Q15 91.9 mm to (42.7, -1.14), turned to 180 degrees
- moved X2 90.6 mm to (98.2, 89.5), turned to 270 degrees
- moved Q16 90.3 mm to (71.0, -1.21), turned to 180 degrees
- moved D18 80.0 mm to (113.1, 82.5)
- moved D9 78.0 mm to (28.0, -3.50)
- moved R23 69.4 mm to (79.7, 10.1), turned to 0 degrees
- moved R21 69.0 mm to (91.5, 9.68), turned to 0 degrees
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Connections:
- removed net ECN1: D16.C, P1.5, Q11.4
- removed net ECN1L: IC5.11, U1.27
- removed net ECN2: D18.C, P1.6, Q13.4
- removed net ECN2L: IC5.14, U1.28
- removed net N$18_P: Q4.2, U1.7
- removed net N$20_N: Q4.1, U1.8
- removed net N$91: D9.C, IC4.2, L1.1
- removed net N$92: 1K-1%.1, 3K-1%.2, IC4.4
- new net 5V-USB: D11.A, X2.1
- new net D+: U$2.PA_12, X2.3
- new net D-: U$2.PA_11, X2.2
- new net GND2: F2.2, Q1.S, Q14.S, Q20.S, Q23.S, Q6.S, Q7.S
- new net INY5: D7.C, P1.5, Q20.D
- new net INY6: D16.C, P1.6, Q23.D
- new net INYL5A: R47.2
- new net INYL6A: R49.2
- new net N$18: Q13.B, Q8.B, R43.1
- new net N$20: Q13.E, Q8.E, R44.2
- new net N$27: Q7.G, R44.1
- new net N$28: Q18.B, Q19.B, R45.1
- new net N$30: Q18.E, Q19.E, R46.2
- new net N$33: Q14.G, R46.1
- new net N$35: D18.A, PROG.4
- new net N$36: Q4.B, R51.2
- new net N$46: Q21.B, Q22.B, R47.1
- new net N$47: Q21.E, Q22.E, R48.2
- new net N$48: Q20.G, R48.1
- new net N$49: Q24.B, Q25.B, R49.1
- new net N$50: Q24.E, Q25.E, R50.2
- new net N$52: Q23.G, R50.1
- new net RL6: R51.1
- new net RL6IN: D20.C, J1.6, Q4.C
- net 5V: no longer 3K-1%.1, C10.+, L1.2, U1.18, U1.20, U1.4, U1.6
- net 5V1: now also D11.C, D18.C; no longer PROG.4
- net ACC: now also Q11.C, Q18.C, Q21.C, Q24.C, Q3.C, Q8.C; no longer C3.+, D13.C, D15.C, D21.C, D23.C, D33.C, IC4.1, IC5.1, X2.50
- net AIN0: no longer X2.13
- net AIN1: no longer X2.29
- net AIN4: no longer X2.12
- net CKPOUT: no longer U1.32
- net GND: now also D15.A, D25.A, F2.1, P3.1, P3.2, P3.3, P3.4, Q10.E, Q12.C, Q13.C, Q15.E, Q16.E, Q19.C, Q22.C, Q25.C, Q26.E, Q4.E, Q5.C, Q9.E, X2.4; no longer 1K-1%.2, C10.-, C3.-, D18.A, D22.A, D32.A, IC4.3, IC4.5, IC4.6, IC5.8, Q1.3, Q10.3, Q11.3, Q13.3, Q15.3, Q16.3, Q17.3, Q3.3, Q5.3, Q7.3, Q9.3, U1.21, U1.3, U1.5
- net IAC_A: no longer X2.14
- net IAC_B: no longer X2.31
- net IAC_C: no longer X2.48
- net IAC_D: no longer X2.15
- net INY1: now also D25.C, Q6.D; no longer D1.C, Q1.4
- net INY2: now also D1.C, Q1.D; no longer D4.C, Q3.4
- net INY3: now also D4.C, Q7.D; no longer D6.C, Q5.4
- net INY4: now also D6.C, Q14.D; no longer D7.C, Q7.4
- net INYL1A: now also R31.2; no longer IC5.3, U1.23
- net INYL2A: now also R33.2; no longer IC5.5, U1.24
- net INYL3A: now also R43.2; no longer IC5.7, U1.25
- net INYL4A: now also R45.2; no longer IC5.9, U1.26
- net MISO: no longer U1.16
- net MOSI: no longer U1.15
- net N$10: now also Q1.G, R34.1; no longer IC5.15, Q13.1
- net N$19: now also Q10.B; no longer Q15.1
- net N$2: now also Q11.B, Q12.B, R31.1; no longer IC5.2, Q1.1
- net N$29: now also Q15.B; no longer Q16.1
- net N$3: now also Q11.E, Q12.E, R32.2; no longer IC5.4, Q3.1
- net N$4: now also Q26.B; no longer Q9.1
- net N$5: now also Q3.B, Q5.B, R33.1; no longer IC5.6, Q5.1
- net N$6: now also Q6.G, R32.1; no longer IC5.10, Q7.1
- net N$7: now also Q16.B; no longer Q17.1
- net N$8: now also Q9.B; no longer Q10.1
- net N$9: now also Q3.E, Q5.E, R34.2; no longer IC5.12, Q11.1
- net PWM: no longer U1.1
- net RCK: no longer U1.11
- net RL1IN: now also D9.C, J1.1, Q26.C; no longer D12.C, D13.A, Q9.4, X2.17
- net RL2IN: now also D12.C, J1.2, Q9.C; no longer D14.C, D15.A, Q10.4, X2.33
- net RL3IN: now also D13.C, J1.3, Q10.C; no longer D20.C, D21.A, Q15.4, X2.16
- net RL4IN: now also D14.C, J1.4, Q15.C; no longer D22.C, D23.A, Q16.4, X2.49
- net RL5IN: now also D15.C, J1.5, Q16.C; no longer D32.C, D33.A, Q17.4, X2.32
- net SCK: no longer U1.17
- net SCK2: no longer U1.10
- net SER: no longer U1.9
- net SS: no longer U1.14
- net TPSM_A: no longer X2.30
- net TPSM_B: no longer X2.47
Routing:
- net 5V: track 215.8 -> 48.0 mm, vias 3 -> 0
- net GND2: track 0.00 -> 130.0 mm
- net INY6: track 0.00 -> 120.2 mm
- net INY5: track 0.00 -> 104.4 mm
- net RL6IN: track 0.00 -> 101.9 mm
- net PWM: track 96.7 -> 0.00 mm, vias 4 -> 0
- net ACC: track 191.9 -> 105.7 mm, vias 5 -> 0
- net ECN2: track 74.4 -> 0.00 mm
- net N$2: track 87.2 -> 16.2 mm, vias 1 -> 0
- net RL1: track 61.8 -> 0.00 mm
- net ECN1: track 61.1 -> 0.00 mm
- net N$3: track 69.1 -> 13.9 mm, vias 1 -> 0
- net RL2: track 51.8 -> 0.15 mm
- net RL4IN: track 88.4 -> 40.6 mm
- net 5V1: track 155.6 -> 115.7 mm
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- removed copper zone on layer 16, net GND
Other:
- board size 149.8 x 100 mm -> 149.9 x 148.8 mm
