File: STM32F rev3/STM32F rev3.sch (KiCad schematic (older format))
At the start: 25 parts, among them J1 USB_B, J2 Tag connect, SW1 SW_Push, U1 MCZ33810EK, U3 STM32F407VGTx, Y1 25MHz

Commit message: WIP v3 on STM32
Connections:
- net labels added: +12V
- net labels removed: +12P, ENC1, SPI2_OSI
Changed lines of the file:
@@
 INY4
 Text Label 7350 3550 0    50   ~ 0
-ENC1
+ECN1
 Text Label 7350 3650 0    50   ~ 0
 ECN2
@@
 Wire Wire Line
 	6000 4700 6300 4700
-$Comp
-L power:+12P #PWR0122
-U 1 1 5FF8B92F
-P 7200 1700
-F 0 "#PWR0122" H 7200 1550 50  0001 C CNN
-F 1 "+12P" H 7215 1873 50  0000 C CNN
-F 2 "" H 7200 1700 50  0001 C CNN
-F 3 "" H 7200 1700 50  0001 C CNN
-	1    7200 1700
-	1    0    0    -1
-$EndComp
 Wire Wire Line
 	7200 1700 7200 1750
-Wire Wire Line
-	7200 1750 7500 1750
 $Comp
 L power:+3.3V #PWR0123
@@
 SPI2_MISO
 Text Label 7350 2050 0    31   ~ 0
-SPI2_OSI
+SPI2_MOSI
 Wire Wire Line
 	7350 2050 7500 2050
@@
 Wire Wire Line
 	10200 2850 10650 2850
+$Comp
+L power:+12V #PWR0102
+U 1 1 5F8CA51B
+P 7200 1700
+F 0 "#PWR0102" H 7200 1550 50  0001 C CNN
+F 1 "+12V" H 7215 1873 50  0000 C CNN
+F 2 "" H 7200 1700 50  0001 C CNN
+F 3 "" H 7200 1700 50  0001 C CNN
+	1    7200 1700
+	1    0    0    -1
+$EndComp
+Wire Wire Line
+	7200 1750 7500 1750
 Wire Wire Line
 	6950 4450 10650 4450

Commit message: V3 WIP
Parts:
- added LOGO1: Logo_Open_Hardware_Large, Symbol:OSHW-Logo2_14.6x12mm_SilkScreen, symbol Graphic:Logo_Open_Hardware_Large
- added SYM1: SYM_Hot_Small, Symbol:KiCad-Logo2_6mm_SilkScreen, symbol Graphic:SYM_Hot_Small
Changed lines of the file:
@@
 Wire Wire Line
 	7200 1750 7500 1750
+$Comp
+L Graphic:Logo_Open_Hardware_Large LOGO1
+U 1 1 5FAF676D
+P 9700 5300
+F 0 "LOGO1" H 9700 5800 50  0001 C CNN
+F 1 "Logo_Open_Hardware_Large" H 9700 4900 50  0001 C CNN
+F 2 "Symbol:OSHW-Logo2_14.6x12mm_SilkScreen" H 9700 5300 50  0001 C CNN
+F 3 "~" H 9700 5300 50  0001 C CNN
+	1    9700 5300
+	1    0    0    -1
+$EndComp
+$Comp
+L Graphic:SYM_Hot_Small SYM1
+U 1 1 5FAFA26F
+P 10650 6050
+F 0 "SYM1" H 10650 6190 50  0001 C CNN
+F 1 "SYM_Hot_Small" H 10650 5925 50  0001 C CNN
+F 2 "Symbol:KiCad-Logo2_6mm_SilkScreen" H 10650 5875 50  0001 C CNN
+F 3 "~" H 10680 5850 50  0001 C CNN
+	1    10650 6050
+	1    0    0    -1
+$EndComp
 Wire Wire Line
 	6950 4450 10650 4450
