File: STM32F rev3/file5F54B133.sch (KiCad schematic (older format))
At the start: 5 parts

Commit message: WIP v3 on STM32
Parts:
- removed D1: D, symbol Device:D
- added C37, C38, C39, C40, C41, C42, C43, C44, C45, C46, C47, C48, C49, C50: 240pF, Capacitor_SMD:C_0603_1608Metric, symbol Device:C_Small
- added D1, D10, D11, D12, D13, D14, D15, D16, D17, D18, D19, D5, D6, D7, D8, D9: DZ2S033X0L, Diode_SMD:D_MiniMELF, symbol Diode:DZ2S033X0L
- added JP1, JP10, JP11, JP12, JP13, JP14, JP15, JP16, JP2, JP3, JP4, JP5, JP6, JP7, JP8, JP9: Jumper_NC_Small, Jumper:SolderJumper-2_P1.3mm_Open_TrianglePad1.0x1.5mm, symbol Device:Jumper_NC_Small
- added R100, R103, R106, R109, R112, R37, R40, R43, R46, R49, R67, R70, R73, R76, R79, R82: 1k 1/10W +-1%, Resistor_SMD:R_0603_1608Metric, symbol Device:R_Small
- added R101, R104, R107, R110, R113, R38, R41, R44, R47, R50, R68, R71, R74, R77, R80, R83: 33k 1/10W +-1%, Resistor_SMD:R_0603_1608Metric, symbol Device:R_Small
- added R102, R105, R108, R111, R36, R39, R42, R45, R48, R66, R69, R72, R75, R78, R81, R99: 16k 1/10W +-1%, Resistor_SMD:R_0603_1608Metric, symbol Device:R_Small
- added R24, R25, R26, R27, R51, R52, R53, R54, R55, R84, R85, R86, R87, R88: 3.32k +-1%, Resistor_SMD:R_0603_1608Metric, symbol Device:R_Small
- added R28, R29, R30, R31, R56, R57, R58, R59, R60, R89, R90, R91, R92, R93: 28.6k +-1%, Resistor_SMD:R_0603_1608Metric, symbol Device:R_Small
- added R32, R33, R34, R35, R61, R62, R63, R64, R65, R94, R95, R96, R97, R98: 2.2k, Resistor_SMD:R_0603_1608Metric, symbol Device:R_Small
- added U10, U11, U12, U13, U14, U15, U16, U17, U18, U19, U2, U20, U21, U22, U23, U24, U25, U26, U27, U28, U29, U30, U31, U32, U33, U34, U35, U36, U37, U8, U9: LM321, Package_TO_SOT_SMD:SOT-23-5, symbol Amplifier_Operational:LM321
- C17: value 0.245nF -> 240pF; footprint (none) -> Capacitor_SMD:C_0603_1608Metric; LCSC (none) -> C185593
- R3: footprint (none) -> Resistor_SMD:R_0603_1608Metric; LCSC (none) -> C234508
- R4: footprint (none) -> Resistor_SMD:R_0603_1608Metric; LCSC (none) -> C217931
- R5: footprint (none) -> Resistor_SMD:R_0603_1608Metric; LCSC (none) -> C309092
Connections:
- net GND: now also C17.2, R3.2, C37.2, C38.2, C39.2, C40.2, C41.2, C42.2, C43.2, C44.2, C45.2, C46.2, C47.2, C48.2, C49.2, C50.2, D1.2 (A), D10.2 (A), D11.2 (A), D12.2 (A), D13.2 (A), D14.2 (A), D15.2 (A), D16.2 (A), D17.2 (A), D18.2 (A), D19.2 (A), D5.2 (A), D6.2 (A), D7.2 (A), D8.2 (A), D9.2 (A), R101.2, R104.2, R107.2, R110.2, R113.2, R24.2, R25.2, R26.2, R27.2, R38.2, R41.2, R44.2, R47.2, R50.2, R51.2, R52.2, R53.2, R54.2, R55.2, R68.2, R71.2, R74.2, R77.2, R80.2, R83.2, R84.2, R85.2, R86.2, R87.2, R88.2, U10.2 (V-), U11.2 (V-), U12.2 (V-), U13.2 (V-), U14.2 (V-), U15.2 (V-), U16.2 (V-), U17.2 (V-), U18.2 (V-), U19.2 (V-), U2.2 (V-), U20.2 (V-), U21.2 (V-), U22.2 (V-), U23.2 (V-), U24.2 (V-), U25.2 (V-), U26.2 (V-), U27.2 (V-), U28.2 (V-), U29.2 (V-), U30.2 (V-), U31.2 (V-), U32.2 (V-), U33.2 (V-), U34.2 (V-), U35.2 (V-), U36.2 (V-), U37.2 (V-), U8.2 (V-), U9.2 (V-)
- net PA0: now also JP2.2
- net PA1: now also JP1.2
- net PA2: now also JP3.2
- net PA3: now also JP4.2
- net PA4: now also JP5.2
- net PA5: now also JP6.2
- net PA6: now also JP7.2
- net PA7: now also JP8.2
- net PB0: now also JP9.2
- net PB1: now also JP10.2
- net PC0: now also JP16.2
- net PC1: now also JP15.2
- net PC2: now also JP14.2
- net PC3: now also JP13.2
- net PC4: now also JP12.2
- net PC5: now also JP11.2
- net 5V_A renamed +5V
- net +5V: now also R28.2, R29.2, R30.2, R31.2, R56.2, R57.2, R58.2, R59.2, R60.2, R89.2, R90.2, R91.2, R92.2, R93.2, U12.5 (V+), U13.5 (V+), U14.5 (V+), U15.5 (V+), U16.5 (V+), U22.5 (V+), U23.5 (V+), U24.5 (V+), U25.5 (V+), U26.5 (V+), U27.5 (V+), U33.5 (V+), U34.5 (V+), U35.5 (V+), U36.5 (V+), U37.5 (V+)
- net IN renamed CONN_3
- net OUT: no longer names the net of R5.1
- net OUT: now also U2.1 (+)
- new net: R36.1, U2.3 (-), U2.4
- new net: R36.2, R37.2
- new net: D1.1 (K), R37.1, R38.1, U12.1 (+)
- new net: JP2.1, U12.3 (-), U12.4
- new net: R32.1, U8.1 (+)
- new net: R39.1, U8.3 (-), U8.4
- new net: R39.2, R40.2
- new net: D5.1 (K), R40.1, R41.1, U13.1 (+)
- new net: JP1.1, U13.3 (-), U13.4
- new net: R33.1, U9.1 (+)
- new net: R42.1, U9.3 (-), U9.4
- new net: R42.2, R43.2
- new net: D6.1 (K), R43.1, R44.1, U14.1 (+)
- new net: JP3.1, U14.3 (-), U14.4
- new net: R34.1, U10.1 (+)
- new net: R45.1, U10.3 (-), U10.4
- new net: R45.2, R46.2
- new net: D7.1 (K), R46.1, R47.1, U15.1 (+)
- new net: JP4.1, U15.3 (-), U15.4
- new net: R35.1, U11.1 (+)
- new net: R48.1, U11.3 (-), U11.4
- new net: R48.2, R49.2
- new net: D8.1 (K), R49.1, R50.1, U16.1 (+)
- new net: JP5.1, U16.3 (-), U16.4
- new net: R61.1, U17.1 (+)
- new net: R66.1, U17.3 (-), U17.4
- new net: R66.2, R67.2
- new net: D9.1 (K), R67.1, R68.1, U22.1 (+)
- new net: JP6.1, U22.3 (-), U22.4
- new net: R62.1, U18.1 (+)
- new net: R69.1, U18.3 (-), U18.4
- new net: R69.2, R70.2
- new net: D10.1 (K), R70.1, R71.1, U23.1 (+)
- new net: JP7.1, U23.3 (-), U23.4
- new net: R63.1, U19.1 (+)
- new net: R72.1, U19.3 (-), U19.4
- new net: R72.2, R73.2
- new net: D11.1 (K), R73.1, R74.1, U24.1 (+)
- new net: JP8.1, U24.3 (-), U24.4
- new net: R64.1, U20.1 (+)
- new net: R75.1, U20.3 (-), U20.4
- new net: R75.2, R76.2
- new net: D12.1 (K), R76.1, R77.1, U25.1 (+)
- new net: JP9.1, U25.3 (-), U25.4
- new net: R65.1, U21.1 (+)
- new net: R78.1, U21.3 (-), U21.4
- new net: R78.2, R79.2
- new net: D13.1 (K), R79.1, R80.1, U26.1 (+)
- new net: JP10.1, U26.3 (-), U26.4
- new net: R94.1, U28.1 (+)
- new net: R99.1, U28.3 (-), U28.4
- new net: R100.2, R99.2
- new net: D15.1 (K), R100.1, R101.1, U33.1 (+)
- new net: JP12.1, U33.3 (-), U33.4
- new net: R95.1, U29.1 (+)
- new net: R102.1, U29.3 (-), U29.4
- new net: R102.2, R103.2
- new net: D16.1 (K), R103.1, R104.1, U34.1 (+)
- new net: JP13.1, U34.3 (-), U34.4
- new net: R96.1, U30.1 (+)
- new net: R105.1, U30.3 (-), U30.4
- new net: R105.2, R106.2
- new net: D17.1 (K), R106.1, R107.1, U35.1 (+)
- new net: JP14.1, U35.3 (-), U35.4
- new net: R97.1, U31.1 (+)
- new net: C49.1, R87.1, R92.1, R97.2
- new net: R108.1, U31.3 (-), U31.4
- new net: R108.2, R109.2
- new net: D18.1 (K), R109.1, R110.1, U36.1 (+)
- new net: JP15.1, U36.3 (-), U36.4
- new net: R98.1, U32.1 (+)
- new net: C50.1, R88.1, R93.1, R98.2
- new net: R111.1, U32.3 (-), U32.4
- new net: R111.2, R112.2
- new net: D19.1 (K), R112.1, R113.1, U37.1 (+)
- new net: JP16.1, U37.3 (-), U37.4
- new net: R81.2, R82.2
- new net: D14.1 (K), R82.1, R83.1, U27.1 (+)
- new net: JP11.1, U27.3 (-), U27.4
- new net +12V: U10.5 (V+), U11.5 (V+), U17.5 (V+), U18.5 (V+), U19.5 (V+), U2.5 (V+), U20.5 (V+), U21.5 (V+), U28.5 (V+), U29.5 (V+), U30.5 (V+), U31.5 (V+), U32.5 (V+), U8.5 (V+), U9.5 (V+)
- new net CONN_10: C44.1, R54.1, R59.1, R64.2
- new net CONN_11: C45.1, R55.1, R60.1, R65.2
- new net CONN_12: C43.1, R53.1, R58.1, R63.2
- new net CONN_13: C46.1, R84.1, R89.1, R94.2
- new net CONN_14: C47.1, R85.1, R90.1, R95.2
- new net CONN_15: C48.1, R86.1, R91.1, R96.2
- new net CONN_4: C37.1, R24.1, R28.1, R32.2
- new net CONN_5: C38.1, R25.1, R29.1, R33.2
- new net CONN_6: C39.1, R26.1, R30.1, R34.2
- new net CONN_7: C40.1, R27.1, R31.1, R35.2
- new net CONN_8: C41.1, R51.1, R56.1, R61.2
- new net CONN_9: C42.1, R52.1, R57.1, R62.2
Other:
- note added: "TODO: VBAT"
- moved on the sheet: C17, R3, R4, R5

Commit message: V3 WIP
Parts:
- removed R112: 1k 1/10W +-1%, Resistor_SMD:R_0603_1608Metric, symbol Device:R_Small
- removed R113: 33k 1/10W +-1%, Resistor_SMD:R_0603_1608Metric, symbol Device:R_Small
- removed R81: 16k 1/10W +-1%, Resistor_SMD:R_0603_1608Metric, symbol Device:R_Small
- removed U36, U37: LM321, Package_TO_SOT_SMD:SOT-23-5, symbol Amplifier_Operational:LM321
- added C?: 240pF, Capacitor_SMD:C_0603_1608Metric, symbol Device:C_Small
- added JP17, JP18, JP19, JP20, JP21, JP22: Jumper_NC_Small, Jumper:SolderJumper-2_P1.3mm_Open_TrianglePad1.0x1.5mm, symbol Device:Jumper_NC_Small
- R108, R111: value 16k 1/10W +-1% -> 10k; LCSC C217760 -> (none)
- R109: value 1k 1/10W +-1% -> 10k; LCSC C217840 -> (none)
- R110: value 33k 1/10W +-1% -> 10k
- R82: value 1k 1/10W +-1% -> 100k 1/10W +-1%
- R83: value 33k 1/10W +-1% -> 20k 1/10W +-1%
Connections:
- net CONN_10: now also C43.1, R53.1, R58.1, R63.2; no longer C44.1, R54.1, R59.1, R64.2
- net CONN_11: now also C44.1, R54.1, R59.1, R64.2; no longer C45.1, R55.1, R60.1, R65.2
- net CONN_12: now also C45.1, R55.1, R60.1, R65.2; no longer C43.1, R53.1, R58.1, R63.2
- net GND: now also R109.1, R111.1, C?.2; no longer R110.2
- net PC0: now also JP19.2, JP22.2; no longer JP16.2
- net CONN_16: now reaches C49.1, R87.1, R92.1, R97.2
- net at R109.2: now also R108.1, JP18.2; no longer R108.2
- net at JP15.1: now also U31.3 (-), JP17.1
- net CONN_17: now reaches C50.1, R88.1, R93.1, R98.2
- net at R111.2: now also R110.1, JP21.2
- net at D19.1 (K): now also JP16.2, U32.4, JP21.1, JP22.1
- net at JP16.1: now also U32.3 (-), JP20.1
- net CONN_18: now reaches R82.2
- net at D14.1 (K), R82.1, R83.1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: now also C?.1
- net PC1: no longer names the net of JP15.2
- net PC1: now also D18.1 (K), U31.4, JP18.1, JP19.1
- new net: JP20.2, R110.2
- new net: JP17.2, R108.2
Other:
- note added: "Solo en puentear si no te utiliza una wideband"
- moved on the sheet: C49, D14, D18, JP11, R82, R83, R87, R92, R97, U27, U31
