File: STM32F rev3/STM32F rev3.kicad_pcb (KiCad board)
At the start: 4 copper layers, 200.2 x 140.2 mm, 80 parts, among them J1 USB_B, J2 Tag connect, J3 502225-0801, Q1 ISL9V5045S3ST, Q2 ISL9V5045S3ST, Q3 ISL9V5045S3ST, Q4 ISL9V5045S3ST, Q5 2N3904, Q6 IRF540N, Q7 IRF540N, SW1 SW_Push, U1 MCZ33810EK, U3 STM32F407VGTx, U4 MIC2940A-3.3WU, U5 MIC2940A-5.0WT, U6 LT4363IMS, U7 MIC2940A-5.0WT, Y1 25MHz

Commit message: WIP v3 on STM32
Parts:
- removed TP10, TP3, TP4, TP5, TP6, TP7, TP8, TP9: TestPoint, TestPoint:TestPoint_Pad_1.5x1.5mm
- added C17: 240pF, Capacitor_SMD:C_0603_1608Metric, F.Cu at (152.9, 71.6)
- added C37: 240pF, Capacitor_SMD:C_0603_1608Metric, F.Cu at (152.3, 90.0)
- added C38: 240pF, Capacitor_SMD:C_0603_1608Metric, F.Cu at (154.1, 98.7)
- added C39: 240pF, Capacitor_SMD:C_0603_1608Metric, F.Cu at (161.0, 113.7)
- added C40: 240pF, Capacitor_SMD:C_0603_1608Metric, F.Cu at (146.2, 71.6)
- added C41: 240pF, Capacitor_SMD:C_0603_1608Metric, F.Cu at (147.5, 92.9)
- added C42: 240pF, Capacitor_SMD:C_0603_1608Metric, F.Cu at (145.8, 112.8)
- added C43: 240pF, Capacitor_SMD:C_0603_1608Metric, F.Cu at (139.1, 113.2)
- added C44: 240pF, Capacitor_SMD:C_0603_1608Metric, F.Cu at (138.6, 71.6)
- added C45: 240pF, Capacitor_SMD:C_0603_1608Metric, F.Cu at (138.6, 91.7)
- added C46: 240pF, Capacitor_SMD:C_0603_1608Metric, F.Cu at (110.4, 69.9)
- added C47: 240pF, Capacitor_SMD:C_0603_1608Metric, F.Cu at (110.4, 88.9)
- added C48: 240pF, Capacitor_SMD:C_0603_1608Metric, F.Cu at (112.6, 107.1)
- added C49: 240pF, Capacitor_SMD:C_0603_1608Metric, F.Cu at (40.0, 113.3)
- added C50: 240pF, Capacitor_SMD:C_0603_1608Metric, F.Cu at (35.9, 113.3)
- added D1: DZ2S033X0L, Diode_SMD:D_MiniMELF, F.Cu at (153.4, 86.0)
- added D10: DZ2S033X0L, Diode_SMD:D_MiniMELF, F.Cu at (153.3, 117.9)
- added D11: DZ2S033X0L, Diode_SMD:D_MiniMELF, F.Cu at (140.1, 126.8)
- added D12: DZ2S033X0L, Diode_SMD:D_MiniMELF, F.Cu at (142.2, 84.4)
- added D13: DZ2S033X0L, Diode_SMD:D_MiniMELF, F.Cu at (136.9, 105.7)
- added D14: DZ2S033X0L, Diode_SMD:D_MiniMELF, F.Cu at (43.6, 77.3)
- added D15: DZ2S033X0L, Diode_SMD:D_MiniMELF, F.Cu at (114.6, 86.3)
- added D16: DZ2S033X0L, Diode_SMD:D_MiniMELF, F.Cu at (43.5, 90.0)
- added D17: DZ2S033X0L, Diode_SMD:D_MiniMELF, F.Cu at (104.5, 128.0)
- added D18: DZ2S033X0L, Diode_SMD:D_MiniMELF, F.Cu at (43.5, 83.5)
- added D19: DZ2S033X0L, Diode_SMD:D_MiniMELF, F.Cu at (43.6, 80.5)
- added D4: SMAJ58CA, Diode_SMD:D_SMA, F.Cu at (213.5, 49.2)
- added D5: DZ2S033X0L, Diode_SMD:D_MiniMELF, F.Cu at (161.1, 93.7)
- added D6: DZ2S033X0L, Diode_SMD:D_MiniMELF, F.Cu at (161.6, 109.4)
- added D7: DZ2S033X0L, Diode_SMD:D_MiniMELF, F.Cu at (156.8, 121.4)
- added D8: DZ2S033X0L, Diode_SMD:D_MiniMELF, F.Cu at (146.1, 86.1)
- added D9: DZ2S033X0L, Diode_SMD:D_MiniMELF, F.Cu at (147.0, 105.7)
- added JP1: Jumper_NC_Small, Jumper:SolderJumper-2_P1.3mm_Open_TrianglePad1.0x1.5mm, F.Cu at (160.5, 98.8)
- added JP10: Jumper_NC_Small, Jumper:SolderJumper-2_P1.3mm_Open_TrianglePad1.0x1.5mm, F.Cu at (137.1, 110.2)
- added JP11: Jumper_NC_Small, Jumper:SolderJumper-2_P1.3mm_Open_TrianglePad1.0x1.5mm, F.Cu at (39.0, 126.0)
- added JP12: Jumper_NC_Small, Jumper:SolderJumper-2_P1.3mm_Open_TrianglePad1.0x1.5mm, F.Cu at (110.2, 85.6)
- added JP13: Jumper_NC_Small, Jumper:SolderJumper-2_P1.3mm_Open_TrianglePad1.0x1.5mm, F.Cu at (110.4, 100.8)
- added JP14: Jumper_NC_Small, Jumper:SolderJumper-2_P1.3mm_Open_TrianglePad1.0x1.5mm, F.Cu at (52.0, 115.3)
- added JP15: Jumper_NC_Small, Jumper:SolderJumper-2_P1.3mm_Open_TrianglePad1.0x1.5mm, F.Cu at (43.3, 126.0)
- added JP16: Jumper_NC_Small, Jumper:SolderJumper-2_P1.3mm_Open_TrianglePad1.0x1.5mm, F.Cu at (47.7, 122.4)
- added JP2: Jumper_NC_Small, Jumper:SolderJumper-2_P1.3mm_Open_TrianglePad1.0x1.5mm, F.Cu at (158.3, 85.4)
- added JP3: Jumper_NC_Small, Jumper:SolderJumper-2_P1.3mm_Open_TrianglePad1.0x1.5mm, F.Cu at (157.0, 112.1)
- added JP4: Jumper_NC_Small, Jumper:SolderJumper-2_P1.3mm_Open_TrianglePad1.0x1.5mm, F.Cu at (168.1, 115.6)
- added JP5: Jumper_NC_Small, Jumper:SolderJumper-2_P1.3mm_Open_TrianglePad1.0x1.5mm, F.Cu at (149.4, 89.5)
- added JP6: Jumper_NC_Small, Jumper:SolderJumper-2_P1.3mm_Open_TrianglePad1.0x1.5mm, F.Cu at (150.8, 108.9)
- added JP7: Jumper_NC_Small, Jumper:SolderJumper-2_P1.3mm_Open_TrianglePad1.0x1.5mm, F.Cu at (150.1, 123.1)
- added JP8: Jumper_NC_Small, Jumper:SolderJumper-2_P1.3mm_Open_TrianglePad1.0x1.5mm, F.Cu at (151.0, 126.9)
- added JP9: Jumper_NC_Small, Jumper:SolderJumper-2_P1.3mm_Open_TrianglePad1.0x1.5mm, F.Cu at (138.8, 88.4)
- added R100: 1k 1/10W +-1%, Resistor_SMD:R_0603_1608Metric, F.Cu at (113.7, 78.8)
- added R101: 33k 1/10W +-1%, Resistor_SMD:R_0603_1608Metric, F.Cu at (114.4, 81.3)
- added R102: 16k 1/10W +-1%, Resistor_SMD:R_0603_1608Metric, F.Cu at (114.5, 94.0)
- added R103: 1k 1/10W +-1%, Resistor_SMD:R_0603_1608Metric, F.Cu at (112.0, 95.1)
- added R104: 33k 1/10W +-1%, Resistor_SMD:R_0603_1608Metric, F.Cu at (110.3, 97.4)
- added R105: 16k 1/10W +-1%, Resistor_SMD:R_0603_1608Metric, F.Cu at (96.8, 115.8)
- added R106: 1k 1/10W +-1%, Resistor_SMD:R_0603_1608Metric, F.Cu at (99.2, 122.2)
- added R107: 33k 1/10W +-1%, Resistor_SMD:R_0603_1608Metric, F.Cu at (107.2, 121.5)
- added R108: 16k 1/10W +-1%, Resistor_SMD:R_0603_1608Metric, F.Cu at (36.8, 104.8)
- added R109: 1k 1/10W +-1%, Resistor_SMD:R_0603_1608Metric, F.Cu at (32.7, 104.5)
- added R110: 33k 1/10W +-1%, Resistor_SMD:R_0603_1608Metric, F.Cu at (41.3, 60.9)
- added R111: 16k 1/10W +-1%, Resistor_SMD:R_0603_1608Metric, F.Cu at (41.4, 65.9)
- added R112: 1k 1/10W +-1%, Resistor_SMD:R_0603_1608Metric, F.Cu at (37.6, 68.5)
- added R113: 33k 1/10W +-1%, Resistor_SMD:R_0603_1608Metric, F.Cu at (31.9, 107.3)
- added R24: 3.32k +-1%, Resistor_SMD:R_0603_1608Metric, F.Cu at (152.3, 91.6)
- added R25: 3.32k +-1%, Resistor_SMD:R_0603_1608Metric, F.Cu at (154.1, 100.3)
- added R26: 3.32k +-1%, Resistor_SMD:R_0603_1608Metric, F.Cu at (161.0, 115.3)
- added R27: 3.32k +-1%, Resistor_SMD:R_0603_1608Metric, F.Cu at (146.2, 73.3)
- added R28: 28.6k +-1%, Resistor_SMD:R_0603_1608Metric, F.Cu at (152.3, 93.2)
- added R29: 28.6k +-1%, Resistor_SMD:R_0603_1608Metric, F.Cu at (154.1, 101.9)
- added R3: 3.32k +-1%, Resistor_SMD:R_0603_1608Metric, F.Cu at (152.9, 73.2)
- added R30: 28.6k +-1%, Resistor_SMD:R_0603_1608Metric, F.Cu at (161.0, 117.0)
- added R31: 28.6k +-1%, Resistor_SMD:R_0603_1608Metric, F.Cu at (146.2, 74.9)
- added R32: 2.2k, Resistor_SMD:R_0603_1608Metric, F.Cu at (151.6, 95.6)
- added R33: 2.2k, Resistor_SMD:R_0603_1608Metric, F.Cu at (153.3, 104.2)
- added R34: 2.2k, Resistor_SMD:R_0603_1608Metric, F.Cu at (160.3, 119.4)
- added R35: 2.2k, Resistor_SMD:R_0603_1608Metric, F.Cu at (145.4, 77.3)
- added R36: 16k 1/10W +-1%, Resistor_SMD:R_0603_1608Metric, F.Cu at (155.4, 80.3)
- added R37: 1k 1/10W +-1%, Resistor_SMD:R_0603_1608Metric, F.Cu at (152.0, 80.3)
- added R38: 33k 1/10W +-1%, Resistor_SMD:R_0603_1608Metric, F.Cu at (151.3, 82.6)
- added R39: 16k 1/10W +-1%, Resistor_SMD:R_0603_1608Metric, F.Cu at (157.7, 96.0)
- added R4: 28.6k +-1%, Resistor_SMD:R_0603_1608Metric, F.Cu at (152.9, 74.7)
- added R40: 1k 1/10W +-1%, Resistor_SMD:R_0603_1608Metric, F.Cu at (157.7, 92.8)
- added R41: 33k 1/10W +-1%, Resistor_SMD:R_0603_1608Metric, F.Cu at (157.7, 89.5)
- added R42: 16k 1/10W +-1%, Resistor_SMD:R_0603_1608Metric, F.Cu at (160.4, 105.9)
- added R43: 1k 1/10W +-1%, Resistor_SMD:R_0603_1608Metric, F.Cu at (160.3, 104.1)
- added R44: 33k 1/10W +-1%, Resistor_SMD:R_0603_1608Metric, F.Cu at (160.3, 102.5)
- added R45: 16k 1/10W +-1%, Resistor_SMD:R_0603_1608Metric, F.Cu at (160.3, 122.5)
- added R46: 1k 1/10W +-1%, Resistor_SMD:R_0603_1608Metric, F.Cu at (162.8, 123.2)
- added R47: 33k 1/10W +-1%, Resistor_SMD:R_0603_1608Metric, F.Cu at (165.9, 123.2)
- added R48: 16k 1/10W +-1%, Resistor_SMD:R_0603_1608Metric, F.Cu at (146.2, 80.5)
- added R49: 1k 1/10W +-1%, Resistor_SMD:R_0603_1608Metric, F.Cu at (145.4, 83.1)
- added R5: 2.2k, Resistor_SMD:R_0603_1608Metric, F.Cu at (152.1, 77.0)
- added R50: 33k 1/10W +-1%, Resistor_SMD:R_0603_1608Metric, F.Cu at (148.3, 83.1)
- added R51: 3.32k +-1%, Resistor_SMD:R_0603_1608Metric, F.Cu at (147.5, 94.5)
- added R52: 3.32k +-1%, Resistor_SMD:R_0603_1608Metric, F.Cu at (145.8, 114.6)
- added R53: 3.32k +-1%, Resistor_SMD:R_0603_1608Metric, F.Cu at (139.2, 114.9)
- added R54: 3.32k +-1%, Resistor_SMD:R_0603_1608Metric, F.Cu at (138.6, 73.3)
- added R55: 3.32k +-1%, Resistor_SMD:R_0603_1608Metric, F.Cu at (138.6, 93.4)
- added R56: 28.6k +-1%, Resistor_SMD:R_0603_1608Metric, F.Cu at (147.5, 96.1)
- added R57: 28.6k +-1%, Resistor_SMD:R_0603_1608Metric, F.Cu at (145.8, 116.3)
- added R58: 28.6k +-1%, Resistor_SMD:R_0603_1608Metric, F.Cu at (139.2, 116.5)
- added R59: 28.6k +-1%, Resistor_SMD:R_0603_1608Metric, F.Cu at (138.6, 75.1)
- added R60: 28.6k +-1%, Resistor_SMD:R_0603_1608Metric, F.Cu at (138.6, 95.1)
- added R61: 2.2k, Resistor_SMD:R_0603_1608Metric, F.Cu at (145.5, 98.5)
- added R62: 2.2k, Resistor_SMD:R_0603_1608Metric, F.Cu at (145.0, 118.9)
- added R63: 2.2k, Resistor_SMD:R_0603_1608Metric, F.Cu at (137.7, 118.9)
- added R64: 2.2k, Resistor_SMD:R_0603_1608Metric, F.Cu at (138.6, 76.7)
- added R65: 2.2k, Resistor_SMD:R_0603_1608Metric, F.Cu at (138.6, 96.9)
- added R66: 16k 1/10W +-1%, Resistor_SMD:R_0603_1608Metric, F.Cu at (149.2, 101.9)
- added R67: 1k 1/10W +-1%, Resistor_SMD:R_0603_1608Metric, F.Cu at (146.0, 101.9)
- added R68: 33k 1/10W +-1%, Resistor_SMD:R_0603_1608Metric, F.Cu at (146.0, 103.5)
- added R69: 16k 1/10W +-1%, Resistor_SMD:R_0603_1608Metric, F.Cu at (150.1, 116.8)
- added R70: 1k 1/10W +-1%, Resistor_SMD:R_0603_1608Metric, F.Cu at (146.8, 118.9)
- added R71: 33k 1/10W +-1%, Resistor_SMD:R_0603_1608Metric, F.Cu at (149.4, 119.6)
- added R72: 16k 1/10W +-1%, Resistor_SMD:R_0603_1608Metric, F.Cu at (139.0, 122.0)
- added R73: 1k 1/10W +-1%, Resistor_SMD:R_0603_1608Metric, F.Cu at (139.0, 123.7)
- added R74: 33k 1/10W +-1%, Resistor_SMD:R_0603_1608Metric, F.Cu at (141.6, 122.9)
- added R75: 16k 1/10W +-1%, Resistor_SMD:R_0603_1608Metric, F.Cu at (143.2, 75.9)
- added R76: 1k 1/10W +-1%, Resistor_SMD:R_0603_1608Metric, F.Cu at (141.7, 79.6)
- added R77: 33k 1/10W +-1%, Resistor_SMD:R_0603_1608Metric, F.Cu at (138.6, 79.6)
- added R78: 16k 1/10W +-1%, Resistor_SMD:R_0603_1608Metric, F.Cu at (142.3, 96.1)
- added R79: 1k 1/10W +-1%, Resistor_SMD:R_0603_1608Metric, F.Cu at (142.7, 99.3)
- added R80: 33k 1/10W +-1%, Resistor_SMD:R_0603_1608Metric, F.Cu at (139.6, 104.8)
- added R81: 16k 1/10W +-1%, Resistor_SMD:R_0603_1608Metric, F.Cu at (41.6, 68.5)
- added R82: 1k 1/10W +-1%, Resistor_SMD:R_0603_1608Metric, F.Cu at (35.9, 107.3)
- added R83: 33k 1/10W +-1%, Resistor_SMD:R_0603_1608Metric, F.Cu at (37.6, 71.0)
- added R84: 3.32k +-1%, Resistor_SMD:R_0603_1608Metric, F.Cu at (110.4, 71.6)
- added R85: 3.32k +-1%, Resistor_SMD:R_0603_1608Metric, F.Cu at (110.4, 90.6)
- added R86: 3.32k +-1%, Resistor_SMD:R_0603_1608Metric, F.Cu at (108.5, 107.3)
- added R87: 3.32k +-1%, Resistor_SMD:R_0603_1608Metric, F.Cu at (37.4, 63.4)
- added R88: 3.32k +-1%, Resistor_SMD:R_0603_1608Metric, F.Cu at (36.9, 92.7)
- added R89: 28.6k +-1%, Resistor_SMD:R_0603_1608Metric, F.Cu at (110.4, 73.3)
- added R90: 28.6k +-1%, Resistor_SMD:R_0603_1608Metric, F.Cu at (110.3, 92.2)
- added R91: 28.6k +-1%, Resistor_SMD:R_0603_1608Metric, F.Cu at (108.3, 111.6)
- added R92: 28.6k +-1%, Resistor_SMD:R_0603_1608Metric, F.Cu at (36.4, 116.7)
- added R93: 28.6k +-1%, Resistor_SMD:R_0603_1608Metric, F.Cu at (41.3, 58.4)
- added R94: 2.2k, Resistor_SMD:R_0603_1608Metric, F.Cu at (109.6, 75.7)
- added R95: 2.2k, Resistor_SMD:R_0603_1608Metric, F.Cu at (109.6, 94.6)
- added R96: 2.2k, Resistor_SMD:R_0603_1608Metric, F.Cu at (98.8, 102.7)
- added R97: 2.2k, Resistor_SMD:R_0603_1608Metric, F.Cu at (36.9, 90.2)
- added R98: 2.2k, Resistor_SMD:R_0603_1608Metric, F.Cu at (37.3, 60.9)
- added R99: 16k 1/10W +-1%, Resistor_SMD:R_0603_1608Metric, F.Cu at (110.4, 78.8)
- added U10: LM321, Package_TO_SOT_SMD:SOT-23-5, F.Cu at (163.2, 119.9)
- added U11: LM321, Package_TO_SOT_SMD:SOT-23-5, F.Cu at (148.2, 77.6)
- added U12: LM321, Package_TO_SOT_SMD:SOT-23-5, F.Cu at (154.9, 82.9)
- added U13: LM321, Package_TO_SOT_SMD:SOT-23-5, F.Cu at (160.6, 89.2)
- added U14: LM321, Package_TO_SOT_SMD:SOT-23-5, F.Cu at (156.6, 108.8)
- added U15: LM321, Package_TO_SOT_SMD:SOT-23-5, F.Cu at (167.3, 119.8)
- added U16: LM321, Package_TO_SOT_SMD:SOT-23-5, F.Cu at (145.3, 89.5)
- added U17: LM321, Package_TO_SOT_SMD:SOT-23-5, F.Cu at (148.9, 99.1)
- added U18: LM321, Package_TO_SOT_SMD:SOT-23-5, F.Cu at (149.9, 114.0)
- added U19: LM321, Package_TO_SOT_SMD:SOT-23-5, F.Cu at (140.9, 119.3)
- added U2: LM321, Package_TO_SOT_SMD:SOT-23-5, F.Cu at (155.1, 77.5)
- added U20: LM321, Package_TO_SOT_SMD:SOT-23-5, F.Cu at (142.1, 72.3)
- added U21: LM321, Package_TO_SOT_SMD:SOT-23-5, F.Cu at (138.9, 99.8)
- added U22: LM321, Package_TO_SOT_SMD:SOT-23-5, F.Cu at (146.2, 108.9)
- added U23: LM321, Package_TO_SOT_SMD:SOT-23-5, F.Cu at (146.2, 122.6)
- added U24: LM321, Package_TO_SOT_SMD:SOT-23-5, F.Cu at (146.1, 126.4)
- added U25: LM321, Package_TO_SOT_SMD:SOT-23-5, F.Cu at (138.9, 83.5)
- added U26: LM321, Package_TO_SOT_SMD:SOT-23-5, F.Cu at (140.3, 109.1)
- added U27: LM321, Package_TO_SOT_SMD:SOT-23-5, F.Cu at (49.1, 90.7)
- added U28: LM321, Package_TO_SOT_SMD:SOT-23-5, F.Cu at (112.9, 76.0)
- added U29: LM321, Package_TO_SOT_SMD:SOT-23-5, F.Cu at (114.3, 91.2)
- added U30: LM321, Package_TO_SOT_SMD:SOT-23-5, F.Cu at (99.6, 110.5)
- added U31: LM321, Package_TO_SOT_SMD:SOT-23-5, F.Cu at (46.1, 109.3)
- added U32: LM321, Package_TO_SOT_SMD:SOT-23-5, F.Cu at (50.9, 101.4)
- added U33: LM321, Package_TO_SOT_SMD:SOT-23-5, F.Cu at (110.7, 81.7)
- added U34: LM321, Package_TO_SOT_SMD:SOT-23-5, F.Cu at (114.8, 98.0)
- added U35: LM321, Package_TO_SOT_SMD:SOT-23-5, F.Cu at (109.5, 132.0)
- added U36: LM321, Package_TO_SOT_SMD:SOT-23-5, F.Cu at (49.8, 79.9)
- added U37: LM321, Package_TO_SOT_SMD:SOT-23-5, F.Cu at (41.2, 109.8)
- added U8: LM321, Package_TO_SOT_SMD:SOT-23-5, F.Cu at (154.4, 95.9)
- added U9: LM321, Package_TO_SOT_SMD:SOT-23-5, F.Cu at (156.6, 105.0)
- D2, D3: footprint Diode_THT:D_DO-35_SOD27_P7.62mm_Horizontal -> Diode_SMD:D_0805_2012Metric
- Q5: footprint Package_TO_SOT_THT:TO-92_Inline -> Package_TO_SOT_SMD:TSOT-23
- moved C33 97.4 mm to (180.6, 43.2)
- moved R20 93.6 mm to (180.6, 44.7), turned to 180 degrees
- moved R18 85.5 mm to (180.6, 61.0), turned to 180 degrees
- moved R19 68.4 mm to (179.6, 74.9)
- moved C36 68.2 mm to (216.5, 135.6)
- moved R17 67.9 mm to (179.6, 72.9), turned to 180 degrees
- moved D2 60.9 mm to (183.0, 70.9)
- moved D3 60.0 mm to (176.8, 73.8), turned to 270 degrees
- moved R22 57.8 mm to (207.9, 124.1), turned to 90 degrees
- moved R23 53.2 mm to (207.1, 121.7)
- moved Q5 52.6 mm to (183.1, 74.4), turned to 270 degrees
- moved C10 18.4 mm to (76.7, 159.6)
- moved C13 18.4 mm to (76.8, 166.4)
- moved C14 18.4 mm to (72.2, 159.6)
- moved Y1 18.4 mm to (54.7, 169.3)
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Connections:
- J3 pad 23: CONN_23 -> GND
- J3 pad 24: CONN_24 -> GND
- J3 pad 25: CONN_25 -> GND
- J3 pad 26: CONN_26 -> GND
- J3 pad 27: CONN_27 -> GND
- J3 pad 28: CONN_28 -> GND
- J3 pad 29: CONN_29 -> GND
- J3 pad 30: CONN_30 -> GND
- J3 pad 31: CONN_31 -> GND
- J3 pad 32: CONN_32 -> GND
- J3 pad 33: CONN_33 -> GND
- J3 pad 34: CONN_34 -> GND
- J3 pad 35: CONN_35 -> GND
- J3 pad 36: CONN_36 -> GND
- J3 pad 37: CONN_37 -> GND
- J3 pad 38: CONN_38 -> GND
- J3 pad 59: CONN_59 -> +12VA
- J3 pad 61: +12VA -> CONN_61
- U1 pad 24: /ENC1 -> /ECN1
- U1 pad 25: +12P -> +12V
- U1 pad 6: /SPI2_OSI -> /SPI2_MOSI
- U6 pad 5: Net-(Q5-Pad3) -> Net-(D4-Pad1)
Routing:
- net GND: track 14.0 -> 266.4 mm, vias 16 -> 61
- net Net-(D4-Pad1): track 0.00 -> 155.1 mm, vias 0 -> 3
- net +12VA: track 0.00 -> 143.0 mm
- net Net-(C33-Pad1): track 0.00 -> 124.4 mm, vias 0 -> 4
- net +12V: track 23.6 -> 146.4 mm, vias 0 -> 13
- net Net-(C22-Pad2): track 0.00 -> 114.3 mm
- net Net-(Q7-Pad2): track 14.1 -> 118.4 mm, vias 0 -> 2
- net /Sheet5FA9324A/GD3: track 0.00 -> 73.4 mm, vias 0 -> 4
- net +5V: track 0.00 -> 66.3 mm, vias 0 -> 23
- net CONN_6: track 0.00 -> 63.2 mm, vias 0 -> 1
- net /Sheet5FA9324A/FB1: track 3.54 -> 66.4 mm, vias 0 -> 2
- net /Sheet5FA9324A/FB3: track 3.18 -> 65.3 mm, vias 0 -> 2
- net /Sheet5FA9324A/GD1: track 0.00 -> 59.3 mm, vias 0 -> 2
- net CONN_12: track 0.00 -> 59.0 mm, vias 0 -> 1
- net CONN_9: track 0.00 -> 58.8 mm, vias 0 -> 1
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- added copper zone on In2.Cu, net +12V
- added copper zone on In1.Cu, net +5V
- added copper zone on B.Cu, net GND
Other:
- board text added: "can"
- board text added: "ckp"
- board text added: "cmp"
- board text added: "pap"
- board text added: "pwm?"
- board text added: "relays"

Commit message: V3 WIP
Parts:
- removed R112: 1k 1/10W +-1%, Resistor_SMD:R_0603_1608Metric
- removed R113: 33k 1/10W +-1%, Resistor_SMD:R_0603_1608Metric
- removed R81: 16k 1/10W +-1%, Resistor_SMD:R_0603_1608Metric
- removed U36, U37: LM321, Package_TO_SOT_SMD:SOT-23-5
- added C51: 240pF, Capacitor_SMD:C_0603_1608Metric, F.Cu at (89.1, 123.6)
- added JP17: Jumper_NC_Small, Jumper:SolderJumper-2_P1.3mm_Open_TrianglePad1.0x1.5mm, F.Cu at (96.4, 86.1)
- added JP18: Jumper_NC_Small, Jumper:SolderJumper-2_P1.3mm_Open_TrianglePad1.0x1.5mm, F.Cu at (100.4, 86.1)
- added JP19: Jumper_NC_Small, Jumper:SolderJumper-2_P1.3mm_Open_TrianglePad1.0x1.5mm, F.Cu at (100.4, 89.4)
- added JP20: Jumper_NC_Small, Jumper:SolderJumper-2_P1.3mm_Open_TrianglePad1.0x1.5mm, F.Cu at (96.4, 108.6)
- added JP21: Jumper_NC_Small, Jumper:SolderJumper-2_P1.3mm_Open_TrianglePad1.0x1.5mm, F.Cu at (100.4, 108.6)
- added JP22: Jumper_NC_Small, Jumper:SolderJumper-2_P1.3mm_Open_TrianglePad1.0x1.5mm, F.Cu at (100.4, 111.9)
- added LOGO1: Logo_Open_Hardware_Large, Symbol:OSHW-Logo2_14.6x12mm_SilkScreen, F.Cu at (209.7, 150.2)
- added SYM1: SYM_Hot_Small, Symbol:KiCad-Logo2_6mm_SilkScreen, F.Cu at (192.2, 150.7)
- R108, R111: value 16k 1/10W +-1% -> 10k
- R109: value 1k 1/10W +-1% -> 10k
- R110: value 33k 1/10W +-1% -> 10k
- R82: value 1k 1/10W +-1% -> 100k 1/10W +-1%
- R83: value 33k 1/10W +-1% -> 20k 1/10W +-1%
- moved C33 86.8 mm to (200.2, 127.7)
- moved R20 85.0 mm to (204.2, 126.3), turned to 0 degrees
- moved R92 76.4 mm to (100.6, 75.4), turned to 180 degrees
- moved R98 74.2 mm to (100.6, 99.5)
- moved C49 73.4 mm to (100.6, 72.0), turned to 180 degrees
- moved JP15 71.9 mm to (100.4, 82.3)
- moved R93 71.3 mm to (100.6, 97.9), turned to 180 degrees
- moved R83 71.0 mm to (88.1, 120.9), turned to 90 degrees
- moved R18 70.4 mm to (208.2, 125.8), turned to 0 degrees
- moved D16 69.6 mm to (112.8, 95.8), turned to 270 degrees
- moved C50 67.3 mm to (100.6, 94.5), turned to 180 degrees
- moved D14 67.1 mm to (90.0, 125.7), turned to 180 degrees
- moved R110 66.4 mm to (93.7, 101.5), turned to 270 degrees
- moved R97 65.0 mm to (100.6, 77.1)
- moved R109 64.6 mm to (92.1, 79.1), turned to 90 degrees
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Connections:
- C18 pad 1: CONN_1 -> CONN_62
- C19 pad 1: CONN_2 -> CONN_42
- C20 pad 1: CONN_21 -> CONN_61
- C21 pad 1: CONN_22 -> CONN_41
- C23 pad 1: CONN_21 -> CONN_61
- C24 pad 1: CONN_22 -> CONN_41
- C25 pad 1: CONN_1 -> CONN_62
- C26 pad 1: CONN_2 -> CONN_42
- C27 pad 2: CONN_41 -> CONN_22
- C28 pad 2: CONN_61 -> CONN_21
- C29 pad 2: CONN_42 -> CONN_2
- C30 pad 2: CONN_62 -> CONN_1
- C43 pad 1: CONN_12 -> CONN_10
- C44 pad 1: CONN_10 -> CONN_11
- C45 pad 1: CONN_11 -> CONN_12
- C49 pad 1: Net-(C49-Pad1) -> CONN_16
- C50 pad 1: Net-(C50-Pad1) -> CONN_17
- JP15 pad 2: /Sensores/PC1 -> Net-(D18-Pad1)
- JP16 pad 2: /Sensores/PC0 -> Net-(D19-Pad1)
- Q1 pad 2: CONN_2 -> CONN_42
- Q2 pad 2: CONN_1 -> CONN_62
- Q3 pad 2: CONN_21 -> CONN_61
- Q4 pad 2: CONN_22 -> CONN_41
- R108 pad 1: Net-(R108-Pad1) -> Net-(JP18-Pad2)
- R108 pad 2: Net-(R108-Pad2) -> Net-(JP17-Pad2)
- R109 pad 1: Net-(D18-Pad1) -> GND
- R109 pad 2: Net-(R108-Pad2) -> Net-(JP18-Pad2)
- R110 pad 1: Net-(D18-Pad1) -> Net-(JP21-Pad2)
- R110 pad 2: GND -> Net-(JP20-Pad2)
- R111 pad 1: Net-(R111-Pad1) -> GND
- R111 pad 2: Net-(R111-Pad2) -> Net-(JP21-Pad2)
- R13 pad 2: CONN_1 -> CONN_62
- R14 pad 2: CONN_2 -> CONN_42
- R15 pad 2: CONN_21 -> CONN_61
- R16 pad 2: CONN_22 -> CONN_41
- R53 pad 1: CONN_12 -> CONN_10
- R54 pad 1: CONN_10 -> CONN_11
- R55 pad 1: CONN_11 -> CONN_12
- R58 pad 1: CONN_12 -> CONN_10
- R59 pad 1: CONN_10 -> CONN_11
- R60 pad 1: CONN_11 -> CONN_12
- R63 pad 2: CONN_12 -> CONN_10
- R64 pad 2: CONN_10 -> CONN_11
- R65 pad 2: CONN_11 -> CONN_12
- R82 pad 2: Net-(R81-Pad2) -> CONN_18
- R87 pad 1: Net-(C49-Pad1) -> CONN_16
- R88 pad 1: Net-(C50-Pad1) -> CONN_17
- R92 pad 1: Net-(C49-Pad1) -> CONN_16
- R93 pad 1: Net-(C50-Pad1) -> CONN_17
- R97 pad 2: Net-(C49-Pad1) -> CONN_16
- R98 pad 2: Net-(C50-Pad1) -> CONN_17
- U1 pad 1: CONN_62 -> CONN_1
- U1 pad 16: CONN_42 -> CONN_2
- U1 pad 17: CONN_41 -> CONN_22
- U1 pad 32: CONN_61 -> CONN_21
- U31 pad 3: Net-(R108-Pad1) -> Net-(JP15-Pad1)
- U31 pad 4: Net-(R108-Pad1) -> Net-(D18-Pad1)
- U32 pad 3: Net-(R111-Pad1) -> Net-(JP16-Pad1)
- U32 pad 4: Net-(R111-Pad1) -> Net-(D19-Pad1)
Routing:
- net Net-(D4-Pad1): track 155.1 -> 29.6 mm, vias 3 -> 0
- net Net-(C33-Pad1): track 124.4 -> 0.00 mm, vias 4 -> 0
- net Net-(C22-Pad2): track 114.3 -> 0.00 mm
- net Net-(Q7-Pad2): track 118.4 -> 6.52 mm, vias 2 -> 0
- net +12V: track 146.4 -> 53.1 mm, vias 13 -> 15
- net CONN_21: track 96.8 -> 5.83 mm, vias 3 -> 0
- net CONN_22: track 87.8 -> 5.61 mm, vias 2 -> 0
- net CONN_1: track 75.5 -> 2.07 mm, vias 2 -> 0
- net /Sheet5FA9324A/GD3: track 73.4 -> 0.00 mm, vias 4 -> 0
- net CONN_42: track 103.8 -> 35.8 mm, vias 1 -> 6
- net /Sheet5FA9324A/FB1: track 66.4 -> 0.00 mm, vias 2 -> 0
- net CONN_18: track 0.00 -> 64.3 mm, vias 0 -> 1
- net /Sheet5FA9324A/FB3: track 65.3 -> 3.18 mm, vias 2 -> 0
- net /Sheet5FA9324A/GD1: track 59.3 -> 0.00 mm, vias 2 -> 0
- net CONN_2: track 62.3 -> 3.40 mm
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- added copper zone on B.Cu, net +5V
- added copper zone on B.Cu, net CONN_41
- added copper zone on B.Cu, net CONN_42
- added copper zone on B.Cu, net CONN_61
- added copper zone on B.Cu, net CONN_62
- removed copper zone on In1.Cu, net +5V
- removed copper zone on B.Cu, net GND
Other:
- board text added: "AIN0"
- board text added: "AIN1"
- board text added: "AIN10"
- board text added: "AIN11"
- board text added: "AIN12"
- board text added: "AIN2"
- board text added: "AIN3"
- board text added: "AIN4"
- board text added: "AIN5"
- board text added: "AIN6"
- board text added: "AIN7"
- board text added: "AIN8"
- board text added: "AIN9"
- board text added: "Battery"
- board text added: "CAN"
- board text added: "CKP"
- board text added: "CMP"
- board text added: "CMP / CKP MODS / TESTING"
- board text added: "ENABLE"
- board text added: "Enable"
- board text added: "INPUT ENABLE"
- board text added: "O2 Sensor (A)"
- board text added: "O2 Sensor (B)"
- board text added: "ONLY TYPE C"
- board text added: "ONLY TYPE W"
- board text added: "PAP"
- board text added: "PWM"
- board text added: "RELAYS"
- board text added: "USB"

Commit message: sacando porquerias
Routing:
- net GND: track 215.7 -> 113.5 mm, vias 78 -> 80
- net +5V: track 45.9 -> 22.7 mm
- net +12V: track 53.1 -> 30.0 mm
- net /Sensores/PC0: track 5.35 -> 0.55 mm
- net Net-(R95-Pad1): track 9.59 -> 6.20 mm
- net Net-(D16-Pad1): track 15.0 -> 11.8 mm
- net Net-(R94-Pad1): track 9.74 -> 6.71 mm
- net Net-(D9-Pad1): track 14.6 -> 11.6 mm
- net Net-(D15-Pad1): track 14.8 -> 11.8 mm
- net Net-(D10-Pad1): track 14.6 -> 11.7 mm
- net /Sensores/PA6: track 45.2 -> 42.3 mm
- net /Sensores/PA2: track 21.9 -> 19.1 mm
- net Net-(D5-Pad1): track 14.6 -> 11.8 mm
- net Net-(D8-Pad1): track 14.6 -> 11.8 mm
- net /Sensores/PA1: track 36.2 -> 33.5 mm
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
Commit message: el ci ameo'
Other:
- board text added: "GIT_REV"
