File: STM32F_rev3/file5F54B133.sch (KiCad schematic (older format))
At the start: 173 parts, among them U10 LM321, U11 LM321, U12 LM321, U13 LM321, U14 LM321, U15 LM321, U16 LM321, U17 LM321, U18 LM321, U19 LM321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

Commit message: fix drc error
Parts:
- gave numbers to parts that had none: 1
Changed lines of the file:
@@
 CONN_17
 $Comp
-L Device:C_Small C?
+L Device:C_Small C51
 U 1 1 5FA0BA56
 P 17300 8650
-F 0 "C?" H 17392 8696 50  0000 L CNN
+F 0 "C51" H 17392 8696 50  0000 L CNN
 F 1 "240pF" H 17392 8605 50  0000 L CNN
 F 2 "Capacitor_SMD:C_0603_1608Metric" H 17300 8650 50  0001 C CNN
