File: STM32F_rev3/STM32F_rev3.sch (KiCad schematic (older format))
At the start: 27 parts, among them J1 USB_B, J2 Tag connect, SW1 SW_Push, U1 MCZ33810EK, U3 STM32F407VGTx, Y1 25MHz

Commit message: update paths
Parts:
- U1: footprint OpenEFI-STM32F rev3:SOP65P1030X245-33N -> OpenEFI-STM32F_rev3:SOP65P1030X245-33N
Changed lines of the file:
@@
 F 0 "U1" H 8300 4220 50  0000 C CNN
 F 1 "MCZ33810EK" H 8300 4129 50  0000 C CNN
-F 2 "OpenEFI-STM32F rev3:SOP65P1030X245-33N" H 8300 2650 50  0001 L BNN
+F 2 "OpenEFI-STM32F_rev3:SOP65P1030X245-33N" H 8300 2650 50  0001 L BNN
 F 3 "-" H 8300 2650 50  0001 L BNN
 F 4 "FREESCALE SEMICONDUCTOR" H 8300 2650 50  0001 L BNN "Field4"

Commit message: WIP V3
Parts:
- J1: symbol Connector:USB_B -> STM32F_rev3-rescue:USB_B-Connector
Changed lines of the file:
@@
 $EndComp
 $Comp
-L Connector:USB_B J1
+L STM32F_rev3-rescue:USB_B-Connector J1
 U 1 1 5F7CD2F4
 P 850 7075
