File: STM32F_rev3/STM32F_rev3.kicad_pcb (KiCad board)
At the start: 4 copper layers, 200.2 x 140.2 mm, 248 parts, among them J1 USB_B, J2 Tag connect, J3 502225-0801, Q1 ISL9V5045S3ST, Q2 ISL9V5045S3ST, Q3 ISL9V5045S3ST, Q4 ISL9V5045S3ST, Q5 2N3904, Q6 IRF540N, Q7 IRF540N, SW1 SW_Push, U1 MCZ33810EK, U10 LM321, U11 LM321, U12 LM321, U13 LM321, U14 LM321, U15 LM321, U16 LM321, U17 LM321, U18 LM321, U19 LM321, U2 LM321, U20 LM321, U21 LM321, U22 LM321, U23 LM321, U24 LM321, U25 LM321, U26 LM321, U27 LM321, U28 LM321, U29 LM321, U3 STM32F407VGTx, U30 LM321, U31 LM321, U32 LM321, U33 LM321, U34 LM321, U35 LM321, U4 MIC2940A-3.3WU, U5 MIC2940A-5.0WT, U6 LT4363IMS, U7 MIC2940A-5.0WT, U8 LM321, U9 LM321, Y1 25MHz

Commit message: update paths
Parts:
- J3: footprint OpenEFI-STM32F rev3:502225-0801 -> OpenEFI-STM32F_rev3:502225-0801
- U1: footprint OpenEFI-STM32F rev3:SOP65P1030X245-33N -> OpenEFI-STM32F_rev3:SOP65P1030X245-33N
Changed lines of the file:
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@@
     )
   )
-  (module "OpenEFI-STM32F rev3:502225-0801" locked (layer F.Cu)
+  (module "OpenEFI-STM32F_rev3:502225-0801" locked (layer F.Cu)
     (at 159.639 66.4845 180)
     (fp_text reference J3 (at -12.192 9.652) (layer F.SilkS)
@@
     (pad 1 thru_hole circle (at 0 0 180) (size 1.8034 1.8034) (drill 1.2954) (layers *.Cu *.Mask)
       (net 101 CONN_1))
-    (model "../library/OpenEFI-STM32F rev3.pretty/models/5022250801.stp"
+    (model "../library/OpenEFI-STM32F_rev3.pretty/models/5022250801.stp"
       (offset (xyz 10.5 -23.5 22.5))
       (scale (xyz 1 1 1))
@@
     )
   )
-  (module "OpenEFI-STM32F rev3:SOP65P1030X245-33N" (layer F.Cu)
+  (module "OpenEFI-STM32F_rev3:SOP65P1030X245-33N" (layer F.Cu)
     (at 197.2691 108.1278)
     (fp_text reference U1 (at -1.9558 4.318) (layer F.SilkS) hide
@@
     (pad 1 smd rect (at -4.699 -4.8768) (size 1.6002 0.4318) (layers F.Cu F.Paste F.Mask)
       (net 101 CONN_1))
-    (model "../library/OpenEFI-STM32F rev3.pretty/models/MCZ33810EK.STEP"
+    (model "../library/OpenEFI-STM32F_rev3.pretty/models/MCZ33810EK.STEP"
       (offset (xyz 0 0 1.2))
       (scale (xyz 1 1 1))

Commit message: WIP V3
Parts:
- removed C17, C37, C38, C39, C40, C41, C42, C43: 240pF, Capacitor_SMD:C_0603_1608Metric
- removed D1, D10, D11, D5, D6, D7, D8, D9: DZ2S033X0L, Diode_SMD:D_MiniMELF
- removed JP1, JP2, JP3, JP4, JP5, JP6, JP7, JP8: Jumper_NC_Small, Jumper:SolderJumper-2_P1.3mm_Open_TrianglePad1.0x1.5mm
- removed R24, R25, R26, R27, R3, R51, R52, R53: 3.32k +-1%, Resistor_SMD:R_0603_1608Metric
- removed R28, R29, R30, R31, R4, R56, R57, R58: 28.6k +-1%, Resistor_SMD:R_0603_1608Metric
- removed R32, R33, R34, R35, R5, R61, R62, R63: 2.2k, Resistor_SMD:R_0603_1608Metric
- removed R36, R39, R42, R45, R48, R66, R69, R72: 16k 1/10W +-1%, Resistor_SMD:R_0603_1608Metric
- removed R37, R40, R43, R46, R49, R67, R70, R73: 1k 1/10W +-1%, Resistor_SMD:R_0603_1608Metric
- removed R38, R41, R44, R47, R50, R68, R71, R74: 33k 1/10W +-1%, Resistor_SMD:R_0603_1608Metric
- removed U15, U16, U17, U18, U19, U22, U23, U24: LM321, Package_TO_SOT_SMD:SOT-23-5
- added C52: 0.01uF, Capacitor_SMD:C_0603_1608Metric, F.Cu at (80.2, 95.0)
- added C53: 0.01uF, Capacitor_SMD:C_0603_1608Metric, F.Cu at (80.2, 91.8)
- added C54: 0.01uF, Capacitor_SMD:C_0603_1608Metric, F.Cu at (80.2, 98.4)
- added C55: 0.01uF, Capacitor_SMD:C_0603_1608Metric, F.Cu at (80.1, 79.4)
- added C56: 0.01uF, Capacitor_SMD:C_0603_1608Metric, F.Cu at (80.1, 76.2)
- added C57: 0.01uF, Capacitor_SMD:C_0603_1608Metric, F.Cu at (80.1, 82.8)
- added JP23: SolderJumper_2_Open, Jumper:SolderJumper-2_P1.3mm_Open_RoundedPad1.0x1.5mm, F.Cu at (77.4, 101.7)
- added JP24: SolderJumper_2_Open, Jumper:SolderJumper-2_P1.3mm_Open_RoundedPad1.0x1.5mm, F.Cu at (77.3, 86.2)
- added R112: 4.99K 1/2W, Resistor_SMD:R_1210_3225Metric, F.Cu at (77.3, 92.6)
- added R113: 4.99K 1/2W, Resistor_SMD:R_1210_3225Metric, F.Cu at (83.0, 97.6)
- added R114: 4.99K 1/2W, Resistor_SMD:R_1210_3225Metric, F.Cu at (77.4, 97.6)
- added R115: 4.99K 1/2W, Resistor_SMD:R_1210_3225Metric, F.Cu at (82.3, 101.7)
- added R116: 4.99K 1/2W, Resistor_SMD:R_1210_3225Metric, F.Cu at (83.0, 77.1)
- added R117: 4.99K 1/2W, Resistor_SMD:R_1210_3225Metric, F.Cu at (77.3, 77.1)
- added R118: 4.99K 1/2W, Resistor_SMD:R_1210_3225Metric, F.Cu at (83.0, 82.0)
- added R119: 4.99K 1/2W, Resistor_SMD:R_1210_3225Metric, F.Cu at (77.3, 82.0)
- added R120: 4.99K 1/2W, Resistor_SMD:R_1210_3225Metric, F.Cu at (82.3, 86.2)
- added R121: R_Small, Resistor_SMD:R_0603_1608Metric, F.Cu at (77.7, 113.6)
- added R122: R_Small, Resistor_SMD:R_0603_1608Metric, F.Cu at (82.1, 113.5)
- added R81: 4.99K 1/2W, Resistor_SMD:R_1210_3225Metric, F.Cu at (83.0, 92.6)
- added U36: MAX9926UAEE+, OpenEFI-STM32F_rev3:SOP63P602X175-16N, F.Cu at (79.9, 109.6)
- C33, D2, D3, Q5, R17, R18, R19, R20, R22, R23: moved to B.Cu
- U10, U11, U12, U2: value LM321 -> SensorsV1; footprint Package_TO_SOT_SMD:SOT-23-5 -> OpenEFI-STM32F_rev3:SensorsV1
- U13, U14, U8, U9: value LM321 -> SensorsV1; footprint Package_TO_SOT_SMD:SOT-23-5 -> OpenEFI-STM32F_rev3:SensorsV1; moved to B.Cu
- moved R82 83.7 mm to (172.7, 106.3)
- moved C51 83.7 mm to (171.5, 109.1)
- moved JP11 83.7 mm to (176.7, 110.8)
- moved U27 83.7 mm to (176.0, 105.9)
- moved D14 83.7 mm to (172.5, 111.3)
- moved R83 83.7 mm to (170.6, 106.4)
- moved C19 70.0 mm to (223.2, 68.2), turned to 180 degrees
- moved R14 69.4 mm to (223.2, 66.5)
- moved C26 66.2 mm to (223.2, 69.8), turned to 180 degrees
- moved R54 65.2 mm to (192.3, 135.8)
- moved R75 65.0 mm to (193.1, 131.1), turned to 0 degrees
- moved R10 64.7 mm to (220.8, 67.3), turned to 90 degrees
- moved R23 64.6 mm to (173.7, 71.6)
- moved U20 64.4 mm to (188.7, 132.2), turned to 0 degrees
- moved C44 63.9 mm to (188.3, 138.3)
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Connections:
- net /Sheet5FA9324A/FB0 renamed /FB0
- net /Sheet5FA9324A/FB1 renamed /FB1
- net /Sheet5FA9324A/FB2 renamed /FB2
- net /Sheet5FA9324A/FB3 renamed /FB3
- net /Sheet5FA9324A/GD0 renamed /GD0
- net /Sheet5FA9324A/GD1 renamed /GD1
- net /Sheet5FA9324A/GD2 renamed /GD2
- net /Sheet5FA9324A/GD3 renamed /GD3
- net Net-(U3-Pad16) renamed /PC1
- C29 pad 2: CONN_2 -> CONN_1
- C30 pad 2: CONN_1 -> CONN_2
- C49 pad 1: CONN_16 -> CONN_17
- C50 pad 1: CONN_17 -> CONN_16
- J3 pad 67: CONN_67 -> GND
- J3 pad 70: CONN_70 -> GND
- J3 pad 71: CONN_71 -> CONN71+
- J3 pad 72: CONN_72 -> CONN72-
- JP10 pad 2: /Sensores/PB1 -> /PB1
- JP11 pad 2: /Sensores/PC5 -> /PC5
- JP12 pad 2: /Sensores/PC4 -> /PC4
- JP13 pad 2: /Sensores/PC3 -> /PC3
- JP14 pad 2: /Sensores/PC2 -> /PC2
- JP19 pad 2: /Sensores/PC0 -> /PC0
- JP22 pad 2: /Sensores/PC0 -> /PC0
- JP9 pad 2: /Sensores/PB0 -> /PB0
- R82 pad 2: CONN_18 -> +12VA
- R87 pad 1: CONN_16 -> CONN_17
- R88 pad 1: CONN_17 -> CONN_16
- R92 pad 1: CONN_16 -> CONN_17
- R93 pad 1: CONN_17 -> CONN_16
- R97 pad 2: CONN_16 -> CONN_17
- R98 pad 2: CONN_17 -> CONN_16
- U1 pad 1: CONN_1 -> CONN_2
- U1 pad 16: CONN_2 -> CONN_1
- U1 pad 17: CONN_22 -> /OUT4
- U10 pad 1: Net-(R34-Pad1) -> +5V
- U10 pad 2: GND -> CONN_6
- U10 pad 3: Net-(R45-Pad1) -> GND
- U10 pad 4: Net-(R45-Pad1) -> GND
- U10 pad 5: +12V -> /PA3
- U11 pad 1: Net-(R35-Pad1) -> +5V
- U11 pad 2: GND -> CONN_7
- U11 pad 3: Net-(R48-Pad1) -> GND
- U11 pad 4: Net-(R48-Pad1) -> GND
- U11 pad 5: +12V -> /PA4
- U12 pad 1: Net-(D1-Pad1) -> +5V
- U12 pad 2: GND -> CONN_8
- U12 pad 3: Net-(JP2-Pad1) -> GND
- U12 pad 4: Net-(JP2-Pad1) -> GND
- U12 pad 5: +5V -> /PA5
- U13 pad 1: Net-(D5-Pad1) -> +5V
- U13 pad 2: GND -> CONN_9
- U13 pad 3: Net-(JP1-Pad1) -> GND
- U13 pad 4: Net-(JP1-Pad1) -> GND
- U13 pad 5: +5V -> /PA6
- U14 pad 1: Net-(D6-Pad1) -> +5V
- U14 pad 2: GND -> CONN_10
- U14 pad 3: Net-(JP3-Pad1) -> GND
- U14 pad 4: Net-(JP3-Pad1) -> GND
- U14 pad 5: +5V -> /PA7
- U2 pad 1: Net-(R5-Pad1) -> +5V
- U2 pad 2: GND -> CONN_3
- U2 pad 3: Net-(R36-Pad1) -> GND
- U2 pad 4: Net-(R36-Pad1) -> GND
- U2 pad 5: +12V -> /PA0
- U3 pad 15: Net-(U3-Pad15) -> /PC0
- U3 pad 17: Net-(U3-Pad17) -> /PC2
- U3 pad 18: Net-(U3-Pad18) -> /PC3
- U3 pad 23: Net-(U3-Pad23) -> /PA0
- U3 pad 24: Net-(U3-Pad24) -> /PA1
- U3 pad 25: Net-(U3-Pad25) -> /PA2
- U3 pad 26: Net-(U3-Pad26) -> /PA3
- U3 pad 29: Net-(U3-Pad29) -> /PA4
- U3 pad 30: Net-(U3-Pad30) -> /PA5
- U3 pad 31: Net-(U3-Pad31) -> /PA6
- U3 pad 32: Net-(U3-Pad32) -> /PA7
- U3 pad 33: Net-(U3-Pad33) -> /PC4
- U3 pad 34: Net-(U3-Pad34) -> /PC5
- U3 pad 35: Net-(U3-Pad35) -> /PB0
- U3 pad 36: Net-(U3-Pad36) -> /PB1
- U7 pad 3: +5V -> +5VA
- U8 pad 1: Net-(R32-Pad1) -> +5V
- U8 pad 2: GND -> CONN_4
- U8 pad 3: Net-(R39-Pad1) -> GND
- U8 pad 4: Net-(R39-Pad1) -> GND
- U8 pad 5: +12V -> /PA1
- U9 pad 1: Net-(R33-Pad1) -> +5V
- U9 pad 2: GND -> CONN_5
- U9 pad 3: Net-(R42-Pad1) -> GND
- U9 pad 4: Net-(R42-Pad1) -> GND
- U9 pad 5: +12V -> /PA2
Routing:
- net Net-(C22-Pad2): track 0.00 -> 122.8 mm, vias 0 -> 3
- net CONN_22: track 5.61 -> 116.8 mm, vias 0 -> 1
- net CONN_1: track 2.07 -> 106.1 mm, vias 0 -> 1
- net CONN_2: track 3.40 -> 98.4 mm, vias 0 -> 1
- net CONN_21: track 5.83 -> 90.8 mm, vias 0 -> 1
- net CONN_18: track 64.3 -> 0.89 mm, vias 1 -> 0
- net CONN_5: track 62.1 -> 0.00 mm, vias 1 -> 0
- net CONN_42: track 35.8 -> 87.5 mm
- net CONN_11: track 49.6 -> 0.00 mm, vias 2 -> 0
- net /Sensores/PA0: track 48.6 -> 0.00 mm, vias 1 -> 0
- net GND: track 113.5 -> 67.8 mm, vias 80 -> 62
- net /Sensores/PA3: track 45.5 -> 0.00 mm, vias 1 -> 0
- net Net-(Q6-Pad1): track 0.00 -> 42.7 mm
- net (no net): track 42.4 -> 0.00 mm
- net /Sensores/PA6: track 42.3 -> 0.00 mm, vias 1 -> 0
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Other:
- net class Default removed
- board text added: "BP"
- board text added: "CKP Sensor"
- board text added: "CKP/CMP"
- board text added: "FB0"
- board text added: "FB1"
- board text added: "FB2"
- board text added: "FB3"
- board text added: "RSP"
- board text added: "Surge Stopper"
- board text added: "in case of poor signal, short "BP""
- board text added: "mil"
- board text removed: "AIN0"
- board text removed: "AIN1"
- board text removed: "AIN2"
- board text removed: "AIN4"
- board text removed: "AIN5"
- board text removed: "AIN6"
- board text removed: "AIN7"
- board text removed: "AIN8"
- board text removed: "AIN9"
- board text removed: "CAN"
- board text removed: "CKP"
- board text removed: "CMP"
- board text removed: "Enable"

Commit message: Update on PMIC
Parts:
- removed C44, C45, C46, C47, C48: 240pF, Capacitor_SMD:C_0603_1608Metric
- removed D15, D16, D17: DZ2S033X0L, Diode_SMD:D_MiniMELF
- removed JP10, JP12, JP13, JP14, JP9: Jumper_NC_Small, Jumper:SolderJumper-2_P1.3mm_Open_TrianglePad1.0x1.5mm
- removed R100, R103, R106, R76, R79: 1k 1/10W +-1%, Resistor_SMD:R_0603_1608Metric
- removed R101, R104, R107, R77, R80: 33k 1/10W +-1%, Resistor_SMD:R_0603_1608Metric
- removed R102, R105, R75, R78, R99: 16k 1/10W +-1%, Resistor_SMD:R_0603_1608Metric
- removed R54, R55, R84, R85, R86: 3.32k +-1%, Resistor_SMD:R_0603_1608Metric
- removed R59, R60, R89, R90, R91: 28.6k +-1%, Resistor_SMD:R_0603_1608Metric
- removed R64, R65, R94, R95, R96: 2.2k, Resistor_SMD:R_0603_1608Metric
- removed U25, U26, U28, U29, U30, U33, U34, U35: LM321, Package_TO_SOT_SMD:SOT-23-5
- removed U7: MIC2940A-5.0WT, Package_TO_SOT_THT:TO-220-3_Vertical
- added D1: LED, LED_SMD:LED_0603_1608Metric, B.Cu at (137.5, 135.3)
- added D10: LED, LED_SMD:LED_0603_1608Metric, B.Cu at (137.5, 129.4)
- added D11: LED, LED_SMD:LED_0603_1608Metric, B.Cu at (146.8, 135.2)
- added D5: LED, LED_SMD:LED_0603_1608Metric, B.Cu at (142.2, 135.3)
- added D6: LED, LED_SMD:LED_0603_1608Metric, B.Cu at (130.7, 135.0)
- added D7: LED, LED_SMD:LED_0603_1608Metric, B.Cu at (132.8, 134.9)
- added D8: LED, LED_SMD:LED_0603_1608Metric, B.Cu at (146.8, 129.4)
- added D9: LED, LED_SMD:LED_0603_1608Metric, B.Cu at (142.1, 129.4)
- added R24: R_Small, Resistor_SMD:R_0603_1608Metric, B.Cu at (132.8, 131.5)
- added R25: R_Small, Resistor_SMD:R_0603_1608Metric, B.Cu at (144.9, 129.4)
- added R26: R_Small, Resistor_SMD:R_0603_1608Metric, B.Cu at (140.2, 129.4)
- added R27: R_Small, Resistor_SMD:R_0603_1608Metric, B.Cu at (135.7, 129.4)
- added R28: R_Small, Resistor_SMD:R_0603_1608Metric, B.Cu at (144.9, 135.2)
- added R29: R_Small, Resistor_SMD:R_0603_1608Metric, F.Cu at (122.3, 135.1)
- added R3: R_Small, Resistor_SMD:R_0603_1608Metric, B.Cu at (135.7, 135.3)
- added R30: R_Small, Resistor_SMD:R_0603_1608Metric, F.Cu at (122.3, 137.7)
- added R4: R_Small, Resistor_SMD:R_0603_1608Metric, B.Cu at (140.2, 135.3)
- added R5: R_Small, Resistor_SMD:R_0603_1608Metric, B.Cu at (130.7, 131.5)
- added U15: SensorsV1, OpenEFI-STM32F_rev3:SensorsV1, B.Cu at (87.3, 107.4)
- added U16: SensorsV1, OpenEFI-STM32F_rev3:SensorsV1, F.Cu at (91.1, 108.8)
- added U17: SensorsV1, OpenEFI-STM32F_rev3:SensorsV1, B.Cu at (57.5, 84.8)
- added U18: SensorsV1, OpenEFI-STM32F_rev3:SensorsV1, F.Cu at (58.9, 103.0)
- added U19: SensorsV1, OpenEFI-STM32F_rev3:SensorsV1, F.Cu at (58.9, 80.2)
- added U22: TPL7407LAPWR, Package_SO:TSSOP-16_4.4x5mm_P0.65mm, B.Cu at (94.6, 50.2)
- C18, C19, C2, C20, C21, C23, C24, C25, C26, C3, C36, C8, C9, R10, R11, R12, R13, R14, R15, R16, R9, SW1, TP1, TP2, U3, U6, Y1: moved to B.Cu
- D12, D13: value DZ2S033X0L -> LED; footprint Diode_SMD:D_MiniMELF -> LED_SMD:LED_0603_1608Metric
- J2: footprint Connector:Tag-Connect_TC2030-IDC-FP_2x03_P1.27mm_Vertical -> Connector:Tag-Connect_TC2030-IDC-NL_2x03_P1.27mm_Vertical; moved to B.Cu
- U20, U21: value LM321 -> TPL7407LAPWR; footprint Package_TO_SOT_SMD:SOT-23-5 -> Package_SO:TSSOP-16_4.4x5mm_P0.65mm; moved to B.Cu
- moved U20 160.0 mm to (51.2, 50.3), turned to -90 degrees
- moved U21 135.7 mm to (40.9, 50.3), turned to -90 degrees
- moved J1 128.5 mm to (159.5, 130.9), turned to 0 degrees
- moved R1 105.2 mm to (155.2, 129.3), turned to -90 degrees
- moved C5 92.5 mm to (123.8, 105.5), turned to -45 degrees
- moved C6 84.3 mm to (122.4, 106.9), turned to -45 degrees
- moved C19 84.0 mm to (140.2, 55.5)
- moved R10 83.7 mm to (137.8, 56.5), turned to -90 degrees
- moved R14 83.5 mm to (140.2, 57.2)
- moved C21 83.1 mm to (140.2, 81.9)
- moved R12 83.1 mm to (137.9, 82.7), turned to -90 degrees
- moved R16 83.1 mm to (140.2, 83.4)
- moved Y1 82.1 mm to (112.1, 102.8), turned to 90 degrees
- moved SW1 81.5 mm to (103.8, 104.2), turned to 90 degrees
- moved C3 81.1 mm to (114.9, 102.0), turned to -90 degrees
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Connections:
- net Net-(U3-Pad68) renamed /VBUS
- C28 pad 2: CONN_21 -> CONN_2
- C30 pad 2: CONN_2 -> CONN_21
- D12 pad 2: GND -> +3V3
- D13 pad 2: GND -> +3V3
- U1 pad 1: CONN_2 -> CONN_21
- U1 pad 17: /OUT4 -> CONN_22
- U1 pad 32: CONN_21 -> CONN_2
- U10 pad 1: +5V -> +12V
- U11 pad 1: +5V -> +12V
- U12 pad 1: +5V -> +12V
- U13 pad 1: +5V -> +12V
- U14 pad 1: +5V -> +12V
- U2 pad 1: +5V -> +12V
- U20 pad 1: Net-(R64-Pad1) -> /PWM0
- U20 pad 2: GND -> /PWM0
- U20 pad 3: Net-(R75-Pad1) -> /PWM0
- U20 pad 4: Net-(R75-Pad1) -> /PWM1
- U20 pad 5: +12V -> /PWM1
- U21 pad 1: Net-(R65-Pad1) -> /PWM2
- U21 pad 2: GND -> /PWM2
- U21 pad 3: Net-(R78-Pad1) -> /PWM2
- U21 pad 4: Net-(R78-Pad1) -> /PWM3
- U21 pad 5: +12V -> /PWM3
- U3 pad 5: /ECN4 -> Net-(U3-Pad5)
- U3 pad 59: /PMIC_ENABLE -> /ECN1
- U3 pad 60: /ECN1 -> /ECN2
- U3 pad 61: /ECN2 -> /ECN3
- U3 pad 62: /ECN3 -> /ECN4
- U4 pad 1: +5V -> +12V
- U8 pad 1: +5V -> +12V
- U9 pad 1: +5V -> +12V
Routing:
- net +12V: track 31.6 -> 223.6 mm, vias 6 -> 5
- net +3V3: track 0.00 -> 99.2 mm, vias 0 -> 14
- net +12VA: track 194.0 -> 255.6 mm, vias 2 -> 3
- net Net-(D4-Pad1): track 50.8 -> 108.9 mm, vias 0 -> 1
- net Net-(Q7-Pad2): track 22.2 -> 75.8 mm, vias 0 -> 2
- net CONN_42: track 87.5 -> 42.4 mm
- net /PMIC_SPARK: track 0.00 -> 44.0 mm, vias 0 -> 3
- net CONN_11: track 0.00 -> 43.3 mm
- net Net-(Q6-Pad1): track 42.7 -> 0.00 mm
- net CONN_9: track 0.00 -> 41.2 mm
- net /ECN4: track 0.00 -> 38.1 mm, vias 0 -> 1
- net /ECN3: track 0.00 -> 38.0 mm, vias 0 -> 1
- net /ECN1: track 0.00 -> 37.8 mm, vias 0 -> 1
- net /ECN2: track 0.00 -> 37.8 mm, vias 0 -> 1
- net CONN_6: track 0.00 -> 37.2 mm
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- added copper zone on B.Cu, net +12V
- added copper zone on In2.Cu, net +5V
- added copper zone on B.Cu, net GND
- removed copper zone on In2.Cu, net +12V
- removed copper zone on B.Cu, net +5V
Other:
- board size 200.2 x 140.2 mm -> 159.6 x 99.6 mm
- board text added: "3v"
- board text added: "4050"
- board text added: "5v"
- board text added: "CAN"
- board text added: "EEPROM"
- board text added: "GNC"
- board text added: "GPIO"
- board text added: "LED0"
- board text added: "LED1"
- board text added: "LED2"
- board text added: "OpenEFI V2.x"
- board text added: "Prototype"
- board text added: "RX"
- board text added: "TX"
- board text added: "VREF"
- board text removed: "AIN10"
- board text removed: "AIN11"
- board text removed: "AIN12"
- board text removed: "AIN3"
- board text removed: "CMP / CKP MODS / TESTING"
- board text removed: "ENABLE"
- board text removed: "PAP"
- board text removed: "PWM"
- board text removed: "RELAYS"
- board text removed: "USB"
- board text removed: "mil"
- board text removed: "pwm?"
