File: STM32F_rev3/STM32F_rev3.kicad_pcb (KiCad board)
At the start: 4 copper layers, 159.6 x 99.6 mm, 335 parts, among them J1 USB_B, J2 Tag connect, J3 502225-0801, Q1 ISL9V5045S3ST, Q2 ISL9V5045S3ST, Q3 ISL9V5045S3ST, Q4 ISL9V5045S3ST, Q5 2N3904, Q6 IRF540N, Q7 IRF540N, Q8 SS8050, Q9 SS8050, SW1 SW_Push, U1 MCZ33810EK, U10 SensorsV1, U11 SensorsV1, U12 SensorsV1, U13 SensorsV1, U14 SensorsV1, U15 SensorsV1, U16 SensorsV1, U17 SensorsV1, U18 SensorsV1, U19 SensorsV1, U2 SensorsV1, U20 TPL7407LAPWR, U21 TPL7407LAPWR, U22 TPL7407LAPWR, U27 LM321, U3 STM32F407VGTx, U31 LM321, U32 LM321, U36 MAX9926UAEE+, U4 MIC2940A-3.3WU, U5 MIC2940A-5.0WT, U6 LT4363IMS, U7 25LCxxx, U8 SensorsV1, U9 SensorsV1, Y1 25MHz

Commit message: WIP: PAP Driver
Parts:
- added C34: 100nF, Capacitor_SMD:C_0805_2012Metric, F.Cu at (156.3, 128.5)
- added C35: 100nF, Capacitor_SMD:C_0805_2012Metric, F.Cu at (148.8, 130.3)
- added C37: 100nF, Capacitor_SMD:C_0805_2012Metric, F.Cu at (132.3, 128.0)
- added JP1: SolderJumper_2_Open, Jumper:SolderJumper-2_P1.3mm_Open_RoundedPad1.0x1.5mm, F.Cu at (44.1, 85.7)
- added JP2: SolderJumper_2_Open, Jumper:SolderJumper-2_P1.3mm_Open_RoundedPad1.0x1.5mm, F.Cu at (46.6, 85.7)
- added JP3: SolderJumper_2_Open, Jumper:SolderJumper-2_P1.3mm_Open_RoundedPad1.0x1.5mm, F.Cu at (41.5, 85.7)
- added R33: R_Small, Resistor_SMD:R_0603_1608Metric, F.Cu at (153.3, 133.3)
- added U23: PaP_Driver_v1, OpenEFI-STM32F_rev3:DIP-16_598_ELL, B.Cu at (40.3, 81.7)
- added U24: ADUM4160, Package_SO:SOIC-16W_7.5x10.3mm_P1.27mm, F.Cu at (141.0, 127.5)
- Q8, Q9, R31, R32, U18: moved to B.Cu
- R1: value 10k -> R_Small; moved to F.Cu
- moved Q9 112.9 mm to (122.4, 136.1)
- moved R32 112.8 mm to (122.2, 138.9), turned to 180 degrees
- moved Q8 101.3 mm to (130.0, 125.0), turned to 180 degrees
- moved R31 96.8 mm to (132.8, 124.7), turned to 90 degrees
- moved LOGO1 30.1 mm to (172.2, 113.5)
- moved E 21.2 mm to (79.4, 123.5)
- moved E 21.2 mm to (109.9, 136.2)
- moved E 21.2 mm to (64.1, 133.6)
- moved E 21.2 mm to (107.3, 123.5)
- moved E 21.2 mm to (56.5, 123.5)
- moved E 21.2 mm to (59.1, 133.6)
- moved E 21.2 mm to (74.3, 133.6)
- moved E 21.2 mm to (89.5, 133.6)
- moved E 21.2 mm to (74.3, 126.0)
- moved E 21.2 mm to (56.5, 133.6)
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Connections:
- net Net-(U3-Pad42) renamed /RPM_OUT
- net Net-(U3-Pad45) renamed /AUX_CS_1
- net Net-(U3-Pad46) renamed /AUX_CS_2
- net Net-(U3-Pad67) renamed no_connect_244
- net Net-(U3-Pad69) renamed /AUX_OUT_4
- net Net-(U3-Pad77) renamed no_connect_245
- net Net-(U3-Pad80) renamed no_connect_246
- net Net-(U3-Pad81) renamed /CAN1_RX
- net Net-(U3-Pad82) renamed /CAN1_TX
- net Net-(U3-Pad83) renamed /AUX_IN_1
- net Net-(U3-Pad84) renamed /AUX_IN_2
- net Net-(U3-Pad85) renamed /AUX_IN_3
- net Net-(U3-Pad86) renamed /AUX_IN_4
- net Net-(U3-Pad87) renamed /LED_CAN_RX
- net Net-(U3-Pad88) renamed /LED_CAN_TX
- net Net-(U3-Pad90) renamed no_connect_247
- net Net-(U3-Pad97) renamed /R_LMB
- net Net-(U3-Pad98) renamed no_connect_248
- net Net-(U36-Pad12) renamed no_connect_249
- net Net-(U36-Pad2) renamed no_connect_250
- net Net-(U36-Pad7) renamed no_connect_251
- net Net-(U6-Pad10) renamed no_connect_252
- net Net-(U6-Pad11) renamed no_connect_253
- net Net-(U6-Pad6) renamed no_connect_254
- net Net-(U6-Pad7) renamed no_connect_255
- net Net-(U6-Pad8) renamed no_connect_256
- J1 pad 1: Net-(J1-Pad1) -> Net-(C34-Pad1)
- J1 pad 2: /USB_D- -> /d-
- J1 pad 3: /USB_D+ -> /d+
- J1 pad 4: GND -> GND1
- J1 pad 5: Net-(J1-Pad5) -> GND1
- R1 pad 1: GND -> /D+
- R1 pad 2: Net-(J1-Pad1) -> /d+
- U20 pad 1: /PWM0 -> /TIM9_CH1
- U20 pad 2: /PWM0 -> /TIM9_CH1
- U20 pad 3: /PWM0 -> /TIM9_CH1
- U20 pad 4: /PWM1 -> /TIM9_CH2
- U20 pad 5: /PWM1 -> /TIM9_CH2
- U20 pad 6: /PWM1 -> /TIM9_CH2
- U3 pad 38: Net-(U3-Pad38) -> /MTR_STEP
- U3 pad 39: Net-(U3-Pad39) -> /MTR_DIR
- U3 pad 40: Net-(U3-Pad40) -> /MTR_FAULT
- U3 pad 41: Net-(U3-Pad41) -> /MTR_ENABLE
- U3 pad 63: Net-(U3-Pad63) -> /CKP
- U3 pad 64: Net-(U3-Pad64) -> /CMP
- U3 pad 65: Net-(U3-Pad65) -> /MIL_OUT
- U3 pad 66: Net-(U3-Pad66) -> /CHK_OUT
- U3 pad 7: Net-(U3-Pad7) -> /LED0
- U3 pad 78: Net-(U3-Pad78) -> /PMIC_NOMI
- U3 pad 79: Net-(U3-Pad79) -> /PMIC_MAXI
- U3 pad 8: Net-(U3-Pad8) -> /LED1
- U3 pad 9: Net-(U3-Pad9) -> /LED2
Routing:
- net +5V: track 1.87 -> 82.2 mm, vias 4 -> 5
- net +3V3: track 123.8 -> 168.1 mm, vias 16 -> 17
- net GND1: track 0.00 -> 40.5 mm, vias 0 -> 1
- net CONN_75: track 0.00 -> 39.1 mm
- net CONN_76: track 0.00 -> 36.0 mm
- net CONN_77: track 0.00 -> 29.6 mm
- net GND: track 93.2 -> 118.0 mm, vias 71 -> 74
- net CONN_78: track 0.00 -> 22.2 mm
- net Net-(C34-Pad1): track 0.00 -> 18.6 mm, vias 0 -> 1
- net CONN_16: track 42.3 -> 59.9 mm
- net CONN_17: track 19.0 -> 36.0 mm
- net /PC5: track 0.00 -> 12.2 mm, vias 0 -> 1
- net /GD2: track 41.4 -> 52.7 mm
- net /D-: track 0.00 -> 11.1 mm
- net /D+: track 0.00 -> 11.1 mm
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- added copper zone on F.Cu, net +3V3
- added copper zone on B.Cu, net GND1
- added copper zone on F.Cu, net GND1
Other:
- board text added: "CMP Sensor"
- board text added: "GNC_IN"
- board text added: "RPM_OUT"
- board text added: "RSP ?"
- board text added: "USB ISOLATOR"
- board text removed: "pap"
- board text removed: "relays"

Commit message: Last commit to rev3
Parts:
- moved TP2 3.63 mm to (131.4, 101.2)
Routing:
- net /R_AAC: track 0.65 -> 221.4 mm, vias 0 -> 2
- net /R_GNC_GLP: track 0.65 -> 221.2 mm, vias 0 -> 2
- net /R_ECN_INY: track 0.65 -> 220.7 mm, vias 0 -> 2
- net /MIL_OUT: track 1.31 -> 219.9 mm, vias 1 -> 3
- net /CHK_OUT: track 1.55 -> 213.0 mm, vias 1 -> 2
- net /R3: track 0.00 -> 196.8 mm
- net /TIM9_CH2: track 1.30 -> 186.4 mm, vias 0 -> 2
- net /TIM9_CH1: track 1.30 -> 184.3 mm, vias 0 -> 2
- net Net-(Q7-Pad1): track 0.00 -> 139.3 mm, vias 0 -> 3
- net Net-(Q6-Pad1): track 0.00 -> 104.4 mm, vias 0 -> 1
- net /PC4: track 0.00 -> 83.4 mm, vias 0 -> 2
- net /GD1: track 0.00 -> 83.2 mm, vias 0 -> 3
- net /FB0: track 5.25 -> 80.8 mm
- net /FB1: track 3.35 -> 75.2 mm, vias 1 -> 3
- net /GD0: track 1.96 -> 72.4 mm, vias 1 -> 2
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