File: STM32F_rev3/_autosave-STM32F_rev3.kicad_pcb (KiCad board)
At the start: 4 copper layers, 159.6 x 99.6 mm, 335 parts, among them J1 USB_B, J2 Tag connect, J3 502225-0801, Q1 ISL9V5045S3ST, Q2 ISL9V5045S3ST, Q3 ISL9V5045S3ST, Q4 ISL9V5045S3ST, Q5 2N3904, Q6 IRF540N, Q7 IRF540N, Q8 SS8050, Q9 SS8050, SW1 SW_Push, U1 MCZ33810EK, U10 SensorsV1, U11 SensorsV1, U12 SensorsV1, U13 SensorsV1, U14 SensorsV1, U15 SensorsV1, U16 SensorsV1, U17 SensorsV1, U18 SensorsV1, U19 SensorsV1, U2 SensorsV1, U20 TPL7407LAPWR, U21 TPL7407LAPWR, U22 TPL7407LAPWR, U27 LM321, U3 STM32F407VGTx, U31 LM321, U32 LM321, U36 MAX9926UAEE+, U4 MIC2940A-3.3WU, U5 MIC2940A-5.0WT, U6 LT4363IMS, U7 25LCxxx, U8 SensorsV1, U9 SensorsV1, Y1 25MHz

Commit message: GPIO
Parts:
- Q8, Q9, R31, R32: moved to B.Cu
- moved Q9 112.9 mm to (122.4, 136.1)
- moved R32 112.8 mm to (122.2, 138.9), turned to 180 degrees
- moved Q8 101.3 mm to (130.0, 125.0), turned to 180 degrees
- moved R31 96.8 mm to (132.8, 124.7), turned to 90 degrees
Routing:
- net +5V: track 1.87 -> 38.3 mm, vias 4 -> 5
- net /MIL: track 0.00 -> 8.92 mm
- net /CHK: track 0.00 -> 3.61 mm
- net Net-(Q8-Pad1): track 0.00 -> 2.01 mm
- net Net-(Q9-Pad1): track 0.00 -> 1.88 mm
- net GND: vias 71 -> 73
