File: STM32F_rev3/STM32F_rev3.kicad_sch (KiCad schematic)
At the start: 27 parts, among them J1 USB_B, J2 Tag connect, SW1 SW_Push, U1 MCZ33810EK, U3 STM32F407VGTx, Y1 25MHz

Commit message: Update on PMIC
Parts:
- added D1, D10, D11, D12, D13, D5, D6, D7, D8, D9: LED, LED_SMD:LED_0603_1608Metric, symbol Device:LED
- added R24, R25, R26, R27, R28, R29, R3, R30, R4, R5: R_Small, Resistor_SMD:R_0603_1608Metric, symbol Device:R_Small
- J2: footprint Connector:Tag-Connect_TC2030-IDC-FP_2x03_P1.27mm_Vertical -> Connector:Tag-Connect_TC2030-IDC-NL_2x03_P1.27mm_Vertical
Connections:
- net +3V3: now also D1.2 (A), D10.2 (A), D11.2 (A), D12.2 (A), D13.2 (A), D6.2 (A), D7.2 (A), D8.2 (A), D9.2 (A)
- net ECN1: now also U3.59 (PD12); no longer U3.60 (PD13)
- net ECN2: now also U3.60 (PD13); no longer U3.61 (PD14)
- net ECN3: now also U3.61 (PD14); no longer U3.62 (PD15)
- net ECN4: now also U3.62 (PD15); no longer U3.5 (PE6)
- net GND: now also R3.2, R4.2
- net PMIC_ENABLE: no longer U3.59 (PD12)
- net VBUS: now reaches U3.68 (PA9)
- net OUT4 renamed OUT3
- new net: D6.1 (K), R5.1
- new net: D12.1 (K), R29.1
- new net: D7.1 (K), R24.1
- new net: D13.1 (K), R30.1
- new net: D8.1 (K), R25.1
- new net: D9.1 (K), R26.1
- new net: D5.1 (K), R4.1
- new net: D10.1 (K), R27.1
- new net: D1.1 (K), R3.1
- new net: D11.1 (K), R28.1
- new net +5V: D5.2 (A)
- new net CAN_RX: R24.2
- new net CAN_TX: R5.2
- new net CHK: R30.2
- new net GNC: R28.2
- new net LED0: R25.2
- new net LED1: R26.2
- new net LED2: R27.2
- new net MIL: R29.2
Other:
- added sheet PWM/Relays (pwm_relays.kicad_sch)
- moved on the sheet: H1

Commit message: GPIO
Parts:
- added C17: 100nF, Capacitor_SMD:C_0805_2012Metric, symbol Device:C_Small
- added Q? (x2): SS8050, Package_TO_SOT_SMD:SOT-23, symbol Transistor_BJT:2N3055
- added R? (x2): 1k, Resistor_SMD:R_0603_1608Metric, symbol Device:R
- added U7: 25LCxxx, Package_SO:SOIC-8_3.9x4.9mm_P1.27mm, symbol Memory_EEPROM:25LCxxx
Connections:
- net GNC is gone; now on net GNC_GLP: R28.2
- net +3V3: now also C17.1, U7.8 (VCC)
- net CHK: now also Q?.3 (C)
- net GND: now also C17.2, Q?.2 (E), Q?.2 (E), U7.4 (GND)
- net MIL: now also Q?.3 (C)
- net SPI2_MISO: now also U7.2 (MISO)
- net SPI2_MOSI: now also U7.5 (MOSI)
- net SPI2_SCK: now also U7.6 (SCK)
- net R_ECN_INY: now reaches U3.1 (PE2)
- net R_GNC_GLP: now reaches U3.2 (PE3)
- net R_AAC: now reaches U3.3 (PE4)
- net TIM9_CH1: now reaches U3.4 (PE5)
- net MEMORY_CS: now reaches U3.44 (PE13)
- net MEMORY_CS: now also U7.1 (~CS)
- net TIM9_CH2: now reaches U3.5 (PE6)
- new net: Q?.1 (B), R?.2 (x2)
- new net CHK_OUT: R?.1
- new net MIL_OUT: R?.1
Other:
- note added: "CAN"
- note added: "LED_Aux"
- note added: "NEXT RELEASE"
- note added: "VDD"
- moved on the sheet: C7, C8, C9, D1, D10, D11, D12, D13, D5, D6, D7, D8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

Commit message: WIP: PAP Driver
Parts:
- added C34, C35, C37: 100nF, Capacitor_SMD:C_0805_2012Metric, symbol Device:C_Small
- added JP1, JP2, JP3: SolderJumper_2_Open, Jumper:SolderJumper-2_P1.3mm_Open_RoundedPad1.0x1.5mm, symbol Jumper:SolderJumper_2_Open
- added R33: R_Small, Resistor_SMD:R_0603_1608Metric, symbol Device:R_Small
- added U23: PaP_Driver_v1, OpenEFI-STM32F_rev3:DIP-16_598_ELL, symbol OpenEFI-STM32-rev3:PaP_Driver_v1
- added U24: ADUM4160, Package_SO:SOIC-16W_7.5x10.3mm_P1.27mm, symbol Interface_USB:ADUM4160
- R1: value 10k -> R_Small; LCSC C25804 -> (none)
- gave numbers to parts that had none: 4
Connections:
- net +12V: now also U23.16 (VMOT)
- net +3V3: now also C37.1, JP1.1 (A), JP2.1 (A), JP3.1 (A), U23.5 (RESET), U23.6 (SLEEP), U24.12 (PIN), U24.13 (SPD), U24.14 (VDD2), U24.16 (VBUS2)
- net CHK_OUT: now also U3.66 (PC9)
- net GND: now also C37.2, U23.15 (GND), U23.9 (GND), U24.15 (GND2), U24.9 (GND2); no longer J1.4 (GND), R1.1
- net LED0: now also U3.7 (PC13)
- net LED1: now also U3.8 (PC14)
- net LED2: now also U3.9 (PC15)
- net MIL_OUT: now also U3.65 (PC8)
- net PMIC_MAXI: now also U3.79 (PC11)
- net PMIC_NOMI: now also U3.78 (PC10)
- net USB_D+: now also U24.10 (DD+); no longer J1.3 (D+)
- net USB_D-: now also U24.11 (DD-); no longer J1.2 (D-)
- net MTR_STEP: now reaches U3.38 (PE7)
- net MTR_STEP: now also U23.7 (STEP)
- net MTR_DIR: now reaches U3.39 (PE8)
- net MTR_DIR: now also U23.8 (DIR)
- net MTR_FAULT: now reaches U3.40 (PE9)
- net MTR_FAULT: now also U23.10 (FAULT)
- net MTR_ENABLE: now reaches U3.41 (PE10)
- net MTR_ENABLE: now also U23.1 (ENABLE)
- net RPM_OUT: now reaches U3.42 (PE11)
- net AUX_CS_1: now reaches U3.45 (PE14)
- net AUX_CS_2: now reaches U3.46 (PE15)
- net CKP: now reaches U3.63 (PC6)
- net CMP: now reaches U3.64 (PC7)
- net AUX_OUT_4: now reaches U3.69 (PA10)
- net CAN1_RX: now reaches U3.81 (PD0)
- net CAN1_TX: now reaches U3.82 (PD1)
- net AUX_IN_1: now reaches U3.83 (PD2)
- net AUX_IN_2: now reaches U3.84 (PD3)
- net AUX_IN_3: now reaches U3.85 (PD4)
- net AUX_IN_4: now reaches U3.86 (PD5)
- net LED_CAN_RX: now reaches U3.87 (PD6)
- net LED_CAN_TX: now reaches U3.88 (PD7)
- net R_LMB: now reaches U3.97 (PE0)
- net at J1.1 (VBUS): now also C34.1, U24.1 (VBUS1); no longer R1.2
- net GND1: now reaches J1.5 (Shield)
- net GND1: now also J1.4 (GND), C34.2, C35.2, U24.2 (GND1), U24.8 (GND1)
- new net: JP1.2 (B), U23.3 (M1)
- new net: JP2.2 (B), U23.2 (M0)
- new net: JP3.2 (B), U23.4 (M2)
- new net: C35.1, U24.3 (VDD1), U24.4 (PDEN), U24.5 (SPU)
- new net CONN_75: U23.11 (A2)
- new net CONN_76: U23.12 (A1)
- new net CONN_77: U23.13 (B1)
- new net CONN_78: U23.14 (B2)
- new net D+: R1.1, U24.7 (UD+)
- new net D-: R33.1, U24.6 (UD-)
- new net d+: J1.3 (D+), R1.2
- new net d-: J1.2 (D-), R33.2
- no-connect marks 1 -> 5
Other:
- note added: "DEBUG PIN"
- note added: "PAP MOTOR DRIVER"
- moved on the sheet: C7, C8, C9, J1, R2, SW1, TP1, TP2, U3
