File: STM32F_rev3/file5F54B133.kicad_sch (KiCad schematic)
At the start: 93 parts, among them U10 SensorsV1, U11 SensorsV1, U12 SensorsV1, U13 SensorsV1, U14 SensorsV1, U2 SensorsV1, U20 LM321, U21 LM321, U25 LM321, U26 LM321, U27 LM321, U28 LM321, U29 LM321, U30 LM321, U31 LM321, U32 LM321, U33 LM321, U34 LM321, U35 LM321, U8 SensorsV1, U9 SensorsV1

Commit message: Update on PMIC
Parts:
- removed C44, C45, C46, C47, C48: 240pF, Capacitor_SMD:C_0603_1608Metric, symbol Device:C_Small
- removed D12, D13, D15, D16, D17: DZ2S033X0L, Diode_SMD:D_MiniMELF, symbol Diode:DZ2S033X0L
- removed JP10, JP12, JP13, JP14, JP9: Jumper_NC_Small, Jumper:SolderJumper-2_P1.3mm_Open_TrianglePad1.0x1.5mm, symbol Device:Jumper_NC_Small
- removed R100, R103, R106, R76, R79: 1k 1/10W +-1%, Resistor_SMD:R_0603_1608Metric, symbol Device:R_Small
- removed R101, R104, R107, R77, R80: 33k 1/10W +-1%, Resistor_SMD:R_0603_1608Metric, symbol Device:R_Small
- removed R102, R105, R75, R78, R99: 16k 1/10W +-1%, Resistor_SMD:R_0603_1608Metric, symbol Device:R_Small
- removed R54, R55, R84, R85, R86: 3.32k +-1%, Resistor_SMD:R_0603_1608Metric, symbol Device:R_Small
- removed R59, R60, R89, R90, R91: 28.6k +-1%, Resistor_SMD:R_0603_1608Metric, symbol Device:R_Small
- removed R64, R65, R94, R95, R96: 2.2k, Resistor_SMD:R_0603_1608Metric, symbol Device:R_Small
- removed U20, U21, U25, U26, U28, U29, U30, U33, U34, U35: LM321, Package_TO_SOT_SMD:SOT-23-5, symbol Amplifier_Operational:LM321
- added U15, U16, U17, U18, U19: SensorsV1, OpenEFI-STM32F_rev3:SensorsV1, symbol OpenEFI-STM32-rev3:SensorsV1
Connections:
- net +12V: now also U10.1 (12v), U11.1 (12v), U12.1 (12v), U13.1 (12v), U14.1 (12v), U2.1 (12v), U8.1 (12v), U9.1 (12v), U15.1 (12v), U16.1 (12v), U17.1 (12v), U18.1 (12v), U19.1 (12v); no longer U10.~ (5V), U11.~ (5V), U12.~ (5V), U13.~ (5V), U14.~ (5V), U2.~ (5V), U8.~ (5V), U9.~ (5V)
- net +5V: now also U10.~ (5V), U11.~ (5V), U12.~ (5V), U13.~ (5V), U14.~ (5V), U2.~ (5V), U8.~ (5V), U9.~ (5V), U15.~ (5V), U16.~ (5V), U17.~ (5V), U18.~ (5V), U19.~ (5V); no longer U10.1 (12v), U11.1 (12v), U12.1 (12v), U13.1 (12v), U14.1 (12v), U2.1 (12v), U8.1 (12v), U9.1 (12v)
- net CONN_11: now also U15.2 (AIN)
- net CONN_12: now also U16.2 (AIN)
- net CONN_13: now also U17.2 (AIN)
- net CONN_14: now also U18.2 (AIN)
- net CONN_15: now also U19.2 (AIN)
- net PB0: now also U15.5 (AOUT)
- net PB1: now also U16.5 (AOUT)
- net PC2: now also U17.5 (AOUT)
- net PC3: now also U18.5 (AOUT)
- net PC4: now also U19.5 (AOUT)
- new net: U15.3 (GND), U16.3 (GND), U17.3 (GND), U18.3 (GND), U19.3 (GND)
- new net: U15.4 (GND), U16.4 (GND), U17.4 (GND), U18.4 (GND), U19.4 (GND)
Other:
- moved on the sheet: C49, C50, C51, D14, D18, D19, JP11, JP15, JP16, JP17, JP18, JP19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
