File: STM32F_rev3/pwm_relays.kicad_sch (KiCad schematic)
At the start: 3 parts, among them U20 TPL7407LAPWR, U21 TPL7407LAPWR, U22 TPL7407LAPWR

Commit message: GPIO
Connections:
- net CHK: now also U21.7 (IN7)
- net MIL: now also U20.7 (IN7)
Other:
- note added: "NEXT RELEASE"
Changed lines of the file:
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@@
+    (stroke (width 0) (type dash) (color 0 0 0 0))
+  )
+  (polyline (pts (xy 191.77 73.66) (xy 226.06 73.66))
+    (stroke (width 0) (type dash) (color 0 0 0 0))
+  )
+  (polyline (pts (xy 191.77 83.82) (xy 226.06 83.82))
     (stroke (width 0) (type dash) (color 0 0 0 0))
   )
@@
     (stroke (width 0) (type dash) (color 0 0 0 0))
   )
-  (polyline (pts (xy 228.6 36.83) (xy 228.6 88.9))
+  (polyline (pts (xy 228.6 36.83) (xy 228.6 83.82))
     (stroke (width 0) (type dash) (color 0 0 0 0))
   )
@@
     (stroke (width 0) (type dash) (color 0 0 0 0))
   )
-  (polyline (pts (xy 262.89 36.83) (xy 262.89 88.9))
+  (polyline (pts (xy 228.6 74.93) (xy 262.89 74.93))
     (stroke (width 0) (type dash) (color 0 0 0 0))
   )
-  (polyline (pts (xy 262.89 88.9) (xy 228.6 88.9))
+  (polyline (pts (xy 262.89 36.83) (xy 262.89 83.82))
+    (stroke (width 0) (type dash) (color 0 0 0 0))
+  )
+  (polyline (pts (xy 262.89 83.82) (xy 228.6 83.82))
     (stroke (width 0) (type dash) (color 0 0 0 0))
   )
   (text "CONNECTOR BIND" (at 220.98 41.91 180)
     (effects (font (size 2 2)) (justify right bottom))
+  )
+  (text "NEXT RELEASE" (at 234.95 80.01 180)
+    (effects (font (size 1.27 1.27)) (justify right bottom))
   )
   (text "SCH BIND" (at 252.095 41.275 180)
@@
   (label "PWM0" (at 60.96 63.5 180)
     (effects (font (size 1.27 1.27)) (justify right bottom))
+  )
+  (label "MIL" (at 60.96 78.74 0)
+    (effects (font (size 1.27 1.27)) (justify left bottom))
   )
   (label "PWM1" (at 62.23 71.12 180)
@@
     (effects (font (size 0.8 0.8)) (justify left bottom))
   )
+  (label "CHK" (at 118.11 76.2 0)
+    (effects (font (size 1.27 1.27)) (justify left bottom))
+  )
   (label "PWM2" (at 119.38 60.96 180)
