File: STM32F_rev3/untitled.kicad_sch (KiCad schematic)
At the start: 21 parts, among them U36 MAX9926UAEE+

Commit message: GPIO
Connections:
- net CONN72- renamed CONN71-
Changed lines of the file:
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@@
   (junction (at 180.34 82.55) (diameter 1.016) (color 0 0 0 0))
   (junction (at 191.77 85.09) (diameter 1.016) (color 0 0 0 0))
+  (no_connect (at 135.89 90.17))
+  (no_connect (at 171.45 87.63))
   (no_connect (at 135.89 87.63))
-  (no_connect (at 171.45 87.63))
-  (no_connect (at 135.89 90.17))
   (wire (pts (xy 74.168 104.394) (xy 79.375 104.394))
     (stroke (width 0) (type solid) (color 0 0 0 0))
@@
     (effects (font (size 1.27 1.27)) (justify right bottom))
   )
-  (global_label "CONN72-" (shape input) (at 74.168 104.394 180)
+  (global_label "CONN71-" (shape input) (at 74.168 104.394 180)
     (effects (font (size 1.27 1.27)) (justify right))
   )
