File: µEFI_rev2/connector.kicad_sch (KiCad schematic)
At the start: 23 parts, among them J3 36638-0002, Q5 2N3904, Q6 IRF540N, Q7 IRF540N, U4 MIC2940A-3.3WU, U5 MIC2940A-5.0WT, U6 LT4363IMS

Commit message: uEFI v2 beta release
Parts:
- removed Q5: 2N3904, Package_TO_SOT_SMD:TSOT-23, symbol Transistor_BJT:2N3904
- added Q10: IRF540N, Package_TO_SOT_THT:TO-220-3_Vertical, symbol Transistor_FET:IRF540N
- added Q5: SS8050, Package_TO_SOT_SMD:SOT-23, symbol Transistor_BJT:2N3055
- added R33: 10R 1/10W, Resistor_SMD:R_0603_1608Metric, symbol Device:R_Small
- D2, D3: footprint Diode_SMD:D_0805_2012Metric -> Diode_SMD:D_SOD-523; LCSC (none) -> C511874
- J3: footprint OpenEFI-STM32F_rev3:366380002 -> 366380002
Connections:
- net +12VA: now also J3.A4, Q5.2 (E)
- net +5V: now also Q10.3 (S)
- net at D2.1 (K), R17.1: now also Q5.1 (B)
- net at R18.2, R19.2: now also Q5.3 (C)
- net A1: now reaches J3.A1
- net A2: now reaches J3.A2
- net A3: now reaches J3.A3
- net B1: now reaches J3.B1
- net B2: now reaches J3.B2
- net B3: now reaches J3.B3
- net B4: now reaches J3.B4
- net C1: now reaches J3.C1
- net C2: now reaches J3.C2
- net C3: now reaches J3.C3
- net C4: now reaches J3.C4
- net D1: now reaches J3.D1
- net D2: now reaches J3.D2
- net D3: now reaches J3.D3
- net D4: now reaches J3.D4
- net E1: now reaches J3.E1
- net E2: now reaches J3.E2
- net E3: now reaches J3.E3
- net E4: now reaches J3.E4
- net F1: now reaches J3.F1
- net F2: now reaches J3.F2
- net F3: now reaches J3.F3
- net F4: now reaches J3.F4
- net G1: now reaches J3.G1
- net G2: now reaches J3.G2
- net G3: now reaches J3.G3
- net G4: now reaches J3.G4
- net H1: now reaches J3.H1
- net H2: now reaches J3.H2
- net H3: now reaches J3.H3
- net H4: now reaches J3.H4
- net J1: now reaches J3.J1
- net CAN+: now reaches J3.J2
- net CMP-: now reaches J3.J3
- net CKP-: now reaches J3.J4
- net K1: now reaches J3.K1
- net CAN-: now reaches J3.K2
- net CMP+: now reaches J3.K3
- net CKP+: now reaches J3.K4
- net L1: now reaches J3.L1
- net L2: now reaches J3.L2
- net L3: now reaches J3.L3
- net L4: now reaches J3.L4
- net M1: now reaches J3.M1
- net M2: now reaches J3.M2
- net M3: now reaches J3.M3
- net M4: now reaches J3.M4
- new net: Q10.1 (G), R33.2
- new net +5VA: Q10.2 (D)
- new net 5V_ENABLE: R33.1
