File: µEFI_rev2/file5F54B133.kicad_sch (KiCad schematic)
At the start: 26 parts, among them U10 SensorsV2, U11 SensorsV2, U12 SensorsV2, U13 SensorsV2, U14 SensorsV2, U2 SensorsV2, U27 LM321, U31 LM321, U8 SensorsV2, U9 SensorsV2

Commit message: uEFI v2 beta release
Connections:
- net +12V: now also U10.2 (12v), U11.2 (12v), U12.2 (12v), U13.2 (12v), U14.2 (12v), U2.2 (12v), U8.2 (12v), U9.2 (12v)
- net GND: now also U10.5 (GND), U11.5 (GND), U12.5 (GND), U13.5 (GND), U14.5 (GND), U2.5 (GND), U8.5 (GND), U9.5 (GND)
- net PA0: now also U2.4 (AOUT)
- net PA1: now also U8.4 (AOUT)
- net PA2: now also U9.4 (AOUT)
- net PA3: now also U10.4 (AOUT)
- net PA4: now also U11.4 (AOUT)
- net PA5: now also U12.4 (AOUT)
- net PA6: now also U13.4 (AOUT)
- net PA7: now also U14.4 (AOUT)
- net +5VA: now reaches U8.1 (5V)
- net +5VA: now also U10.1 (5V), U11.1 (5V), U12.1 (5V), U13.1 (5V), U14.1 (5V), U2.1 (5V), U9.1 (5V)
- net E1: now reaches U8.3 (AIN)
- net G1: now reaches U14.3 (AIN)
- net D1: now reaches U11.3 (AIN)
- net J1: now reaches U10.3 (AIN)
- net C1: now reaches U13.3 (AIN)
- net K1: now reaches U2.3 (AIN)
- net H1: now reaches U9.3 (AIN)
- net F1: now reaches U12.3 (AIN)
- net CONN_17 renamed B1
Other:
- moved on the sheet: C49, C51, D14, D18, JP11, JP15, JP17, JP18, JP19, R108, R109, R82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

Commit message: bump to kicad 6, init uEFI v3
Other:
- company: (none) -> Churrosoft
- title: (none) -> uEFI

Commit message: move old boards to __old
Other:
- company: Churrosoft -> (none)
- title: uEFI -> (none)
