File: µEFI_rev2/untitled.kicad_sch (KiCad schematic)
At the start: 21 parts, among them U36 MAX9926UAEE+

Commit message: uEFI v2 beta release
Parts:
- added TP3, TP4, TP5, TP6, TP7, TP8: TestPoint, TestPoint:TestPoint_Pad_1.0x1.0mm, symbol Connector:TestPoint
Connections:
- net CKP: now also TP8.1
- net CMP: now also TP7.1
- net IN1+: now also TP4.1
- net IN1-: now also TP5.1
- net IN2+: now also TP6.1
- net IN2-: now also TP3.1
- net CONN71+ renamed CKP+
- net CONN71- renamed CKP-
- net CONN_68 renamed CMP-
- net CONN_69 renamed CMP+
Changed lines of the file:
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@@
   (junction (at 116.205 58.42) (diameter 1.016) (color 0 0 0 0))
   (junction (at 116.205 78.74) (diameter 1.016) (color 0 0 0 0))
+  (junction (at 124.46 125.095) (diameter 0.9144) (color 0 0 0 0))
   (junction (at 132.08 85.09) (diameter 1.016) (color 0 0 0 0))
   (junction (at 132.08 102.87) (diameter 1.016) (color 0 0 0 0))
@@
   (junction (at 180.34 82.55) (diameter 1.016) (color 0 0 0 0))
   (junction (at 191.77 85.09) (diameter 1.016) (color 0 0 0 0))
+  (junction (at 197.485 85.09) (diameter 0.9144) (color 0 0 0 0))
+  (junction (at 198.12 82.55) (diameter 0.9144) (color 0 0 0 0))
   (no_connect (at 135.89 87.63))
   (no_connect (at 135.89 90.17))
@@
     (stroke (width 0) (type solid) (color 0 0 0 0))
   )
-  (wire (pts (xy 180.34 82.55) (xy 200.66 82.55))
+  (wire (pts (xy 180.34 82.55) (xy 198.12 82.55))
     (stroke (width 0) (type solid) (color 0 0 0 0))
   )
@@
     (stroke (width 0) (type solid) (color 0 0 0 0))
   )
-  (wire (pts (xy 191.77 85.09) (xy 200.66 85.09))
+  (wire (pts (xy 191.77 85.09) (xy 197.485 85.09))
+    (stroke (width 0) (type solid) (color 0 0 0 0))
+  )
+  (wire (pts (xy 197.485 85.09) (xy 200.66 85.09))
+    (stroke (width 0) (type solid) (color 0 0 0 0))
+  )
+  (wire (pts (xy 198.12 82.55) (xy 200.66 82.55))
     (stroke (width 0) (type solid) (color 0 0 0 0))
   )
@@
     (effects (font (size 1.27 1.27)) (justify right bottom))
   )
-  (global_label "CONN71-" (shape input) (at 74.168 104.394 180)
+  (global_label "CKP-" (shape input) (at 74.168 104.394 180)
     (effects (font (size 1.27 1.27)) (justify right))
-    (property "Intersheet References" "${INTERSHEET_REFS}" (id 0) (at 0 0 0)
-      (effects (font (size 1.27 1.27)) hide)
-    )
-  )
-  (global_label "CONN71+" (shape input) (at 74.422 125.222 180)
+    (property "Intersheet References" "${INTERSHEET_REFS}" (id 0) (at 66.3725 104.3146 0)
+      (effects (font (size 1.27 1.27)) (justify right) hide)
+    )
+  )
+  (global_label "CKP+" (shape input) (at 74.422 125.222 180)
     (effects (font (size 1.27 1.27)) (justify right))
-    (property "Intersheet References" "${INTERSHEET_REFS}" (id 0) (at 0 0 0)
-      (effects (font (size 1.27 1.27)) hide)
-    )
-  )
-  (global_label "CONN_68" (shape input) (at 80.01 78.74 180)
+    (property "Intersheet References" "${INTERSHEET_REFS}" (id 0) (at 66.6265 125.1426 0)
+      (effects (font (size 1.27 1.27)) (justify right) hide)
+    )
+  )
+  (global_label "CMP-" (shape input) (at 80.01 78.74 180)
     (effects (font (size 1.27 1.27)) (justify right))
-    (property "Intersheet References" "${INTERSHEET_REFS}" (id 0) (at 0 0 0)
-      (effects (font (size 1.27 1.27)) hide)
-    )
-  )
-  (global_label "CONN_69" (shape input) (at 80.772 58.42 180)
+    (property "Intersheet References" "${INTERSHEET_REFS}" (id 0) (at 72.0331 78.6606 0)
+      (effects (font (size 1.27 1.27)) (justify right) hide)
+    )
+  )
+  (global_label "CMP+" (shape input) (at 80.772 58.42 180)
     (effects (font (size 1.27 1.27)) (justify right))
-    (property "Intersheet References" "${INTERSHEET_REFS}" (id 0) (at 0 0 0)
-      (effects (font (size 1.27 1.27)) hide)
+    (property "Intersheet References" "${INTERSHEET_REFS}" (id 0) (at 72.7951 58.3406 0)
+      (effects (font (size 1.27 1.27)) (justify right) hide)
     )
   )
@@
       (effects (font (size 1.27 1.27)) hide)
     )
+    (pin "1")
+  )
+  (symbol (lib_id "Connector:TestPoint") (at 114.935 104.775 0) (unit 1)
+    (in_bom yes) (on_board yes)
+    (property "Reference" "TP3" (id 0) (at 116.84 102.2984 0)
+      (effects (font (size 1.27 1.27)) (justify left))
+    )
+    (property "Value" "TestPoint" (id 1) (at 116.84 104.8384 0)
+      (effects (font (size 1.27 1.27)) (justify left))
+    )
+    (property "Footprint" "TestPoint:TestPoint_Pad_1.0x1.0mm" (id 2) (at 120.015 104.775 0)
+      (effects (font (size 1.27 1.27)) hide)
+    )
+    (property "Datasheet" "~" (id 3) (at 120.015 104.775 0)
+      (effects (font (size 1.27 1.27)) hide)
+    )
+    (pin "1")
+  )
+  (symbol (lib_id "Connector:TestPoint") (at 116.205 58.42 0) (unit 1)
+    (in_bom yes) (on_board yes)
+    (property "Reference" "TP4" (id 0) (at 118.11 55.9434 0)
+      (effects (font (size 1.27 1.27)) (justify left))
+    )
+    (property "Value" "TestPoint" (id 1) (at 118.11 58.4834 0)
+      (effects (font (size 1.27 1.27)) (justify left))
+    )
+    (property "Footprint" "TestPoint:TestPoint_Pad_1.0x1.0mm" (id 2) (at 121.285 58.42 0)
+      (effects (font (size 1.27 1.27)) hide)
+    )
+    (property "Datasheet" "~" (id 3) (at 121.285 58.42 0)
+      (effects (font (size 1.27 1.27)) hide)
+    )
+    (pin "1")
+  )
+  (symbol (lib_id "Connector:TestPoint") (at 116.205 78.74 180) (unit 1)
+    (in_bom yes) (on_board yes)
+    (property "Reference" "TP5" (id 0) (at 114.3 81.2166 0)
+      (effects (font (size 1.27 1.27)) (justify left))
+    )
+    (property "Value" "TestPoint" (id 1) (at 114.3 78.6766 0)
+      (effects (font (size 1.27 1.27)) (justify left))
+    )
+    (property "Footprint" "TestPoint:TestPoint_Pad_1.0x1.0mm" (id 2) (at 111.125 78.74 0)
+      (effects (font (size 1.27 1.27)) hide)
+    )
+    (property "Datasheet" "~" (id 3) (at 111.125 78.74 0)
+      (effects (font (size 1.27 1.27)) hide)
+    )
+    (pin "1")
+  )
+  (symbol (lib_id "Connector:TestPoint") (at 124.46 125.095 180) (unit 1)
+    (in_bom yes) (on_board yes)
+    (property "Reference" "TP6" (id 0) (at 122.555 127.5716 0)
+      (effects (font (size 1.27 1.27)) (justify left))
+    )
+    (property "Value" "TestPoint" (id 1) (at 122.555 125.0316 0)
+      (effects (font (size 1.27 1.27)) (justify left))
+    )
+    (property "Footprint" "TestPoint:TestPoint_Pad_1.0x1.0mm" (id 2) (at 119.38 125.095 0)
+      (effects (font (size 1.27 1.27)) hide)
+    )
+    (property "Datasheet" "~" (id 3) (at 119.38 125.095 0)
+      (effects (font (size 1.27 1.27)) hide)
+    )
+    (pin "1")
+  )
+  (symbol (lib_id "Connector:TestPoint") (at 197.485 85.09 180) (unit 1)
+    (in_bom yes) (on_board yes)
+    (property "Reference" "TP7" (id 0) (at 195.58 87.5666 0)
+      (effects (font (size 1.27 1.27)) (justify left))
+    )
+    (property "Value" "TestPoint" (id 1) (at 195.58 85.0266 0)
+      (effects (font (size 1.27 1.27)) (justify left))
+    )
+    (property "Footprint" "TestPoint:TestPoint_Pad_1.0x1.0mm" (id 2) (at 192.405 85.09 0)
+      (effects (font (size 1.27 1.27)) hide)
+    )
+    (property "Datasheet" "~" (id 3) (at 192.405 85.09 0)
+      (effects (font (size 1.27 1.27)) hide)
+    )
+    (pin "1")
+  )
+  (symbol (lib_id "Connector:TestPoint") (at 198.12 82.55 0) (unit 1)
+    (in_bom yes) (on_board yes)
+    (property "Reference" "TP8" (id 0) (at 200.025 80.0734 0)
+      (effects (font (size 1.27 1.27)) (justify left))
+    )
+    (property "Value" "TestPoint" (id 1) (at 200.025 82.6134 0)
+      (effects (font (size 1.27 1.27)) (justify left))
+    )
+    (property "Footprint" "TestPoint:TestPoint_Pad_1.0x1.0mm" (id 2) (at 203.2 82.55 0)
+      (effects (font (size 1.27 1.27)) hide)
+    )
+    (property "Datasheet" "~" (id 3) (at 203.2 82.55 0)
+      (effects (font (size 1.27 1.27)) hide)
+    )

Commit message: bump to kicad 6, init uEFI v3
Parts:
- C52, C53, C54, C55, C56, C57: footprint Capacitor_SMD:C_0603_1608Metric -> Capacitor_SMD:C_0805_2012Metric
Other:
- company: (none) -> Churrosoft
- title: (none) -> uEFI

Commit message: move old boards to __old
Parts:
- C52, C53, C54, C55, C56, C57: footprint Capacitor_SMD:C_0805_2012Metric -> Capacitor_SMD:C_0603_1608Metric
Other:
- company: Churrosoft -> (none)
- title: uEFI -> (none)
