File: µEFI_rev2/µEFI_rev2.kicad_sch (KiCad schematic)
At the start: 53 parts, among them J1 USB_B, J2 Tag connect, Q8 SS8050, Q9 SS8050, SW1 SW_Push, U1 MCZ33810EK, U23 PaP_Driver_v1, U3 STM32F407VGTx, U7 25LCxxx, Y1 25MHz

Commit message: uEFI v2 beta release
Parts:
- added C34: 4.7nF, Capacitor_SMD:C_0805_2012Metric, symbol Device:C_Small
- added H1, H2, H3, H4: MountingHole, MountingHole:MountingHole_2.2mm_M2_Pad_Via, symbol Mechanical:MountingHole
- added H5, H6, H7, H8: MountingHole, TestPoint:TestPoint_Pad_D1.0mm, symbol Mechanical:MountingHole
- added R1, R28: R_Small, Resistor_SMD:R_1206_3216Metric, symbol Device:R_Small
- added U15: TJA1042T3118, Package_SO:HTSOP-8-1EP_3.9x4.9mm_P1.27mm_EP2.4x3.2mm, symbol OpenEFI-STM32-rev3:TJA1042T3118
- U1: footprint OpenEFI-STM32F_rev3:SOP65P1030X245-33N -> SOP65P1030X245-33N
Connections:
- net CAN_RX is gone; now on net LED_CAN_RX: R24.2
- net CAN_TX is gone; now on net LED_CAN_TX: R5.2
- net GND1 is gone; now on net GND: J1.4 (GND), J1.5 (Shield)
- net +3V3: now also U15.5 (VIO)
- net +5V: now also U15.3 (VCC)
- net CAN1_RX: now also U15.4 (RXD)
- net CAN1_TX: now also U15.1 (TXD)
- net GND: now also C34.2, U15.2 (GND), U15.8 (STB)
- net VBUS: now also J1.1 (VBUS)
- net 5V_ENABLE: now reaches U3.15 (PC0)
- net CONN_75 renamed H4
- net CONN_76 renamed G4
- net CONN_77 renamed F4
- net CONN_78 renamed E4
- new net: C34.1, R1.1, R28.1
- new net CAN+: R1.2, U15.7 (CANH)
- new net CAN-: R28.2, U15.6 (CANL)
- no-connect marks 13 -> 12
Other:
- moved on the sheet: D1, D10, D12, D13, D5, D6, D7, D8, D9, J1, Q8, Q9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

Commit message: bump to kicad 6, init uEFI v3
Parts:
- added D11: MM3Z24VT1G, Diode_SMD:D_SOD-323, symbol Device:D_Zener
- added H9: MountingHole, MountingHole:MountingHole_2.2mm_M2_Pad_Via, symbol Mechanical:MountingHole
- added J4: Conn_02x08_Odd_Even, Connector_PinHeader_1.27mm:PinHeader_2x08_P1.27mm_Vertical, symbol Connector_Generic:Conn_02x08_Odd_Even
- added J5: Conn_01x03, Connector_PinHeader_2.54mm:PinHeader_1x03_P2.54mm_Vertical, symbol Connector_Generic:Conn_01x03
- added Q11: SS8050, Package_TO_SOT_SMD:SOT-23, symbol Transistor_BJT:2N3055
- added Q12: AO3400A, Package_TO_SOT_SMD:SOT-23, symbol Transistor_FET:AO3400A
- added R34: 1k, Resistor_SMD:R_0603_1608Metric, symbol Device:R
- added R35: 100k, Resistor_SMD:R_0805_2012Metric, symbol Device:R
- added TP9: TestPoint, TestPoint:TestPoint_Pad_1.0x1.0mm, symbol Connector:TestPoint
- R24, R25, R26, R27, R29, R3, R30, R4, R5: value R_Small -> 4.7k; LCSC (none) -> C23162
Connections:
- net +12V: now also R35.1
- net +3V3: now also U7.3 (~{WP}), U7.7 (~{HOLD}), J4.1 (Pin_1)
- net +5V: now also J4.2 (Pin_2)
- net 5V_ENABLE: now also U3.16 (PC1); no longer U3.15 (PC0)
- net AUX_CS_1: now also J4.3 (Pin_3)
- net AUX_CS_2: now also J4.5 (Pin_5)
- net AUX_IN_1: now also J4.7 (Pin_7)
- net AUX_IN_2: now also J4.9 (Pin_9)
- net AUX_IN_3: now also J4.11 (Pin_11)
- net AUX_IN_4: now also J4.13 (Pin_13)
- net GND: now also D11.2 (A), J4.15 (Pin_15), J4.16 (Pin_16), Q11.2 (E), Q12.2 (S)
- net MEMORY_CS: now also TP9.1
- net RPM_OUT: now also R34.1
- net SPI2_MISO: now also J4.6 (Pin_6), J5.3 (Pin_3)
- net SPI2_MOSI: now also J4.8 (Pin_8), J5.2 (Pin_2)
- net SPI2_SCK: now also J4.4 (Pin_4), J5.1 (Pin_1)
- net AUX_OUT_2: now reaches U3.18 (PC3)
- net AUX_OUT_2: now also J4.12 (Pin_12)
- net AUX_OUT_1: now reaches U3.33 (PC4)
- net AUX_OUT_1: now also J4.10 (Pin_10)
- net Sensores/PC5: now reaches U3.34 (PC5)
- net AUX_OUT_3: now reaches U3.35 (PB0)
- net AUX_OUT_3: now also J4.14 (Pin_14)
- net MTR_M1: no longer names the net of U3.92 (PB6)
- net MTR_M_2: no longer names the net of U3.91 (PB5)
- net PAP_ENABLE: no longer names the net of U3.93 (PB7)
- net PWM_ENABLE_1: no longer names the net of U3.96 (PB9)
- net PWM_ENABLE_2: no longer names the net of U3.95 (PB8)
- new net: Q11.1 (B), R34.2
- new net: Q11.3 (C), Q12.1 (G), R35.2
- new net A1: D11.1 (K), Q12.3 (D)
- new net Sensores/PC0: U3.15 (PC0)
- no-connect marks 12 -> 11
Other:
- sheet Sensores ports: added PC0, PC5; removed none
- note added: "SPI"
- note added: "Tachometer out"
- company: (none) -> Churrosoft
- title: (none) -> uEFI
- moved on the sheet: C34, J1, R1, R28, U15

Commit message: move old boards to __old
Parts:
- removed D11: MM3Z24VT1G, Diode_SMD:D_SOD-323, symbol Device:D_Zener
- removed H9: MountingHole, MountingHole:MountingHole_2.2mm_M2_Pad_Via, symbol Mechanical:MountingHole
- removed J4: Conn_02x08_Odd_Even, Connector_PinHeader_1.27mm:PinHeader_2x08_P1.27mm_Vertical, symbol Connector_Generic:Conn_02x08_Odd_Even
- removed J5: Conn_01x03, Connector_PinHeader_2.54mm:PinHeader_1x03_P2.54mm_Vertical, symbol Connector_Generic:Conn_01x03
- removed Q11: SS8050, Package_TO_SOT_SMD:SOT-23, symbol Transistor_BJT:2N3055
- removed Q12: AO3400A, Package_TO_SOT_SMD:SOT-23, symbol Transistor_FET:AO3400A
- removed R34: 1k, Resistor_SMD:R_0603_1608Metric, symbol Device:R
- removed R35: 100k, Resistor_SMD:R_0805_2012Metric, symbol Device:R
- removed TP9: TestPoint, TestPoint:TestPoint_Pad_1.0x1.0mm, symbol Connector:TestPoint
- R24, R25, R26, R27, R29, R3, R30, R4, R5: value 4.7k -> R_Small; LCSC C23162 -> (none)
Connections:
- net Sensores/PC0 is gone; now on net 5V_ENABLE: U3.15 (PC0)
- net +3V3: no longer U7.3 (~{WP}), U7.7 (~{HOLD})
- net 5V_ENABLE: no longer U3.16 (PC1)
- net MTR_M_2: now reaches U3.91 (PB5)
- net MTR_M1: now reaches U3.92 (PB6)
- net PAP_ENABLE: now reaches U3.93 (PB7)
- net PWM_ENABLE_2: now reaches U3.95 (PB8)
- net PWM_ENABLE_1: now reaches U3.96 (PB9)
- net AUX_OUT_1: no longer names the net of U3.33 (PC4)
- net AUX_OUT_2: no longer names the net of U3.18 (PC3)
- net AUX_OUT_3: no longer names the net of U3.35 (PB0)
- net Sensores/PC5: no longer names the net of U3.34 (PC5)
- no-connect marks 11 -> 12
Other:
- sheet Sensores ports: added none; removed PC0, PC5
- note removed: "SPI"
- note removed: "Tachometer out"
- company: Churrosoft -> (none)
- title: uEFI -> (none)
- moved on the sheet: C34, J1, R1, R28, U15
