File: uEFI_rev3/uEFI_rev3.kicad_pcb (KiCad board)
At the start: 4 copper layers, 99.9 x 123 mm, 254 parts, among them J1 USB_B, J2 Tag connect, J3 36638-0002, J4 Conn_02x08_Odd_Even, J5 Conn_01x03, Q1 ISL9V5045S3ST, Q10 IRF540N, Q11 SS8050, Q12 AO3400A, Q2 ISL9V5045S3ST, Q3 ISL9V5045S3ST, Q4 ISL9V5045S3ST, Q5 SS8050, Q6 IRF540N, Q7 IRF540N, Q8 SS8050, Q9 SS8050, SW1 SW_Push, U1 MCZ33810EK, U10 TXS0102DCU, U11 TXS0102DCU, U15 TJA1042T3118, U2 MCP3208, U20 TPL7407LAPWR, U22 TPL7407LAPWR, U23 PaP_Driver_v1, U27 LM321, U3 STM32F407VGTx, U31 LM321, U36 MAX9926UAEE+, U4 MIC2940A-3.3WU, U5 MIC2940A-5.0WT, U6 LT4363IMS, U7 25LCxxx, U8 LM4040DBZ-5, U9 AMS1117, Y1 25MHz

Commit message: rev3, jtag
Parts:
- J2: footprint Connector:Tag-Connect_TC2030-IDC-NL_2x03_P1.27mm_Vertical -> Connector:Tag-Connect_TC2030-IDC-FP_2x03_P1.27mm_Vertical
- TP1: moved to B.Cu
- U6: footprint Package_SO:SOIC-16W_7.5x10.3mm_P1.27mm -> Package_SO:MSOP-12_3x4mm_P0.65mm
- moved C5 44.1 mm to (86.5, 95.0), turned to 0 degrees
- moved C15 20.7 mm to (78.3, 118.3), turned to 45 degrees
- moved C10 18.0 mm to (104.2, 130.8), turned to 180 degrees
- moved C16 14.5 mm to (91.2, 135.1), turned to -45 degrees
- moved C33 10.9 mm to (145.0, 116.5), turned to 0 degrees
- moved D2 7.94 mm to (139.5, 113.3)
- moved Q5 7.69 mm to (139.2, 110.2)
- moved R17 7.69 mm to (139.2, 114.8)
- moved R19 6.35 mm to (139.4, 107.5)
- moved D3 4.69 mm to (139.5, 116.5), turned to 180 degrees
- moved H8 4.06 mm to (76.9, 147.6)
- moved TP1 4.03 mm to (82.8, 117.4), turned to 180 degrees
- moved R2 3.61 mm to (82.0, 120.2)
- moved J4 3.32 mm to (60.4, 140.4)
- moved C13 2.60 mm to (65.2, 135.6), turned to -135 degrees
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Routing:
- net +12V: track 204.6 -> 322.0 mm, vias 7 -> 8
- net +5V: track 113.4 -> 185.6 mm
- net /MTR_ENABLE: track 0.00 -> 69.0 mm
- net /MTR_FAULT: track 0.00 -> 60.6 mm
- net /MTR_STEP: track 0.00 -> 51.9 mm
- net /MTR_DIR: track 0.00 -> 48.0 mm
- net +3V3: track 183.9 -> 230.9 mm, vias 8 -> 13
- net /NRST: track 28.0 -> 74.9 mm, vias 2 -> 3
- net /SYS_SWCLK: track 0.00 -> 45.2 mm, vias 0 -> 2
- net /SYS_SWO: track 0.00 -> 40.8 mm, vias 0 -> 2
- net /SYS_SWDIO: track 0.00 -> 37.3 mm
- net GND: track 185.9 -> 219.2 mm, vias 43 -> 53
- net Net-(C22-Pad2): track 71.8 -> 94.4 mm, vias 0 -> 2
- net /RSP: track 0.00 -> 15.1 mm
- net /RSN: track 0.00 -> 13.6 mm
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Other:
- board text added: "DEBUG"
- board text added: "Deteccion contacto"
- board text removed: "De aca puedo sacar 12v para detectar ACC"
