File: uEFI_rev3/uEFI_rev3.kicad_sch (KiCad schematic)
At the start: 86 parts, among them J1 USB_B, J2 Tag connect, J4 Conn_02x08_Odd_Even, J5 Conn_01x03, Q11 SS8050, Q12 AO3400A, Q8 SS8050, Q9 SS8050, SW1 SW_Push, U1 MCZ33810EK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

Commit message: rev3, analog inputs
Connections:
- net Sensores/PC0 renamed ADC_CS
- net Sensores/PC5: no longer names the net of U3.34 (PC5)
Other:
- sheet Sensores ports: added ADC_CS, SPI2_MISO, SPI2_MOSI, SPI2_SCK; removed PA[0..7], PC0, PC5
- note added: "Sensores"
- moved on the sheet: C34, C7, C8, C9, D1, D10, D5, D6, D7, D8, D9, H1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

Commit message: rev3, PMIC, Relays done
Parts:
- removed TP31: TestPoint, TestPoint:TestPoint_Pad_1.0x1.0mm, symbol Connector:TestPoint
- U7: footprint Package_SO:SOIC-8_3.9x4.9mm_P1.27mm -> Package_SO:SOIC-8_5.275x5.275mm_P1.27mm
Connections:
- net PA0 is gone; now on net AUX_IN_1: U3.23 (PA0)
- net PA1 is gone; now on net AUX_IN_2: U3.24 (PA1)
- net PA2 is gone; now on net AUX_IN_3: U3.25 (PA2)
- net PA3 is gone; now on net AUX_IN_4: U3.26 (PA3)
- net AUX_IN_1: no longer U3.83 (PD2)
- net AUX_IN_2: no longer U3.84 (PD3)
- net AUX_IN_3: no longer U3.85 (PD4)
- net AUX_IN_4: no longer U3.86 (PD5)
- net PMIC_CS: now also U3.77 (PA15); no longer U3.43 (PE12)
- no-connect marks 11 -> 10
Changed lines of the file:
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@@
   (no_connect (at 208.28 158.75))
   (no_connect (at 208.28 151.13))
-  (no_connect (at 205.74 130.81))
   (bus_entry (at 360.68 67.31) (size 2.54 2.54)
     (stroke (width 0.1524) (type solid) (color 0 0 0 0))
@@
     (stroke (width 0.152) (type solid) (color 0 0 0 0))
   )
+  (wire (pts (xy 205.74 130.81) (xy 208.28 130.81))
+    (stroke (width 0) (type solid) (color 0 0 0 0))
+  )
   (polyline (pts (xy 407.035 12.7) (xy 407.035 89.535))
     (stroke (width 0) (type solid) (color 0 0 0 0))
@@
     (stroke (width 0.152) (type solid) (color 0 0 0 0))
   )
-  (wire (pts (xy 320.04 212.09) (xy 321.31 212.09))
-    (stroke (width 0) (type default) (color 0 0 0 0))
-  )
   (wire (pts (xy 177.8 227.33) (xy 177.8 224.79))
     (stroke (width 0) (type solid) (color 0 0 0 0))
@@
     (effects (font (size 1.27 1.27)) (justify right bottom))
   )
-  (text "DEBUG PIN" (at 214.63 131.445 180)
-    (effects (font (size 0.889 0.889)) (justify right bottom))
-  )
   (text "VDD" (at 365.125 141.605 180)
     (effects (font (size 1.27 1.27)) (justify right bottom))
@@
     (effects (font (size 1.27 1.27)) (justify right bottom))
   )
-  (label "PMIC_CS" (at 156.21 166.37 180)
-    (effects (font (size 0.7874 0.7874)) (justify right bottom))
+  (label "PMIC_CS" (at 208.28 130.81 0)
+    (effects (font (size 0.7874 0.7874)) (justify left bottom))
   )
   (label "CAN1_TX" (at 157.48 181.61 180)
@@
     (effects (font (size 1.27 1.27)) (justify left bottom))
   )
-  (label "MEMORY_CS" (at 320.04 212.09 180)
-    (effects (font (size 0.8 0.8)) (justify right bottom))
-  )
   (label "PMIC_MAXI" (at 311.15 49.53 0)
     (effects (font (size 0.7874 0.7874)) (justify left bottom))
@@
     (effects (font (size 0.889 0.889)) (justify right bottom))
   )
-  (label "PA2" (at 212.725 97.79 180)
-    (effects (font (size 1.27 1.27)) (justify right bottom))
-  )
   (label "MTR_STEP" (at 69.85 42.545 180)
     (effects (font (size 1.27 1.27)) (justify right bottom))
@@
     (effects (font (size 0.9906 0.9906)) (justify right bottom))
   )
-  (label "AUX_IN_2" (at 157.48 186.69 180)
+  (label "AUX_IN_2" (at 213.36 95.25 180)
     (effects (font (size 0.889 0.889)) (justify right bottom))
   )
@@
     (effects (font (size 0.8 0.8)) (justify right bottom))
   )
-  (label "AUX_IN_1" (at 157.48 184.15 180)
+  (label "AUX_IN_1" (at 213.36 92.71 180)
     (effects (font (size 0.889 0.889)) (justify right bottom))
   )
@@
     (effects (font (size 0.8 0.8)) (justify right bottom))
   )
-  (label "PA3" (at 212.725 100.33 180)
-    (effects (font (size 1.27 1.27)) (justify right bottom))
-  )
   (label "SPI2_SCK" (at 208.28 161.29 0)
     (effects (font (size 0.7874 0.7874)) (justify left bottom))
@@
     (effects (font (size 0.9906 0.9906)) (justify right bottom))
   )
-  (label "AUX_IN_4" (at 157.48 191.77 180)
+  (label "AUX_IN_4" (at 213.36 100.33 180)
     (effects (font (size 0.889 0.889)) (justify right bottom))
   )
@@
     (effects (font (size 0.889 0.889)) (justify left bottom))
   )
-  (label "PA0" (at 212.725 92.71 180)
-    (effects (font (size 1.27 1.27)) (justify right bottom))
-  )
   (label "SYS_SWDIO" (at 40.005 71.755 0)
     (effects (font (size 0.9906 0.9906)) (justify left bottom))
@@
     (effects (font (size 0.8 0.8)) (justify right bottom))
   )
-  (label "AUX_IN_3" (at 157.48 189.23 180)
+  (label "AUX_IN_3" (at 213.36 97.79 180)
     (effects (font (size 0.889 0.889)) (justify right bottom))
   )
-  (label "PA1" (at 212.725 95.25 180)
-    (effects (font (size 1.27 1.27)) (justify right bottom))
-  )
   (label "INY3" (at 313.69 59.69 0)
     (effects (font (size 1.27 1.27)) (justify left bottom))
@@
     (property "Reference" "U7" (id 0) (at 26.67 168.2558 0))
     (property "Value" "25LCxxx" (id 1) (at 26.67 170.5545 0))
-    (property "Footprint" "Package_SO:SOIC-8_3.9x4.9mm_P1.27mm" (id 2) (at 26.67 180.34 0)
+    (property "Footprint" "Package_SO:SOIC-8_5.275x5.275mm_P1.27mm" (id 2) (at 26.67 180.34 0)
       (effects (font (size 1.27 1.27)) hide)
     )
@@
     (pin "2")
   )
-  (symbol (lib_id "Connector:TestPoint") (at 321.31 212.09 0) (unit 1)
-    (in_bom yes) (on_board yes)
-    (property "Reference" "TP31" (id 0) (at 323.215 209.6134 0)
-      (effects (font (size 1.27 1.27)) (justify left))
-    )
-    (property "Value" "TestPoint" (id 1) (at 323.215 212.1534 0)
-      (effects (font (size 1.27 1.27)) (justify left))
-    )
-    (property "Footprint" "TestPoint:TestPoint_Pad_1.0x1.0mm" (id 2) (at 326.39 212.09 0)
-      (effects (font (size 1.27 1.27)) hide)
-    )
-    (property "Datasheet" "~" (id 3) (at 326.39 212.09 0)
-      (effects (font (size 1.27 1.27)) hide)
-    )
-    (pin "1")
-  )
   (symbol (lib_id "Connector_Generic:Conn_01x03") (at 325.755 124.46 0) (unit 1)
-    (in_bom yes) (on_board no)
+    (in_bom yes) (on_board yes)
     (property "Reference" "J5" (id 0) (at 328.295 123.1899 0)
       (effects (font (size 1.27 1.27)) (justify left))
@@
       (reference "#PWR042") (unit 1) (value "GNDA") (footprint "")
     )
-    (path "/00000000-0000-0000-0000-00005f54b134/9d1b5eb2-4c79-44f3-9c22-d29b24f2a3d3"
-      (reference "#PWR043") (unit 1) (value "GNDA") (footprint "")
-    )
     (path "/1333e0eb-d6cf-4b8a-8a97-298ded665b45"
       (reference "#PWR044") (unit 1) (value "+3V3") (footprint "")
@@
       (reference "#PWR054") (unit 1) (value "GND") (footprint "")
     )
-    (path "/00000000-0000-0000-0000-00005f54b134/5af84632-12ca-4f4d-969f-c188e2d46aa5"
-      (reference "#PWR055") (unit 1) (value "GNDA") (footprint "")
-    )
     (path "/00000000-0000-0000-0000-00005f54b134/1b483365-e24f-40e5-b4c1-401303389a68"
       (reference "#PWR056") (unit 1) (value "GNDA") (footprint "")
@@
       (reference "#PWR057") (unit 1) (value "GNDA") (footprint "")
     )
-    (path "/00000000-0000-0000-0000-00005f54b134/b887083d-575d-45fb-8b23-f4b1c1dc21ec"
-      (reference "#PWR058") (unit 1) (value "GNDA") (footprint "")
-    )
-    (path "/00000000-0000-0000-0000-00005f54b134/bc93973a-9cf9-441b-a1f8-abc482494be4"
-      (reference "#PWR059") (unit 1) (value "GNDA") (footprint "")
-    )
     (path "/00000000-0000-0000-0000-00005f54b134/6f9e6eea-f1a5-4e59-a7b8-03098e367ddb"
       (reference "#PWR060") (unit 1) (value "+5C") (footprint "")
@@
       (reference "#PWR069") (unit 1) (value "GNDA") (footprint "")
     )
-    (path "/00000000-0000-0000-0000-00005f54b134/532e69e2-6055-4d2d-b6b3-2e01d501df5b"
-      (reference "#PWR070") (unit 1) (value "+5C") (footprint "")
-    )
     (path "/00000000-0000-0000-0000-00005f54b134/33b6552b-ec9a-44b7-995a-5c278ca4a586"
       (reference "#PWR071") (unit 1) (value "+5C") (footprint "")
@@
       (reference "#PWR075") (unit 1) (value "+5C") (footprint "")
     )
-    (path "/00000000-0000-0000-0000-00005f54b134/48340eeb-4176-4cbb-bfa6-8bd6a8a41336"
-      (reference "#PWR076") (unit 1) (value "+5C") (footprint "")
-    )
     (path "/00000000-0000-0000-0000-00005f54b134/7b7664bd-b5a0-4337-af80-d11595115b10"
       (reference "#PWR077") (unit 1) (value "GNDA") (footprint "")
@@
       (reference "#PWR0137") (unit 1) (value "+12V") (footprint "")
     )
+    (path "/00000000-0000-0000-0000-00005f54b134/0e6fdc80-8051-4c73-b3eb-29c402a139f7"
+      (reference "#PWR0138") (unit 1) (value "+5V") (footprint "")
+    )
     (path "/4d9b0af3-e2b0-4d93-a19d-62e1cef48392"
       (reference "#PWR0139") (unit 1) (value "GND") (footprint "")
@@
       (reference "#PWR0153") (unit 1) (value "+3V3") (footprint "")
     )
+    (path "/00000000-0000-0000-0000-00005f54b134/cefba56d-6fbd-4947-8a2b-4e6cb2e2b065"
+      (reference "#PWR0154") (unit 1) (value "+5VA") (footprint "")
+    )
+    (path "/00000000-0000-0000-0000-00005f54b134/e4b7cff2-d883-48bd-82a9-00ecae128736"
+      (reference "#PWR0155") (unit 1) (value "+5VA") (footprint "")
+    )
     (path "/00000000-0000-0000-0000-00005f782f71/190e9592-48dd-4b90-9899-59eb2e2f6bcb"
       (reference "#PWR0168") (unit 1) (value "+5VA") (footprint "")
@@
       (reference "#PWR0179") (unit 1) (value "+12VA") (footprint "")
     )
-    (path "/00000000-0000-0000-0000-00005f54b134/0e6fdc80-8051-4c73-b3eb-29c402a139f7"
-      (reference "#PWR?") (unit 1) (value "+5V") (footprint "")
+    (path "/00000000-0000-0000-0000-00005f54b134/2172021a-baf5-4d79-b416-4afde47adedf"
+      (reference "#PWR?") (unit 1) (value "GND") (footprint "")
+    )
+    (path "/00000000-0000-0000-0000-00005f54b134/66dcc784-e0b4-4171-b6ec-1825faa8db59"
+      (reference "#PWR?") (unit 1) (value "GND") (footprint "")
+    )
+    (path "/00000000-0000-0000-0000-00005f54b134/ceeec85b-d741-447a-898f-58717438213d"
+      (reference "#PWR?") (unit 1) (value "GND") (footprint "")
+    )
+    (path "/00000000-0000-0000-0000-00005f54b134/f67ec8d5-4fdb-4d3c-8eba-db9fddd171dd"
+      (reference "#PWR?") (unit 1) (value "GND") (footprint "")
     )
     (path "/00000000-0000-0000-0000-00005f54b134/3e78334a-76d9-456e-9704-a5183b512842"
@@
       (reference "TP30") (unit 1) (value "TestPoint") (footprint "TestPoint:TestPoint_Pad_1.0x1.0mm")
     )
-    (path "/319771cb-995a-4a2b-977e-ae0015814bd4"
-      (reference "TP31") (unit 1) (value "TestPoint") (footprint "TestPoint:TestPoint_Pad_1.0x1.0mm")
-    )
     (path "/00000000-0000-0000-0000-00005f4d8452"
       (reference "U1") (unit 1) (value "MCZ33810EK") (footprint "SOP65P1030X245-33N")
@@
     )
     (path "/28196d4b-da70-496d-ae92-668c3fafb50d"
-      (reference "U7") (unit 1) (value "25LCxxx") (footprint "Package_SO:SOIC-8_3.9x4.9mm_P1.27mm")
+      (reference "U7") (unit 1) (value "25LCxxx") (footprint "Package_SO:SOIC-8_5.275x5.275mm_P1.27mm")
     )
     (path "/00000000-0000-0000-0000-00005f54b134/dbb0226b-20bf-4741-8de0-2d93b92092c8"

Commit message: rev3, jtag
Parts:
- J2: footprint Connector:Tag-Connect_TC2030-IDC-NL_2x03_P1.27mm_Vertical -> Connector:Tag-Connect_TC2030-IDC-FP_2x03_P1.27mm_Vertical
Changed lines of the file:
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@@
       (effects (font (size 1.27 1.27)) (justify left))
     )
-    (property "Footprint" "Connector:Tag-Connect_TC2030-IDC-NL_2x03_P1.27mm_Vertical" (id 2) (at 30.48 74.295 0)
+    (property "Footprint" "Connector:Tag-Connect_TC2030-IDC-FP_2x03_P1.27mm_Vertical" (id 2) (at 30.48 74.295 0)
       (effects (font (size 1.27 1.27)) hide)
     )
@@
       (reference "#PWR0155") (unit 1) (value "+5VA") (footprint "")
     )
+    (path "/00000000-0000-0000-0000-00005f54b134/2172021a-baf5-4d79-b416-4afde47adedf"
+      (reference "#PWR0156") (unit 1) (value "GND") (footprint "")
+    )
+    (path "/00000000-0000-0000-0000-00005f54b134/66dcc784-e0b4-4171-b6ec-1825faa8db59"
+      (reference "#PWR0157") (unit 1) (value "GND") (footprint "")
+    )
+    (path "/00000000-0000-0000-0000-00005f54b134/ceeec85b-d741-447a-898f-58717438213d"
+      (reference "#PWR0158") (unit 1) (value "GND") (footprint "")
+    )
+    (path "/00000000-0000-0000-0000-00005f54b134/f67ec8d5-4fdb-4d3c-8eba-db9fddd171dd"
+      (reference "#PWR0159") (unit 1) (value "GND") (footprint "")
+    )
     (path "/00000000-0000-0000-0000-00005f782f71/190e9592-48dd-4b90-9899-59eb2e2f6bcb"
       (reference "#PWR0168") (unit 1) (value "+5VA") (footprint "")
@@
       (reference "#PWR0179") (unit 1) (value "+12VA") (footprint "")
     )
-    (path "/00000000-0000-0000-0000-00005f54b134/2172021a-baf5-4d79-b416-4afde47adedf"
-      (reference "#PWR?") (unit 1) (value "GND") (footprint "")
-    )
-    (path "/00000000-0000-0000-0000-00005f54b134/66dcc784-e0b4-4171-b6ec-1825faa8db59"
-      (reference "#PWR?") (unit 1) (value "GND") (footprint "")
-    )
-    (path "/00000000-0000-0000-0000-00005f54b134/ceeec85b-d741-447a-898f-58717438213d"
-      (reference "#PWR?") (unit 1) (value "GND") (footprint "")
-    )
-    (path "/00000000-0000-0000-0000-00005f54b134/f67ec8d5-4fdb-4d3c-8eba-db9fddd171dd"
-      (reference "#PWR?") (unit 1) (value "GND") (footprint "")
-    )
     (path "/00000000-0000-0000-0000-00005f54b134/3e78334a-76d9-456e-9704-a5183b512842"
       (reference "C1") (unit 1) (value "240pF") (footprint "Capacitor_SMD:C_0603_1608Metric")
@@
     )
     (path "/00000000-0000-0000-0000-00005f80f0b0"
-      (reference "J2") (unit 1) (value "Tag connect") (footprint "Connector:Tag-Connect_TC2030-IDC-NL_2x03_P1.27mm_Vertical")
+      (reference "J2") (unit 1) (value "Tag connect") (footprint "Connector:Tag-Connect_TC2030-IDC-FP_2x03_P1.27mm_Vertical")
     )
     (path "/00000000-0000-0000-0000-00005f782f71/95a84c7f-8427-45aa-aa8d-5b08de5cde34"
@@
     )
     (path "/00000000-0000-0000-0000-00005f782f71/00000000-0000-0000-0000-00005f782e31"
-      (reference "U6") (unit 1) (value "LT4363IMS") (footprint "Package_SO:SOIC-16W_7.5x10.3mm_P1.27mm")
+      (reference "U6") (unit 1) (value "LT4363IMS") (footprint "Package_SO:MSOP-12_3x4mm_P0.65mm")
     )
     (path "/28196d4b-da70-496d-ae92-668c3fafb50d"

Commit message: rev3, complete routing, ERC
Parts:
- added H10: MountingHole, MountingHole:MountingHole_2.2mm_M2_Pad, symbol Mechanical:MountingHole
Connections:
- net AUX_OUT_2: now also U3.34 (PC5); no longer U3.18 (PC3)
Changed lines of the file:
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@@
     (stroke (width 0) (type solid) (color 0 0 0 0))
   )
+  (wire (pts (xy 205.74 191.77) (xy 208.28 191.77))
+    (stroke (width 0) (type default) (color 0 0 0 0))
+  )
   (polyline (pts (xy 368.935 137.795) (xy 368.935 182.245))
     (stroke (width 0.152) (type solid) (color 0 0 0 0))
@@
     (stroke (width 0) (type solid) (color 0 0 0 0))
   )
-  (wire (pts (xy 205.74 186.69) (xy 208.026 186.69))
+  (wire (pts (xy 205.74 186.69) (xy 208.28 186.69))
     (stroke (width 0) (type solid) (color 0 0 0 0))
   )
@@
     (stroke (width 0.152) (type solid) (color 0 0 0 0))
   )
-  (wire (pts (xy 205.74 191.77) (xy 221.996 191.77))
-    (stroke (width 0) (type solid) (color 0 0 0 0))
-  )
   (wire (pts (xy 157.48 95.25) (xy 157.48 97.79))
     (stroke (width 0) (type solid) (color 0 0 0 0))
@@
     (effects (font (size 1.27 1.27)) (justify left bottom))
   )
-  (label "AUX_OUT_2" (at 208.026 186.69 0)
+  (label "AUX_OUT_2" (at 208.28 191.77 0)
     (effects (font (size 0.889 0.889)) (justify left bottom))
   )
@@
     (pin "2")
   )
+  (symbol (lib_id "Mechanical:MountingHole") (at 344.17 99.695 0) (unit 1)
+    (in_bom yes) (on_board yes)
+    (property "Reference" "H10" (id 0) (at 347.345 99.0599 0)
+      (effects (font (size 1.27 1.27)) (justify left))
+    )
+    (property "Value" "MountingHole" (id 1) (at 347.345 101.5999 0)
+      (effects (font (size 1.27 1.27)) (justify left))
+    )
+    (property "Footprint" "MountingHole:MountingHole_2.2mm_M2_Pad" (id 2) (at 344.17 99.695 0)
+      (effects (font (size 1.27 1.27)) hide)
+    )
+    (property "Datasheet" "~" (id 3) (at 344.17 99.695 0)
+      (effects (font (size 1.27 1.27)) hide)
+    )
+  )
   (symbol (lib_id "Connector:TestPoint") (at 313.69 59.69 90) (unit 1)
     (in_bom yes) (on_board yes)
@@
       (reference "H9") (unit 1) (value "MountingHole") (footprint "MountingHole:MountingHole_2.2mm_M2_Pad_Via")
     )
+    (path "/d319dbef-a888-46e5-8bc0-e7cece3bc254"
+      (reference "H10") (unit 1) (value "MountingHole") (footprint "MountingHole:MountingHole_2.2mm_M2_Pad")
+    )
     (path "/00000000-0000-0000-0000-00005f7cd2f4"
