File: uEFI_rev3/uEFI_rev3.kicad_sch (KiCad schematic)
At the start: 86 parts, among them J1 USB_B, J2 Tag connect, J4 Conn_02x08_Odd_Even, J5 Conn_01x03, Q11 SS8050, Q12 AO3400A, Q8 SS8050, Q9 SS8050, SW1 SW_Push, U1 MCZ33810EK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

Commit message: rev3, added acc detect
Parts:
- added Q13: AO3400A, Package_TO_SOT_SMD:SOT-23, symbol Transistor_FET:AO3400A
- added R58, R59: 10k, Resistor_SMD:R_0603_1608Metric, symbol Device:R_Small
Connections:
- net +3V3: now also R59.1
- net GND: now also Q13.2 (S)
- net ACC_DET: now reaches U3.80 (PC12)
- net ACC_DET: now also R58.1
- new net: Q13.1 (G), R58.2
- new net H1: Q13.3 (D), R59.2
Other:
- note added: "ACC Detect"
Changed lines of the file:
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@@
   (junction (at 40.64 154.305) (diameter 1.016) (color 0 0 0 0)
   )
+  (junction (at 73.025 205.74) (diameter 0) (color 0 0 0 0)
+  )
   (junction (at 185.42 82.55) (diameter 1.016) (color 0 0 0 0)
   )
@@
   (no_connect (at 208.28 153.67))
   (no_connect (at 208.28 146.05))
-  (no_connect (at 208.28 209.55))
+  (no_connect (at 218.44 209.55))
   (no_connect (at 208.28 113.03))
   (no_connect (at 208.28 158.75))
@@
     (stroke (width 0) (type solid) (color 0 0 0 0))
   )
+  (wire (pts (xy 205.74 209.55) (xy 208.28 209.55))
+    (stroke (width 0) (type default) (color 0 0 0 0))
+  )
   (wire (pts (xy 151.13 97.79) (xy 146.05 97.79))
     (stroke (width 0) (type solid) (color 0 0 0 0))
@@
     (stroke (width 0) (type solid) (color 0 0 0 0))
   )
+  (wire (pts (xy 57.15 212.09) (xy 58.42 212.09))
+    (stroke (width 0) (type default) (color 0 0 0 0))
+  )
   (wire (pts (xy 146.05 104.14) (xy 148.59 104.14))
     (stroke (width 0) (type solid) (color 0 0 0 0))
@@
     (stroke (width 0) (type solid) (color 0 0 0 0))
   )
+  (wire (pts (xy 73.025 205.74) (xy 77.47 205.74))
+    (stroke (width 0) (type default) (color 0 0 0 0))
+  )
   (polyline (pts (xy 54.61 40.64) (xy 12.7 40.64))
     (stroke (width 0) (type solid) (color 0 0 0 0))
@@
     (stroke (width 0) (type solid) (color 0 0 0 0))
   )
-  (wire (pts (xy 208.28 209.55) (xy 205.74 209.55))
-    (stroke (width 0) (type solid) (color 0 0 0 0))
-  )
   (wire (pts (xy 313.69 73.66) (xy 317.5 73.66))
     (stroke (width 0) (type solid) (color 0 0 0 0))
@@
     (stroke (width 0) (type solid) (color 0 0 0 0))
   )
+  (wire (pts (xy 73.025 204.47) (xy 73.025 205.74))
+    (stroke (width 0) (type default) (color 0 0 0 0))
+  )
   (wire (pts (xy 313.69 41.91) (xy 317.5 41.91))
     (stroke (width 0) (type solid) (color 0 0 0 0))
@@
     (stroke (width 0) (type solid) (color 0 0 0 0))
   )
+  (polyline (pts (xy 83.82 187.96) (xy 83.82 226.695))
+    (stroke (width 0) (type default) (color 0 0 0 0))
+  )
   (wire (pts (xy 180.34 224.79) (xy 180.34 227.33))
     (stroke (width 0) (type solid) (color 0 0 0 0))
@@
     (stroke (width 0) (type default) (color 0 0 0 0))
   )
+  (wire (pts (xy 73.025 205.74) (xy 73.025 207.01))
+    (stroke (width 0) (type default) (color 0 0 0 0))
+  )
   (wire (pts (xy 96.52 42.545) (xy 102.87 42.545))
     (stroke (width 0) (type solid) (color 0 0 0 0))
@@
     (stroke (width 0) (type solid) (color 0 0 0 0))
   )
+  (polyline (pts (xy 83.82 226.695) (xy 53.975 226.695))
+    (stroke (width 0) (type default) (color 0 0 0 0))
+  )
   (wire (pts (xy 358.14 41.91) (xy 361.95 41.91))
     (stroke (width 0) (type solid) (color 0 0 0 0))
@@
     (stroke (width 0) (type solid) (color 0 0 0 0))
   )
+  (wire (pts (xy 73.025 196.85) (xy 73.025 199.39))
+    (stroke (width 0) (type default) (color 0 0 0 0))
+  )
   (wire (pts (xy 157.48 168.91) (xy 160.02 168.91))
     (stroke (width 0) (type solid) (color 0 0 0 0))
@@
     (stroke (width 0) (type solid) (color 0 0 0 0))
   )
+  (wire (pts (xy 63.5 212.09) (xy 65.405 212.09))
+    (stroke (width 0) (type default) (color 0 0 0 0))
+  )
   (polyline (pts (xy 304.165 89.535) (xy 304.165 12.7))
     (stroke (width 0) (type solid) (color 0 0 0 0))
@@
     (stroke (width 0) (type default) (color 0 0 0 0))
   )
+  (wire (pts (xy 57.15 208.915) (xy 57.15 212.09))
+    (stroke (width 0) (type default) (color 0 0 0 0))
+  )
   (wire (pts (xy 60.96 29.21) (xy 60.96 26.67))
     (stroke (width 0) (type solid) (color 0 0 0 0))
@@
     (stroke (width 0) (type solid) (color 0 0 0 0))
   )
+  (polyline (pts (xy 53.975 187.96) (xy 83.82 187.96))
+    (stroke (width 0) (type default) (color 0 0 0 0))
+  )
   (wire (pts (xy 344.805 168.275) (xy 344.805 172.085))
     (stroke (width 0) (type solid) (color 0 0 0 0))
@@
     (effects (font (size 1.27 1.27)) (justify left bottom))
   )
+  (text "ACC Detect" (at 60.96 199.39 0)
+    (effects (font (size 1 1)) (justify left bottom))
+  )
   (text "Crystal" (at 30.48 16.51 0)
     (effects (font (size 1.27 1.27)) (justify left bottom))
@@
     (effects (font (size 0.889 0.889)) (justify left bottom))
   )
+  (label "ACC_DET" (at 208.28 209.55 0)
+    (effects (font (size 0.889 0.889)) (justify left bottom))
+  )
   (label "VBUS" (at 314.96 248.285 180)
     (effects (font (size 0.8 0.8)) (justify right bottom))
@@
     (effects (font (size 0.889 0.889)) (justify left bottom))
   )
+  (label "ACC_DET" (at 57.15 208.915 0)
+    (effects (font (size 0.889 0.889)) (justify left bottom))
+  )
   (label "SYS_SWCLK" (at 40.005 74.295 0)
     (effects (font (size 0.9906 0.9906)) (justify left bottom))
@@
     )
   )
+  (global_label "H1" (shape input) (at 77.47 205.74 0)
+    (effects (font (size 0.889 0.889)) (justify left))
+    (property "Intersheet References" "${INTERSHEET_REFS}" (id 0) (at 80.937 205.6845 0)
+      (effects (font (size 0.889 0.889)) (justify left) hide)
+    )
+  )
   (global_label "CAN-" (shape input) (at 69.215 267.335 270)
     (effects (font (size 0.889 0.889)) (justify right))
@@
     (pin "1")
   )
+  (symbol (lib_id "Device:R_Small") (at 73.025 201.93 0) (mirror y) (unit 1)
+    (in_bom yes) (on_board yes)
+    (property "Reference" "R59" (id 0) (at 71.12 201.93 90))
+    (property "Value" "10k" (id 1) (at 74.93 201.93 90))
+    (property "Footprint" "Resistor_SMD:R_0603_1608Metric" (id 2) (at 73.025 201.93 0)
+      (effects (font (size 1.27 1.27)) hide)
+    )
+    (property "Datasheet" "~" (id 3) (at 73.025 201.93 0)
+      (effects (font (size 1.27 1.27)) hide)
+    )
+    (pin "1")
+    (pin "2")
+  )
   (symbol (lib_id "Device:LED") (at 372.745 158.115 90) (unit 1)
     (in_bom yes) (on_board yes)
@@
     (pin "1")
   )
+  (symbol (lib_id "power:+3V3") (at 73.025 196.85 0) (unit 1)
+    (in_bom yes) (on_board yes)
+    (property "Reference" "#PWR0161" (id 0) (at 73.025 200.66 0)
+      (effects (font (size 1.27 1.27)) hide)
+    )
+    (property "Value" "+3V3" (id 1) (at 73.406 192.4558 0))
+    (property "Footprint" "" (id 2) (at 73.025 196.85 0)
+      (effects (font (size 1.27 1.27)) hide)
+    )
+    (property "Datasheet" "" (id 3) (at 73.025 196.85 0)
+      (effects (font (size 1.27 1.27)) hide)
+    )
+    (pin "1")
+  )
   (symbol (lib_id "Device:R_Small") (at 372.745 168.275 0) (unit 1)
     (in_bom yes) (on_board yes)
@@
     (pin "2")
   )
+  (symbol (lib_id "Device:R_Small") (at 60.96 212.09 90) (mirror x) (unit 1)
+    (in_bom yes) (on_board yes)
+    (property "Reference" "R58" (id 0) (at 60.96 213.995 90))
+    (property "Value" "10k" (id 1) (at 60.96 210.185 90))
+    (property "Footprint" "Resistor_SMD:R_0603_1608Metric" (id 2) (at 60.96 212.09 0)
+      (effects (font (size 1.27 1.27)) hide)
+    )
+    (property "Datasheet" "~" (id 3) (at 60.96 212.09 0)
+      (effects (font (size 1.27 1.27)) hide)
+    )
+    (pin "1")
+    (pin "2")
+  )
   (symbol (lib_id "Device:R_Small") (at 386.715 212.09 0) (unit 1)
     (in_bom yes) (on_board yes)
@@
     (pin "1")
   )
+  (symbol (lib_id "power:GND") (at 73.025 217.17 0) (unit 1)
+    (in_bom yes) (on_board yes)
+    (property "Reference" "#PWR0160" (id 0) (at 73.025 223.52 0)
+      (effects (font (size 1.27 1.27)) hide)
+    )
+    (property "Value" "GND" (id 1) (at 73.025 221.996 0))
+    (property "Footprint" "" (id 2) (at 73.025 217.17 0)
+      (effects (font (size 1.27 1.27)) hide)
+    )
+    (property "Datasheet" "" (id 3) (at 73.025 217.17 0)
+      (effects (font (size 1.27 1.27)) hide)
+    )
+    (pin "1")
+  )
   (symbol (lib_id "Connector:TestPoint") (at 22.86 191.77 180) (unit 1)
     (in_bom yes) (on_board yes)
@@
     (pin "1")
   )
+  (symbol (lib_id "Transistor_FET:AO3400A") (at 70.485 212.09 0) (unit 1)
+    (in_bom yes) (on_board yes)
+    (property "Reference" "Q13" (id 0) (at 73.914 208.0259 0)
+      (effects (font (size 1.27 1.27)) (justify left))
+    )
+    (property "Value" "AO3400A" (id 1) (at 64.135 206.248 0)
+      (effects (font (size 1.27 1.27)) (justify left))
+    )
+    (property "Footprint" "Package_TO_SOT_SMD:SOT-23" (id 2) (at 75.565 213.995 0)
+      (effects (font (size 1.27 1.27) italic) (justify left) hide)
+    )
+    (property "Datasheet" "http://www.aosmd.com/pdfs/datasheet/AO3400A.pdf" (id 3) (at 70.485 212.09 0)
+      (effects (font (size 1.27 1.27)) (justify left) hide)
+    )
+    (property "LCSC" "C347475" (id 4) (at 70.485 212.09 0)
+      (effects (font (size 0.889 0.889)) hide)
+    )
+    (pin "1")
+    (pin "2")
+    (pin "3")
+  )
   (symbol (lib_id "Device:R_Small") (at 74.93 259.08 270) (unit 1)
     (in_bom yes) (on_board yes)
@@
       (reference "#PWR0159") (unit 1) (value "GND") (footprint "")
     )
+    (path "/5530354c-4c61-4510-8ada-f3233a4ec7f1"
+      (reference "#PWR0160") (unit 1) (value "GND") (footprint "")
+    )
+    (path "/276ef234-ef46-45e1-8284-b23ccabe3e2c"
+      (reference "#PWR0161") (unit 1) (value "+3V3") (footprint "")
+    )
     (path "/00000000-0000-0000-0000-00005f782f71/190e9592-48dd-4b90-9899-59eb2e2f6bcb"
       (reference "#PWR0168") (unit 1) (value "+5VA") (footprint "")
@@
       (reference "Q12") (unit 1) (value "AO3400A") (footprint "Package_TO_SOT_SMD:SOT-23")
     )
+    (path "/98e6bd14-c4d9-4f1a-af49-7e228c75d69d"
+      (reference "Q13") (unit 1) (value "AO3400A") (footprint "Package_TO_SOT_SMD:SOT-23")
+    )
     (path "/998aa3b0-007d-4e6e-8188-0295e07d8264"
       (reference "R1") (unit 1) (value "R_Small") (footprint "Resistor_SMD:R_1206_3216Metric")
@@
       (reference "R57") (unit 1) (value "220") (footprint "Resistor_SMD:R_0603_1608Metric")
     )
+    (path "/4d1c7d0d-0ce4-457a-9ac6-71610fbdc912"
+      (reference "R58") (unit 1) (value "10k") (footprint "Resistor_SMD:R_0603_1608Metric")
+    )
+    (path "/19bf568f-181b-4c09-a22d-a5526a3f0fcf"
+      (reference "R59") (unit 1) (value "10k") (footprint "Resistor_SMD:R_0603_1608Metric")
+    )
     (path "/8d3d2293-e570-4555-b12b-74c389ae5124/e0fc2163-36fb-474e-ad23-a39c6993b4e6"

Commit message: fix 10k res
Parts:
- R35: footprint Resistor_SMD:R_0805_2012Metric -> Resistor_SMD:R_0603_1608Metric
Changed lines of the file:
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@@
     (property "Reference" "R35" (id 0) (at 25.908 93.1418 90))
     (property "Value" "100k" (id 1) (at 25.908 90.8304 90))
-    (property "Footprint" "Resistor_SMD:R_0805_2012Metric" (id 2) (at 25.908 86.106 90)
+    (property "Footprint" "Resistor_SMD:R_0603_1608Metric" (id 2) (at 25.908 86.106 90)
       (effects (font (size 1.27 1.27)) hide)
     )
@@
     )
     (path "/e2d50b7e-967b-4011-b493-b0a5504b221c"
-      (reference "R35") (unit 1) (value "100k") (footprint "Resistor_SMD:R_0805_2012Metric")
+      (reference "R35") (unit 1) (value "100k") (footprint "Resistor_SMD:R_0603_1608Metric")
     )
     (path "/00000000-0000-0000-0000-00005f54b134/4c76534b-7710-410b-a4ce-3373d2652982"
