File: uEFI_rev3/file5F54B133.kicad_sch (KiCad schematic)
At the start: 74 parts, among them U10 TXS0102DCU, U11 TXS0102DCU, U2 MCP3208, U27 LM321, U31 LM321, U8 LM4040DBZ-5, U9 AMS1117

Commit message: uEFI r3.2
Parts:
- D15, D16, D17, D18, D19, D20, D21, D22, D23, D24, D25, D26, D27, D28, D29, D30: footprint Diode_SMD:D_SOD-123F -> Diode_SMD:D_SOD-323
Changed lines of the file:
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@@
       (effects (font (size 1.27 1.27)) (justify left) hide)
     )
-    (property "Footprint" "Diode_SMD:D_SOD-123F" (id 2) (at 208.915 184.15 0)
+    (property "Footprint" "Diode_SMD:D_SOD-323" (id 2) (at 208.915 184.15 0)
       (effects (font (size 1.27 1.27)) hide)
     )
@@
       (effects (font (size 1.27 1.27)) (justify left) hide)
     )
-    (property "Footprint" "Diode_SMD:D_SOD-123F" (id 2) (at 220.345 109.855 0)
+    (property "Footprint" "Diode_SMD:D_SOD-323" (id 2) (at 220.345 109.855 0)
       (effects (font (size 1.27 1.27)) hide)
     )
@@
       (effects (font (size 1.27 1.27)) (justify left) hide)
     )
-    (property "Footprint" "Diode_SMD:D_SOD-123F" (id 2) (at 109.855 140.335 0)
+    (property "Footprint" "Diode_SMD:D_SOD-323" (id 2) (at 109.855 140.335 0)
       (effects (font (size 1.27 1.27)) hide)
     )
@@
       (effects (font (size 1.27 1.27)) (justify left) hide)
     )
-    (property "Footprint" "Diode_SMD:D_SOD-123F" (id 2) (at 109.855 195.58 0)
+    (property "Footprint" "Diode_SMD:D_SOD-323" (id 2) (at 109.855 195.58 0)
       (effects (font (size 1.27 1.27)) hide)
     )
@@
       (effects (font (size 1.27 1.27)) (justify left) hide)
     )
-    (property "Footprint" "Diode_SMD:D_SOD-123F" (id 2) (at 151.13 96.52 0)
+    (property "Footprint" "Diode_SMD:D_SOD-323" (id 2) (at 151.13 96.52 0)
       (effects (font (size 1.27 1.27)) hide)
     )
@@
       (effects (font (size 1.27 1.27)) (justify left) hide)
     )
-    (property "Footprint" "Diode_SMD:D_SOD-123F" (id 2) (at 151.13 152.4 0)
+    (property "Footprint" "Diode_SMD:D_SOD-323" (id 2) (at 151.13 152.4 0)
       (effects (font (size 1.27 1.27)) hide)
     )
@@
       (effects (font (size 1.27 1.27)) (justify left) hide)
     )
-    (property "Footprint" "Diode_SMD:D_SOD-123F" (id 2) (at 151.13 195.58 0)
+    (property "Footprint" "Diode_SMD:D_SOD-323" (id 2) (at 151.13 195.58 0)
       (effects (font (size 1.27 1.27)) hide)
     )
@@
       (effects (font (size 1.27 1.27)) (justify left) hide)
     )
-    (property "Footprint" "Diode_SMD:D_SOD-123F" (id 2) (at 220.345 97.79 0)
+    (property "Footprint" "Diode_SMD:D_SOD-323" (id 2) (at 220.345 97.79 0)
       (effects (font (size 1.27 1.27)) hide)
     )
@@
       (effects (font (size 1.27 1.27)) (justify left) hide)
     )
-    (property "Footprint" "Diode_SMD:D_SOD-123F" (id 2) (at 108.585 97.79 0)
+    (property "Footprint" "Diode_SMD:D_SOD-323" (id 2) (at 108.585 97.79 0)
       (effects (font (size 1.27 1.27)) hide)
     )
@@
       (effects (font (size 1.27 1.27)) (justify left) hide)
     )
-    (property "Footprint" "Diode_SMD:D_SOD-123F" (id 2) (at 151.13 108.585 0)
+    (property "Footprint" "Diode_SMD:D_SOD-323" (id 2) (at 151.13 108.585 0)
       (effects (font (size 1.27 1.27)) hide)
     )
@@
       (effects (font (size 1.27 1.27)) (justify left) hide)
     )
-    (property "Footprint" "Diode_SMD:D_SOD-123F" (id 2) (at 109.855 183.515 0)
+    (property "Footprint" "Diode_SMD:D_SOD-323" (id 2) (at 109.855 183.515 0)
       (effects (font (size 1.27 1.27)) hide)
     )
@@
       (effects (font (size 1.27 1.27)) (justify left) hide)
     )
-    (property "Footprint" "Diode_SMD:D_SOD-123F" (id 2) (at 109.855 152.4 0)
+    (property "Footprint" "Diode_SMD:D_SOD-323" (id 2) (at 109.855 152.4 0)
       (effects (font (size 1.27 1.27)) hide)
     )
@@
       (effects (font (size 1.27 1.27)) (justify left) hide)
     )
-    (property "Footprint" "Diode_SMD:D_SOD-123F" (id 2) (at 108.585 109.855 0)
+    (property "Footprint" "Diode_SMD:D_SOD-323" (id 2) (at 108.585 109.855 0)
       (effects (font (size 1.27 1.27)) hide)
     )
@@
       (effects (font (size 1.27 1.27)) (justify left) hide)
     )
-    (property "Footprint" "Diode_SMD:D_SOD-123F" (id 2) (at 151.13 183.515 0)
+    (property "Footprint" "Diode_SMD:D_SOD-323" (id 2) (at 151.13 183.515 0)
       (effects (font (size 1.27 1.27)) hide)
     )
@@
       (effects (font (size 1.27 1.27)) (justify left) hide)
     )
-    (property "Footprint" "Diode_SMD:D_SOD-123F" (id 2) (at 208.915 172.085 0)
+    (property "Footprint" "Diode_SMD:D_SOD-323" (id 2) (at 208.915 172.085 0)
       (effects (font (size 1.27 1.27)) hide)
     )
@@
       (effects (font (size 1.27 1.27)) (justify left) hide)
     )
-    (property "Footprint" "Diode_SMD:D_SOD-123F" (id 2) (at 151.13 140.335 0)
-      (effects (font (size 1.27 1.27)) hide)
-    )
+    (property "Footprint" "Diode_SMD:D_SOD-323" (id 2) (at 151.13 140.335 0)
+      (effects (font (size 1.27 1.27)) hide)
+    )
