File: uEFI_rev3/connector.kicad_sch (KiCad schematic)
At the start: 23 parts, among them J3 36638-0002, Q10 IRF540N, Q5 SS8050, Q6 IRLZ44N, Q7 IRLZ44N, U4 MIC2940A-3.3WU, U5 MIC2940A-5.0WT, U6 LT4363IMS

Commit message: pre-production files, uEFI v3.4
Parts:
- C36: value 0.1uF -> 100nF; footprint Capacitor_SMD:C_0603_1608Metric -> Capacitor_SMD:C_0805_2012Metric; LCSC (none) -> C49678
Changed lines of the file:
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@@
-    (pin "2")
-  )
-  (symbol (lib_id "Device:C_Small") (at 125.73 127 0) (unit 1)
-    (in_bom yes) (on_board yes)
-    (property "Reference" "C36" (id 0) (at 128.0668 125.8316 0)
-      (effects (font (size 1.27 1.27)) (justify left))
-    )
-    (property "Value" "0.1uF" (id 1) (at 128.0668 128.143 0)
-      (effects (font (size 1.27 1.27)) (justify left))
-    )
-    (property "Footprint" "Capacitor_SMD:C_0603_1608Metric" (id 2) (at 125.73 127 0)
-      (effects (font (size 1.27 1.27)) hide)
-    )
-    (property "Datasheet" "~" (id 3) (at 125.73 127 0)
-      (effects (font (size 1.27 1.27)) hide)
-    )
-    (pin "1")
     (pin "2")
   )
@@
     (pin "1")
   )
+  (symbol (lib_id "Device:C_Small") (at 125.73 127 0) (unit 1)
+    (in_bom yes) (on_board yes)
+    (property "Reference" "C36" (id 0) (at 125.73 125.73 0)
+      (effects (font (size 1.27 1.27)) (justify left))
+    )
+    (property "Value" "100nF" (id 1) (at 125.73 128.27 0)
+      (effects (font (size 1.27 1.27)) (justify left) hide)
+    )
+    (property "Footprint" "Capacitor_SMD:C_0805_2012Metric" (id 2) (at 125.73 127 0)
+      (effects (font (size 1.27 1.27)) hide)
+    )
+    (property "Datasheet" "~" (id 3) (at 125.73 127 0)
+      (effects (font (size 1.27 1.27)) hide)
+    )
+    (property "LCSC" "C49678" (id 4) (at 125.73 127 0)
+      (effects (font (size 1.27 1.27)) hide)
+    )
+    (pin "1")
+    (pin "2")
+  )
   (symbol (lib_id "Device:Jumper_NO_Small") (at 138.684 78.486 0) (unit 1)

Commit message: AA wiring, lib&connector update, added eggbug
Changed lines of the file:
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@@
       (effects (font (size 1.27 1.27)) (justify left))
     )
-    (property "Value" "57.6K 1/10W" (id 1) (at 106.9086 98.933 0)
+    (property "Value" "57.6K 1/10W" (id 1) (at 104.14 92.075 0)
       (effects (font (size 1.27 1.27)) (justify left))
     )
@@
   (symbol (lib_id "Device:R_Small") (at 69.85 109.22 270) (unit 1)
     (in_bom yes) (on_board yes)
-    (property "Reference" "R19" (id 0) (at 69.85 110.49 90))
-    (property "Value" "1M 1/10W" (id 1) (at 69.85 111.76 90))
+    (property "Reference" "R19" (id 0) (at 69.215 107.315 90))
+    (property "Value" "1M 1/10W" (id 1) (at 66.04 111.125 90))
     (property "Footprint" "Resistor_SMD:R_0603_1608Metric" (id 2) (at 69.85 109.22 0)
       (effects (font (size 1.27 1.27)) hide)
@@
       (effects (font (size 1.27 1.27)) (justify left))
     )
-    (property "Value" "10R 1/10W" (id 1) (at 55.88 101.6 0)
+    (property "Value" "10R 1/10W" (id 1) (at 52.07 104.14 0)
       (effects (font (size 1.27 1.27)) (justify left))
     )
@@
   (symbol (lib_id "Device:R_Small") (at 113.03 104.14 270) (unit 1)
     (in_bom yes) (on_board yes)
-    (property "Reference" "R23" (id 0) (at 114.1984 105.6386 0)
-      (effects (font (size 1.27 1.27)) (justify left))
-    )
-    (property "Value" "4.99K 1/10W" (id 1) (at 110.49 101.6 90)
+    (property "Reference" "R23" (id 0) (at 111.125 102.235 90)
+      (effects (font (size 1.27 1.27)) (justify left))
+    )
+    (property "Value" "4.99K 1/10W" (id 1) (at 115.57 102.87 90)
       (effects (font (size 1.27 1.27)) (justify left))
     )
@@
       (effects (font (size 1.27 1.27)) hide)
     )
-    (property "Value" "GND" (id 1) (at 75.057 125.0442 0))
+    (property "Value" "GND" (id 1) (at 77.47 123.19 0)
+      (effects (font (size 0.8 0.8)))
+    )
     (property "Footprint" "" (id 2) (at 74.93 120.65 0)
       (effects (font (size 1.27 1.27)) hide)
@@
       (effects (font (size 1.27 1.27)) (justify left))
     )
-    (property "Value" "SMAJ58CA" (id 1) (at 75.692 101.473 90)
+    (property "Value" "SMAJ58CA" (id 1) (at 74.93 102.235 90)
       (effects (font (size 1.27 1.27)) (justify left))
     )
@@
   (symbol (lib_id "Transistor_BJT:2N3055") (at 55.88 111.76 270) (mirror x) (unit 1)
     (in_bom yes) (on_board yes)
-    (property "Reference" "Q5" (id 0) (at 57.0484 106.934 0)
-      (effects (font (size 1.27 1.27)) (justify left))
-    )
-    (property "Value" "SS8050" (id 1) (at 54.737 106.934 0)
+    (property "Reference" "Q5" (id 0) (at 57.0484 106.934 90)
+      (effects (font (size 1.27 1.27)) (justify left))
+    )
+    (property "Value" "SS8050" (id 1) (at 57.15 116.205 90)
       (effects (font (size 1.27 1.27)) (justify left))
     )
@@
   (symbol (lib_id "Device:C_Small") (at 125.73 127 0) (unit 1)
     (in_bom yes) (on_board yes)
-    (property "Reference" "C36" (id 0) (at 125.73 125.73 0)
-      (effects (font (size 1.27 1.27)) (justify left))
-    )
+    (property "Reference" "C36" (id 0) (at 127 125.095 0)
+      (effects (font (size 1.27 1.27)) (justify left))
+    )
