File: uEFI_rev3/pwm_relays.kicad_sch (KiCad schematic)
At the start: 16 parts, among them U20 TPL7407LAPWR, U22 TPL7407LAPWR

Commit message: fix bom output
Parts:
- U20, U22: LCSC (none) -> C91443
Changed lines of the file:
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@@
       (effects (font (size 1.27 1.27)) hide)
+    )
+    (property "LCSC" "C91443" (id 4) (at 132.715 164.465 0)
+      (effects (font (size 0.889 0.889)) hide)
     )
     (pin "1")
@@
       (effects (font (size 1.27 1.27)) hide)
     )
+    (property "LCSC" "C91443" (id 4) (at 132.08 123.19 0)
+      (effects (font (size 0.889 0.889)) hide)
+    )
     (pin "1")
