File: OpenEFI_rev4/uEFI_rev3.kicad_pcb (KiCad board)
At the start: 4 copper layers, 99 x 113 mm, 267 parts, among them J1 USB_B, J2 Tag connect, J3 36638-0002, J4 Conn_02x08_Odd_Even, J5 Conn_01x03, Q1 ISL9V5045S3ST, Q10 IRF540N, Q11 SS8050, Q12 AO3400A, Q13 AO3400A, Q14 AO3400A, Q15 AO3400A, Q16 AO3400A, Q2 ISL9V5045S3ST, Q3 ISL9V5045S3ST, Q4 ISL9V5045S3ST, Q5 SS8050, Q6 IRLZ44N, Q7 IRLZ44N, Q8 SS8050, Q9 SS8050, SW1 SW_Push, U1 MCZ33810EK, U12 OPA340NA, U15 TJA1042T3118, U2 74HC4851, U20 TPL7407LAPWR, U22 TPL7407LAPWR, U23 PaP_Driver_v1, U27 LM321, U3 STM32F407VGTx, U31 LM321, U36 MAX9926UAEE+, U4 MIC2940A-3.3WU, U5 MIC2940A-5.0WT, U6 LT4363IMS, U7 25LCxxx, U9 OPA340NA, Y1 25MHz

Commit message: import PCB outline from rusEFI / hellen board
Parts:
- added J6: 1241434-1, Library:TE_1241434-1, F.Cu at (199.2, 50.0)
- moved C31 40.7 mm to (90.6, 99.4)
- moved C37 40.7 mm to (109.6, 124.8)
- moved C40 40.7 mm to (102.1, 132.8)
- moved D21 40.7 mm to (106.1, 124.4)
- moved D23 40.7 mm to (106.1, 126.4)
- moved D27 40.7 mm to (106.1, 132.3)
- moved D30 40.7 mm to (106.1, 134.3)
- moved H4 40.7 mm to (109.1, 153.0)
- moved Q6 40.7 mm to (109.6, 88.4)
- moved R18 40.7 mm to (107.6, 91.8)
- moved R22 40.7 mm to (98.6, 106.2)
- moved R51 40.7 mm to (93.1, 145.0)
- moved R58 40.7 mm to (87.6, 116.4)
- moved TP15 40.7 mm to (110.1, 129.1)
- moved TP16 40.7 mm to (109.2, 138.0)
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Connections:
- C53 pad 1: CMP+ -> Net-(SW2-A)
- C55 pad 1: CKP+ -> /CKP/CMP_sensors/CKP_VR
- R117 pad 1: CKP+ -> /CKP/CMP_sensors/CKP_VR
- R121 pad 2: /CKP/CMP_sensors/CKP_VR -> /CMP
- R122 pad 2: /CMP -> /CKP
- R81 pad 1: CMP+ -> Net-(SW2-A)
- TP7 pad 1: /CMP -> /CKP
- TP8 pad 1: /CKP/CMP_sensors/CKP_VR -> /CMP
- U3 pad 6: +3V3 -> Net-(BT1-+)
- U36 pad 4: /CKP/CMP_sensors/CKP_VR -> /CMP
- U36 pad 5: /CMP -> /CKP
Other:
- board size 99 x 113 mm -> 266.7 x 118.1 mm

Commit message: wip PMIC on rev4 board
Parts:
- removed C27, C28, C29, C30: 10nF, Capacitor_SMD:C_0603_1608Metric
- removed F10, F11, F12, F13, F14, F2, F3, F4, F5, F6, F7, F8, F9: 750mA, Fuse:Fuse_0805_2012Metric
- removed the G*** at (67.1, 53.3)
- removed J3: 36638-0002, OpenEFI-STM32F_rev3:366380002
- removed JP11: vr/hall, Jumper:SolderJumper-3_P1.3mm_Bridged2Bar12_Pad1.0x1.5mm_NumberLabels
- removed JP12: Jumper_NC_Small, Jumper:SolderJumper-2_P1.3mm_Open_TrianglePad1.0x1.5mm
- removed Q2, Q3, Q4: ISL9V5045S3ST, Package_TO_SOT_SMD:TO-263-2
- removed R10: 4.02k, Resistor_SMD:R_0603_1608Metric
- removed TP20, TP23, TP25, TP26, TP27: TestPoint, TestPoint:TestPoint_Pad_1.0x1.0mm
- removed U1: MCZ33810EK, uEFI_Library:SOP65P1030X245-33N
- removed U23: PaP_Driver_v1, uEFI_Library:IC_DRV8825_STEPPER_MOTOR_DRIVER_CARRIER
- removed U36: MAX9926UAEE+, OpenEFI-STM32F_rev3:SOP63P602X175-16N
- added BT1: Battery_Cell, Battery:BatteryHolder_Keystone_103_1x20mm, F.Cu at (269.2, 98.6)
- added C45: 0.22uF, Capacitor_SMD:C_0603_1608Metric, F.Cu at (289.7, 133.8)
- added C47: 4700pF, Capacitor_SMD:C_0805_2012Metric, F.Cu at (178.1, 140.0)
- added C50: 0.1uF, Capacitor_SMD:C_0805_2012Metric, F.Cu at (240.8, 179.2)
- added C58: 0.22uF, Capacitor_SMD:C_0603_1608Metric, F.Cu at (289.7, 136.3)
- added C59: 1uF, Capacitor_SMD:C_0805_2012Metric, F.Cu at (228.8, 174.7)
- added C60: 0.1uF, Capacitor_SMD:C_0805_2012Metric, F.Cu at (231.8, 174.7)
- added C61: 0.22uF, Capacitor_SMD:C_0805_2012Metric, F.Cu at (234.8, 174.7)
- added C62: 0.22uF, Capacitor_SMD:C_0805_2012Metric, F.Cu at (237.8, 174.7)
- added C63: 0.1uF, Capacitor_SMD:C_0805_2012Metric, F.Cu at (240.8, 174.7)
- added C64: 100uF, Capacitor_SMD:C_1206_3216Metric, F.Cu at (307.4, 156.5)
- added C65: 0.22uF, Capacitor_SMD:C_0805_2012Metric, F.Cu at (285.4, 129.1)
- added C66: 100nF, Capacitor_SMD:C_0805_2012Metric, F.Cu at (285.4, 132.1)
- added C67: 0.22uF, Capacitor_SMD:C_0603_1608Metric, F.Cu at (289.7, 138.8)
- added C68: 100nF, Capacitor_SMD:C_0805_2012Metric, F.Cu at (285.4, 135.1)
- added C69: 0.22uF, Capacitor_SMD:C_0603_1608Metric, F.Cu at (293.7, 128.8)
- added C70: 100nF, Capacitor_SMD:C_0805_2012Metric, F.Cu at (285.4, 138.1)
- added C71: 0.22uF, Capacitor_SMD:C_0603_1608Metric, F.Cu at (293.7, 131.3)
- added C72: 0.01uF, Capacitor_SMD:C_0805_2012Metric, F.Cu at (189.4, 174.9)
- added C73: 1uF, Capacitor_SMD:C_0805_2012Metric, F.Cu at (185.0, 146.4)
- added C74: 0.1uF, Capacitor_SMD:C_0805_2012Metric, F.Cu at (185.0, 149.4)
- added C75: 0.1uF, Capacitor_SMD:C_0805_2012Metric, F.Cu at (185.0, 152.4)
- added C76: 0.1uF, Capacitor_SMD:C_0805_2012Metric, F.Cu at (185.0, 155.4)
- added D31: K26, Diode_SMD:D_SOD-323, F.Cu at (294.1, 144.5)
- added D32: K26, Diode_SMD:D_SOD-323, F.Cu at (294.1, 147.5)
- added D33: LED, LED_SMD:LED_0805_2012Metric, F.Cu at (190.8, 119.6)
- added D34: LED, LED_SMD:LED_0805_2012Metric, F.Cu at (190.8, 122.6)
- added D35: K26, Diode_SMD:D_SOD-323, F.Cu at (294.1, 150.4)
- added D36: K26, Diode_SMD:D_SOD-323, F.Cu at (294.1, 153.4)
- added D37: K26, Diode_SMD:D_SOD-323, F.Cu at (298.4, 141.6)
- added D38: K26, Diode_SMD:D_SOD-323, F.Cu at (298.4, 144.5)
- added D39: LED, LED_SMD:LED_0805_2012Metric, F.Cu at (190.8, 125.7)
- added D40: LED, LED_SMD:LED_0805_2012Metric, F.Cu at (190.8, 128.7)
- added D41: K26, Diode_SMD:D_SOD-323, F.Cu at (298.4, 147.5)
- added D42: K26, Diode_SMD:D_SOD-323, F.Cu at (298.4, 150.4)
- added D43: LED, LED_SMD:LED_0805_2012Metric, F.Cu at (132.9, 73.8)
- added D44: LED, LED_SMD:LED_0805_2012Metric, F.Cu at (190.8, 134.8)
- added D45: LED, LED_SMD:LED_0805_2012Metric, F.Cu at (190.8, 137.8)
- added D46: LED, LED_SMD:LED_0805_2012Metric, F.Cu at (190.8, 140.9)
- added D47: D, Diode_SMD:D_SOD-323_HandSoldering, F.Cu at (185.7, 119.7)
- added D48: D, Diode_SMD:D_SOD-323, F.Cu at (195.2, 181.8)
- added D49: D, Diode_SMD:D_SOD-323, F.Cu at (198.2, 181.8)
- added D50: D, Diode_SMD:D_SOD-323, F.Cu at (201.1, 181.8)
- added D51: D, Diode_SMD:D_SOD-323, F.Cu at (204.1, 181.8)
- added D52: D, Diode_SMD:D_SOD-323, F.Cu at (207.0, 181.8)
- added D53: D, Diode_SMD:D_SOD-323, F.Cu at (210.0, 181.8)
- added D54: D, Diode_SMD:D_SOD-323, F.Cu at (212.9, 181.8)
- added D55: LED, LED_SMD:LED_0805_2012Metric, F.Cu at (195.3, 119.6)
- added D56: LED, LED_SMD:LED_0805_2012Metric, F.Cu at (195.3, 122.6)
- added D57: LED, LED_SMD:LED_0805_2012Metric, F.Cu at (195.3, 125.7)
- added D58: LED, LED_SMD:LED_0805_2012Metric, F.Cu at (195.3, 128.7)
- added D59: LED, LED_SMD:LED_0805_2012Metric, F.Cu at (195.3, 131.7)
- added D60: LED, LED_SMD:LED_0805_2012Metric, F.Cu at (195.3, 134.8)
- added D61: LED, LED_SMD:LED_0805_2012Metric, F.Cu at (195.3, 137.8)
- added D62: LED, LED_SMD:LED_0805_2012Metric, F.Cu at (195.3, 140.9)
- added D63: LED, LED_SMD:LED_0805_2012Metric, F.Cu at (132.8, 75.9)
- added D64: D, Diode_SMD:D_SOD-323_HandSoldering, F.Cu at (28.9, 0.97)
- added D65: LED, LED_SMD:LED_0805_2012Metric, F.Cu at (132.8, 78.1)
- added D66: D, Diode_SMD:D_SOD-323_HandSoldering, F.Cu at (28.9, 3.92)
- added D67: LED, LED_SMD:LED_0805_2012Metric, F.Cu at (132.9, 80.3)
- added D68: D, Diode_SMD:D_SOD-323_HandSoldering, F.Cu at (28.9, 6.88)
- added D69: LED, LED_SMD:LED_0805_2012Metric, F.Cu at (132.9, 82.4)
- added D70: D, Diode_SMD:D_SOD-323_HandSoldering, F.Cu at (28.9, 9.82)
- added D71: LED, LED_SMD:LED_0805_2012Metric, F.Cu at (132.9, 84.6)
- added D72: D, Diode_SMD:D_SOD-323_HandSoldering, F.Cu at (28.9, 12.8)
- added D73: LED, LED_SMD:LED_0805_2012Metric, F.Cu at (132.9, 86.7)
- added D74: D, Diode_SMD:D_SOD-323_HandSoldering, F.Cu at (28.9, 15.7)
- added D75: LED, LED_SMD:LED_0805_2012Metric, F.Cu at (132.9, 88.9)
- added D76: D, Diode_SMD:D_SOD-123, F.Cu at (185.7, 143.2)
- added D77: LED, LED_SMD:LED_0805_2012Metric, F.Cu at (141.6, 73.7)
- added D78: LED, LED_SMD:LED_0805_2012Metric, F.Cu at (141.6, 75.8)
- added D79: LED, LED_SMD:LED_0805_2012Metric, F.Cu at (141.6, 78.0)
- added D80: LED, LED_SMD:LED_0805_2012Metric, F.Cu at (141.6, 80.2)
- added D81: LED, LED_SMD:LED_0805_2012Metric, F.Cu at (141.6, 82.3)
- added D82: LED, LED_SMD:LED_0805_2012Metric, F.Cu at (141.6, 84.4)
- added D83: LED, LED_SMD:LED_0805_2012Metric, F.Cu at (141.6, 86.6)
- added D84: LED, LED_SMD:LED_0805_2012Metric, F.Cu at (141.6, 88.7)
- added J8: Micro_SD_Card_Det1, Connector_Card:microSD_HC_Hirose_DM3AT-SF-PEJM5, F.Cu at (271.8, 109.2)
- added JP6: Jumper_NO_Small, Jumper:SolderJumper-2_P1.3mm_Open_Pad1.0x1.5mm, F.Cu at (223.1, 159.2)
- added Q17: AO3400A, Package_TO_SOT_SMD:SOT-23, F.Cu at (166.9, 139.8)
- added Q18: AO3400A, Package_TO_SOT_SMD:SOT-23, F.Cu at (171.3, 139.8)
- added R100: 1k, Resistor_SMD:R_0805_2012Metric, F.Cu at (201.1, 168.7)
- added R129: 10k, Resistor_SMD:R_0805_2012Metric, F.Cu at (204.1, 168.7)
- added R130: 10k, Resistor_SMD:R_0805_2012Metric, F.Cu at (207.0, 168.7)
- added R64: 1k, Resistor_SMD:R_0603_1608Metric, F.Cu at (178.8, 152.1)
- added R65: 1k, Resistor_SMD:R_0603_1608Metric, F.Cu at (181.3, 152.1)
- added R66: 0, Resistor_SMD:R_0805_2012Metric, F.Cu at (249.7, 179.3)
- added R67: 180k, Resistor_SMD:R_0805_2012Metric, F.Cu at (252.6, 179.3)
- added R68: 180k, Resistor_SMD:R_0805_2012Metric, F.Cu at (255.6, 179.3)
- added R69: 348k, Resistor_SMD:R_0805_2012Metric, F.Cu at (258.5, 179.3)
- added R70: 348k, Resistor_SMD:R_0805_2012Metric, F.Cu at (261.5, 179.3)
- added R71: 470R, Resistor_SMD:R_0805_2012Metric, F.Cu at (243.8, 174.8)
- added R72: 180k, Resistor_SMD:R_0805_2012Metric, F.Cu at (246.7, 174.8)
- added R73: 180k, Resistor_SMD:R_0805_2012Metric, F.Cu at (249.7, 174.8)
- added R74: 348k, Resistor_SMD:R_0805_2012Metric, F.Cu at (252.6, 174.8)
- added R75: 348k, Resistor_SMD:R_0805_2012Metric, F.Cu at (255.6, 174.8)
- added R76: 2.49k +-1%, Resistor_SMD:R_0603_1608Metric, F.Cu at (301.7, 128.8)
- added R77: 470R, Resistor_SMD:R_0603_1608Metric, F.Cu at (301.7, 131.3)
- added R78: 2.49k +-1%, Resistor_SMD:R_0603_1608Metric, F.Cu at (301.7, 133.8)
- added R79: 470R, Resistor_SMD:R_0603_1608Metric, F.Cu at (301.7, 136.3)
- added R80: 1k, Resistor_SMD:R_0805_2012Metric, F.Cu at (189.4, 170.5)
- added R84: 1k, Resistor_SMD:R_0805_2012Metric, F.Cu at (198.2, 177.5)
- added R85: 1k, Resistor_SMD:R_0805_2012Metric, F.Cu at (201.1, 177.5)
- added R86: 1k, Resistor_SMD:R_0805_2012Metric, F.Cu at (204.1, 177.5)
- added R88: 1k, Resistor_SMD:R_0805_2012Metric, F.Cu at (207.0, 177.5)
- added R89: 1k, Resistor_SMD:R_0805_2012Metric, F.Cu at (210.0, 177.5)
- added R90: 1k, Resistor_SMD:R_0805_2012Metric, F.Cu at (212.9, 177.5)
- added R91: 10k, Resistor_SMD:R_0805_2012Metric, F.Cu at (195.2, 173.1)
- added R92: 10k, Resistor_SMD:R_0805_2012Metric, F.Cu at (198.2, 173.1)
- added R93: 1k, Resistor_SMD:R_0805_2012Metric, F.Cu at (201.1, 173.1)
- added R94: 1k, Resistor_SMD:R_0805_2012Metric, F.Cu at (204.1, 173.1)
- added R95: 1k, Resistor_SMD:R_0805_2012Metric, F.Cu at (207.0, 173.1)
- added R96: 1k, Resistor_SMD:R_0805_2012Metric, F.Cu at (210.0, 173.1)
- added R97: 1k, Resistor_SMD:R_0805_2012Metric, F.Cu at (212.9, 173.1)
- added R98: 1k, Resistor_SMD:R_0805_2012Metric, F.Cu at (195.2, 168.7)
- added R99: 1k, Resistor_SMD:R_0805_2012Metric, F.Cu at (198.2, 168.7)
- added RN1: 1k, Resistor_SMD:R_Array_Convex_4x0603, F.Cu at (138.4, 92.6)
- added RN2: 1k, Resistor_SMD:R_Array_Convex_4x0603, F.Cu at (134.6, 92.6)
- added RN3: 1k, Resistor_SMD:R_Array_Convex_4x0603, F.Cu at (150.1, 96.8)
- added RN4: 1k, Resistor_SMD:R_Array_Convex_4x0603, F.Cu at (154.3, 96.8)
- added SW2: SW_SPDT, Button_Switch_THT:SW_Slide_1P2T_CK_OS102011MS2Q, F.Cu at (168.2, 150.2)
- added SW3: SW_SPDT, Button_Switch_THT:SW_Slide_1P2T_CK_OS102011MS2Q, F.Cu at (174.6, 150.2)
- added TP17: TestPoint_Alt, TestPoint:TestPoint_THTPad_1.0x1.0mm_Drill0.5mm, F.Cu at (305.2, 135.2)
- added U14: ~, Package_SO:SOP-16_3.9x9.9mm_P1.27mm, F.Cu at (304.8, 145.8)
- added U17: LMV324LIDT, Package_SO:SOIC-14_3.9x8.7mm_P1.27mm, F.Cu at (300.3, 160.0)
- added U18: SP720, Package_SO:SOIC-16_3.9x9.9mm_P1.27mm, F.Cu at (291.9, 160.6)
- added U19: TC4424A, Package_SO:SOIC-8_3.9x4.9mm_P1.27mm, F.Cu at (192.8, 145.6)
- added U21: TC4424A, Package_SO:SOIC-8_3.9x4.9mm_P1.27mm, F.Cu at (192.8, 152.1)
- added U26: TC4424A, Package_SO:SOIC-8_3.9x4.9mm_P1.27mm, F.Cu at (192.8, 158.5)
- added U28: MCP2562-E-SN, Package_SO:SOIC-8_3.9x4.9mm_P1.27mm, F.Cu at (201.2, 152.1)
- added U29: TC4424A, Package_SO:SOIC-8_3.9x4.9mm_P1.27mm, F.Cu at (201.2, 158.5)
- added U30: TC4424A, Package_SO:SOIC-8_3.9x4.9mm_P1.27mm, F.Cu at (209.7, 145.6)
- added U32: TC4424A, Package_SO:SOIC-8_3.9x4.9mm_P1.27mm, F.Cu at (209.7, 158.5)
- added U8: BMP280, Package_LGA:Bosch_LGA-8_2x2.5mm_P0.65mm_ClockwisePinNumbering, F.Cu at (306.6, 160.0)
- C18, C20: value 10pF -> 100nF; footprint Capacitor_SMD:C_0603_1608Metric -> Capacitor_SMD:C_0805_2012Metric
- C19, C22: value 10pF -> 0.1uF; footprint Capacitor_SMD:C_0603_1608Metric -> Capacitor_SMD:C_0805_2012Metric
- C21: value 10pF -> 0.22uF
- C23: value 10nF -> 0.22uF
- C24, C26: value 10nF -> 100nF; footprint Capacitor_SMD:C_0603_1608Metric -> Capacitor_SMD:C_0805_2012Metric
- C25: value 10nF -> 270nF; footprint Capacitor_SMD:C_0603_1608Metric -> Capacitor_SMD:C_0805_2012Metric
- C40, C43: value 100nF -> 0.22uF
- C46: value 0.22uF -> 270nF; footprint Capacitor_SMD:C_0603_1608Metric -> Capacitor_SMD:C_0805_2012Metric
- C48: value 0.22uF -> 0.01uF; footprint Capacitor_SMD:C_0603_1608Metric -> Capacitor_SMD:C_0805_2012Metric
- C51: value 240pF -> 0.1uF; footprint Capacitor_SMD:C_0603_1608Metric -> Capacitor_SMD:C_0805_2012Metric
- D14: value K26 -> 1N914WT; footprint Diode_SMD:D_SOD-323 -> Diode_SMD:D_SOD-523
- F1: value 750mA -> Polyfuse; footprint Fuse:Fuse_0805_2012Metric -> Fuse:Fuse_1812_4532Metric; moved to F.Cu
- H2, JP1, JP2, JP3, JP4, JP5, R18, TP1, TP16, TP18, TP2, TP28, TP29, TP3, TP30, TP4, TP5, TP6, TP7, TP8, TP9: moved to F.Cu
- Q1: value ISL9V5045S3ST -> Q_DUAL_NMOS_S1G1D2S2G2D1; footprint Package_TO_SOT_SMD:TO-263-2 -> Package_TO_SOT_SMD:SOT-363_SC-70-6
- R11, R9: value 4.02k -> 470R
- R12: value 4.02k -> 2.49k +-1%
- R13: value 36K -> 470R; footprint Resistor_SMD:R_0603_1608Metric -> Resistor_SMD:R_0805_2012Metric
- R14: value 36K -> 2.49k +-1%
- R15: value 36K -> 470R
- R16: value 36K -> 2.4k; footprint Resistor_SMD:R_0603_1608Metric -> Resistor_SMD:R_0805_2012Metric
- R44: value 2.49k +-1% -> 470R; footprint Resistor_SMD:R_0603_1608Metric -> Resistor_SMD:R_0805_2012Metric
- R45: value 2.49k +-1% -> 1k; footprint Resistor_SMD:R_0603_1608Metric -> Resistor_SMD:R_0805_2012Metric
- R47, R48: value 470R -> 2.49k; footprint Resistor_SMD:R_0603_1608Metric -> Resistor_SMD:R_0805_2012Metric
- R6: value 100R -> 2.49k +-1%
- R60: value 10k -> 470R
- R62, R63: footprint Resistor_SMD:R_0603_1608Metric -> Resistor_SMD:R_0805_2012Metric
- R7: value 100R -> 604R; footprint Resistor_SMD:R_0603_1608Metric -> Resistor_SMD:R_0805_2012Metric
- R8: value 0.02R -> 2.49k +-1%; footprint Resistor_SMD:R_2512_6332Metric -> Resistor_SMD:R_0603_1608Metric
- R82: value 100k 1/10W +-1% -> 470R
- R83: value 20k 1/10W +-1% -> 1k; footprint Resistor_SMD:R_0603_1608Metric -> Resistor_SMD:R_0805_2012Metric
- TP19: value TestPoint -> TestPoint_Alt; footprint TestPoint:TestPoint_Pad_2.0x2.0mm -> TestPoint:TestPoint_THTPad_1.0x1.0mm_Drill0.5mm; moved to F.Cu
- TP21, TP22, TP24: value TestPoint -> TestPoint_Alt; footprint TestPoint:TestPoint_Pad_1.0x1.0mm -> TestPoint:TestPoint_THTPad_1.0x1.0mm_Drill0.5mm; moved to F.Cu
- U27, U31: value LM321 -> TC4424A; footprint Package_TO_SOT_SMD:SOT-23-5 -> Package_SO:SOIC-8_3.9x4.9mm_P1.27mm
- moved R60 273.9 mm to (297.7, 138.8)
- moved TP21 253.2 mm to (308.3, 129.1), turned to 0 degrees
- moved TP22 247.7 mm to (308.3, 132.1), turned to 0 degrees
- moved R8 242.9 mm to (293.7, 136.3), turned to 0 degrees
- moved R9 239.0 mm to (293.7, 138.8)
- moved R14 236.6 mm to (297.7, 133.8)
- moved TP24 233.7 mm to (308.3, 135.2), turned to 0 degrees
- moved R62 232.0 mm to (243.8, 179.3)
- moved R11 228.4 mm to (297.7, 128.8)
- moved R15 226.4 mm to (297.7, 136.3), turned to 0 degrees
- moved R12 226.1 mm to (297.7, 131.3)
- moved TP19 225.6 mm to (305.2, 138.2), turned to 0 degrees
- moved C23 221.2 mm to (289.7, 131.3), turned to 0 degrees
- moved R82 219.8 mm to (301.7, 138.8), turned to 0 degrees
- moved R6 215.5 mm to (293.7, 133.8), turned to 0 degrees
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Connections:
- C18 pad 1: M1 -> B1
- C18 pad 2: /Sheet5FA9324A/FB0 -> GNDA
- C19 pad 1: M2 -> O2_Sensor
- C19 pad 2: /Sheet5FA9324A/FB1 -> GND
- C20 pad 1: L1 -> D1
- C20 pad 2: /Sheet5FA9324A/FB2 -> GNDA
- C21 pad 1: L2 -> /Sensores/CH2
- C21 pad 2: /Sheet5FA9324A/FB3 -> GNDA
- C22 pad 1: GND -> Net-(C22-Pad1)
- C22 pad 2: Net-(Q1-E) -> GND
- C23 pad 1: L1 -> /Sensores/CH6
- C23 pad 2: GND -> GNDA
- C24 pad 1: L2 -> E1
- C24 pad 2: GND -> GNDA
- C25 pad 1: M1 -> ADC-Clamp-5
- C26 pad 1: M2 -> C1
- C26 pad 2: GND -> GNDA
- C38 pad 1: /Sensores/CH2 -> /Sensores/CH4
- C40 pad 1: F1 -> O2-5V
- C40 pad 2: GNDA -> GND
- C41 pad 1: CKP+ -> /CKP
- C41 pad 2: GND -> Net-(C41-Pad2)
- C43 pad 1: G1 -> ADC-Clamp-7
- C43 pad 2: GNDA -> GND
- C44 pad 1: /Sensores/CH3 -> /Sensores/CH5
- C46 pad 1: /Sensores/CH4 -> ADC-Clamp-6
- C46 pad 2: GNDA -> GND
- C48 pad 1: /Sensores/CH5 -> GND
- C48 pad 2: GNDA -> VDDA
- C49 pad 1: Net-(U31-+) -> /Sensores/CH6
- C51 pad 1: Net-(U27-+) -> CLT_Sensor
- C51 pad 2: GNDA -> GND
- D14 pad 1: +3V3 -> Net-(BT1-+)
- D14 pad 2: CKP+ -> +3V3
- D21 pad 2: /Sensores/CH2 -> /Sensores/CH4
- D22 pad 2: /Sensores/CH3 -> /Sensores/CH5
- D23 pad 1: /Sensores/CH2 -> /Sensores/CH4
- D24 pad 1: /Sensores/CH3 -> /Sensores/CH5
- D25 pad 2: /Sensores/CH7 -> /Sensores/CH5
- D26 pad 1: +5C -> /Sensores/CH5
- D26 pad 2: /Sensores/CH4 -> GNDA
- D28 pad 1: /Sensores/CH7 -> /Sensores/CH5
- D29 pad 1: /Sensores/CH4 -> +5C
- D29 pad 2: GNDA -> /Sensores/CH5
- F1 pad 1: Net-(U22-OUT2) -> Net-(SW6-NO_1)
- F1 pad 2: H3 -> VDD
- Q1 pad 1: /Sheet5FA9324A/GD1 -> MCU-D23
- Q1 pad 2: M2 -> +3V3
- Q1 pad 3: Net-(Q1-E) -> (no net)
- R11 pad 1: GND -> /Sensores/CH6
- R11 pad 2: /Sheet5FA9324A/FB2 -> D1
- R12 pad 1: GND -> E1
- R12 pad 2: /Sheet5FA9324A/FB3 -> +5C
- R13 pad 1: /Sheet5FA9324A/FB0 -> O2-5V
- R13 pad 2: M1 -> O2_Sensor
- R14 pad 1: /Sheet5FA9324A/FB1 -> C1
- R14 pad 2: M2 -> +5C
- R15 pad 1: /Sheet5FA9324A/FB2 -> /Sensores/CH7
- R15 pad 2: L1 -> E1
- R16 pad 1: /Sheet5FA9324A/FB3 -> +3V3
- R16 pad 2: L2 -> ADC-Clamp-5
- R42 pad 1: /Sensores/CH2 -> /Sensores/CH4
- R43 pad 1: /Sensores/CH3 -> /Sensores/CH5
- R44 pad 1: F1 -> ADC-Clamp-7
- R44 pad 2: +5C -> Net-(C22-Pad1)
- R45 pad 1: G1 -> ADC-Clamp-6
- R45 pad 2: +5C -> +3V3
- R47 pad 1: /Sensores/CH4 -> IAT_Sensor
- R47 pad 2: F1 -> +3V3
- R48 pad 1: /Sensores/CH5 -> CLT_Sensor
- R48 pad 2: G1 -> +3V3
- R56 pad 1: Net-(U31-+) -> /Sensores/CH6
- R6 pad 1: GND -> B1
- R6 pad 2: /RSN -> +5C
- R60 pad 1: +3V3 -> /Sensores/CH3
- R60 pad 2: CKP+ -> C1
- R62 pad 1: /Sensores/CH6 -> ADC-Clamp-11
- R62 pad 2: Net-(U31--) -> IAT_Sensor
- R63 pad 1: /Sensores/CH7 -> ADC-Clamp-12
- R63 pad 2: Net-(U27--) -> CLT_Sensor
- R7 pad 1: Net-(Q1-E) -> GND
- R7 pad 2: /RSP -> Net-(C22-Pad1)
- R8 pad 1: Net-(Q1-E) -> D1
- R8 pad 2: GND -> +5C
- R82 pad 1: Net-(U27-+) -> /Sensores/CH5
- R82 pad 2: +12VA -> E1
- R83 pad 1: Net-(U27-+) -> Net-(D33-A)
- R83 pad 2: GNDA -> IGN1
- R9 pad 1: GND -> /Sensores/CH2
- R9 pad 2: /Sheet5FA9324A/FB0 -> B1
- TP12 pad 1: /Sensores/CH2 -> /Sensores/CH4
- TP13 pad 1: /Sensores/CH3 -> /Sensores/CH5
- TP14 pad 1: /Sensores/CH4 -> /Sensores/CH5
- TP18 pad 1: Net-(U31--) -> /Sensores/CH6
- TP19 pad 1: Net-(U27--) -> /Sensores/CH5
- TP21 pad 1: /INY2 -> /Sensores/CH6
- TP22 pad 1: /INY3 -> /Sensores/CH7
- TP24 pad 1: /ECN1 -> /Sensores/CH3
- U2 pad 4: Net-(U2-CH7) -> /Sensores/CH7
- U20 pad 10: /PWM/Relays/MIL_OUT -> D3
- U20 pad 11: /PWM/Relays/CHECK_ENGINE -> E3
- U20 pad 12: Net-(U20-OUT5) -> B4
- U20 pad 13: Net-(U20-OUT4) -> B4
- U20 pad 14: Net-(U20-OUT3) -> C4
- U20 pad 15: Net-(U20-OUT2) -> C4
- U20 pad 16: Net-(U20-OUT1) -> C4
- U22 pad 10: /PWM/Relays/R3_OUT -> F3
- U22 pad 11: Net-(U22-OUT6) -> D4
- U22 pad 12: Net-(U22-OUT5) -> D4
- U22 pad 13: Net-(U22-OUT4) -> G3
- U22 pad 14: Net-(U22-OUT3) -> G3
- U22 pad 15: Net-(U22-OUT2) -> H3
- U22 pad 16: Net-(U22-OUT1) -> H3
- U27 pad 1: Net-(U27-+) -> unconnected-(U27-NC-Pad1)
- U27 pad 2: GNDA -> Net-(U25-GD2)
- U27 pad 3: Net-(U27--) -> GND
- U27 pad 4: Net-(U27--) -> Net-(U25-GD3)
- U27 pad 5: +5C -> IGN8
- U3 pad 23: /MUX_OUT -> /PA0
- U3 pad 24: unconnected-(U3-PA1-Pad24) -> /PA1
- U3 pad 25: unconnected-(U3-PA2-Pad25) -> /PA2
- U3 pad 26: unconnected-(U3-PA3-Pad26) -> /PA3
- U3 pad 32: /PA7 -> /MUX_OUT
- U31 pad 1: Net-(U31-+) -> unconnected-(U31-NC-Pad1)
- U31 pad 2: GND -> /PMIC/GD0
- U31 pad 3: Net-(U31--) -> unconnected-(U31-GND-Pad3)
- U31 pad 4: Net-(U31--) -> /PMIC/GD1
- U31 pad 5: +12V -> IGN6
Routing:
- net +3V3: track 404.5 -> 0.00 mm, vias 22 -> 0
- net +5C: track 293.4 -> 0.00 mm, vias 18 -> 0
- net +12V: track 266.7 -> 0.00 mm, vias 4 -> 0
- net GND: track 240.7 -> 0.00 mm, vias 57 -> 0
- net /MIL_OUT: track 178.3 -> 0.00 mm, vias 4 -> 0
- net /CHK_OUT: track 171.8 -> 0.00 mm, vias 4 -> 0
- net 5V_ENABLE: track 148.5 -> 0.00 mm, vias 2 -> 0
- net /R_LMB: track 124.8 -> 0.00 mm, vias 2 -> 0
- net /R_ECN_INY: track 123.4 -> 0.00 mm, vias 2 -> 0
- net /R_GNC_GLP: track 122.7 -> 0.00 mm, vias 2 -> 0
- net CKP+: track 122.0 -> 0.00 mm, vias 2 -> 0
- net /R_AAC: track 121.9 -> 0.00 mm, vias 2 -> 0
- net +12VA: track 115.0 -> 0.00 mm, vias 2 -> 0
- net /Sensores/CH6: track 112.7 -> 0.00 mm, vias 4 -> 0
- net /TIM9_CH2: track 112.2 -> 0.00 mm, vias 2 -> 0
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- removed copper zone on B.Cu, net +3V3
- removed copper zone on In1.Cu, net +5C
- removed copper zone on In2.Cu, net GND
- removed copper zone on B.Cu, net GNDA
- removed copper zone on F.Cu, net GNDA
Other:
- board size 266.7 x 118.1 mm -> 164 x 118 mm
- board text added: "1"
- board text added: "8"
- board text added: "Encendido"
- board text added: "Inyección"
- board text removed: "A4"
- board text removed: "A5"
- board text removed: "ACC detect"
- board text removed: "BP"
- board text removed: "Battery"
- board text removed: "CKP SENSOR SETUP"
- board text removed: "CKP Sensor"
- board text removed: "CKP/CMP"
- board text removed: "CMP"
- board text removed: "DEBUG"
- board text removed: "Entradas SW"
- board text removed: "Esta parte del conector tiene que quedar afuera del pcb:"
- board text removed: "Flash"
- board text removed: "HALL"
- board text removed: "O2 Sensor"
- board text removed: "PWM0"
- board text removed: "PWM1"
- board text removed: "PaP Driver"
- board text removed: "RESET"
- board text removed: "RPM Out"
- board text removed: "RSP"
- board text removed: "VR"
- board text removed: "in case of poor signal, short "BP""
- board text removed: "®"
