File: OpenEFI_rev4/uEFI_rev3.kicad_sch (KiCad schematic)
At the start: 91 parts, among them J1 USB_B, J2 Tag connect, J4 Conn_02x08_Odd_Even, J5 Conn_01x03, Q11 SS8050, Q12 AO3400A, Q13 AO3400A, Q8 SS8050, Q9 SS8050, SW1 SW_Push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

Commit message: wip PMIC on rev4 board
Parts:
- removed TP20, TP21, TP22, TP23, TP24, TP25, TP26, TP27: TestPoint, TestPoint:TestPoint_Pad_1.0x1.0mm, symbol Connector:TestPoint
- removed U1: MCZ33810EK, SOP65P1030X245-33N, symbol OpenEFI-STM32-rev3:MCZ33810EK
- added C72: 0.01uF, Capacitor_SMD:C_0805_2012Metric, symbol Device:C
- added J8: Micro_SD_Card_Det1, Connector_Card:microSD_HC_Hirose_DM3AT-SF-PEJM5, symbol Connector:Micro_SD_Card_Det1
- added Q1: Q_DUAL_NMOS_S1G1D2S2G2D1, Package_TO_SOT_SMD:SOT-363_SC-70-6, symbol Device:Q_DUAL_NMOS_S1G1D2S2G2D1
- added R80: 1k, Resistor_SMD:R_0805_2012Metric, symbol Device:R
Connections:
- net PA7 is gone; now on net MUX_OUT: U3.32 (PA7)
- net +3V3: now also Q1.2 (G), R80.2
- net GND: now also C72.1
- net MUX_OUT: no longer U3.23 (PA0)
- net PA1: now reaches U3.24 (PA1)
- net PA2: now reaches U3.25 (PA2)
- net PA3: now reaches U3.26 (PA3)
- new net MCU-D23: C72.2, Q1.1 (S), R80.1
- new net PA0: U3.23 (PA0)
- new net SPARE1-Digital: Q1.6 (D)
Other:
- sheet Sheet5FA9324A renamed PMIC
- sheet PMIC: file Drivers.kicad_sch -> PMIC.kicad_sch
