File: OpenEFI_rev4/file5F54B133.kicad_sch (KiCad schematic)
At the start: 85 parts, among them Q14 AO3400A, Q15 AO3400A, Q16 AO3400A, U10 LMV324, U11 LMV324, U12 OPA340NA, U2 74HC4851, U27 LM321, U31 LM321, U8 BMP280, U9 OPA340NA

Commit message: wip PMIC on rev4 board
Parts:
- removed C40, C43: 100nF, Capacitor_SMD:C_0805_2012Metric, symbol Device:C_Small
- removed C46, C48: 0.22uF, Capacitor_SMD:C_0603_1608Metric, symbol Device:C_Small
- removed C51: 240pF, Capacitor_SMD:C_0603_1608Metric, symbol Device:C_Small
- removed D33, D34: K26, Diode_SMD:D_SOD-323, symbol Diode:BAS316
- removed JP12: Jumper_NC_Small, Jumper:SolderJumper-2_P1.3mm_Open_TrianglePad1.0x1.5mm, symbol Device:Jumper_NC_Small
- removed R44, R45: 2.49k +-1%, Resistor_SMD:R_0603_1608Metric, symbol Device:R_Small
- removed R47, R48, R62, R63: 470R, Resistor_SMD:R_0603_1608Metric, symbol Device:R_Small
- removed R83: 20k 1/10W +-1%, Resistor_SMD:R_0603_1608Metric, symbol Device:R_Small
- removed TP19: TestPoint, TestPoint:TestPoint_Pad_2.0x2.0mm, symbol Connector:TestPoint
- removed U27, U31: LM321, Package_TO_SOT_SMD:SOT-23-5, symbol Amplifier_Operational:LM321
- added C18, C20, C24, C26, C66, C68, C70: 100nF, Capacitor_SMD:C_0805_2012Metric, symbol Device:C_Small
- added C19, C22, C50, C51, C60, C63: 0.1uF, Capacitor_SMD:C_0805_2012Metric, symbol Device:C
- added C21, C23, C58, C67, C69, C71: 0.22uF, Capacitor_SMD:C_0603_1608Metric, symbol Device:C_Small
- added C25, C46: 270nF, Capacitor_SMD:C_0805_2012Metric, symbol Device:C
- added C40, C43, C61, C62, C65: 0.22uF, Capacitor_SMD:C_0805_2012Metric, symbol Device:C
- added C48: 0.01uF, Capacitor_SMD:C_0805_2012Metric, symbol Device:C
- added C59: 1uF, Capacitor_SMD:C_0805_2012Metric, symbol Device:C
- added C64: 100uF, Capacitor_SMD:C_1206_3216Metric, symbol Device:C
- added D36, D37, D38, D41, D42: K26, Diode_SMD:D_SOD-323, symbol Diode:BAS316
- added J7: EBC05DRXN, Misc:EBC05DRXN, symbol Misc:EBC05DRXN
- added R10: 3.88k, Resistor_SMD:R_0603_1608Metric_Pad1.05x0.95mm_HandSolder, symbol Device:R
- added R11, R15, R60, R77, R79, R9: 470R, Resistor_SMD:R_0603_1608Metric, symbol Device:R_Small
- added R12, R14, R6, R76, R78, R8: 2.49k +-1%, Resistor_SMD:R_0603_1608Metric, symbol Device:R_Small
- added R13, R44, R62, R63, R71: 470R, Resistor_SMD:R_0805_2012Metric, symbol Device:R
- added R16: 2.4k, Resistor_SMD:R_0805_2012Metric, symbol Device:R
- added R45: 1k, Resistor_SMD:R_0805_2012Metric, symbol Device:R
- added R47, R48: 2.49k, Resistor_SMD:R_0805_2012Metric, symbol Device:R
- added R66: 0, Resistor_SMD:R_0805_2012Metric, symbol Device:R
- added R67, R68, R72, R73: 180k, Resistor_SMD:R_0805_2012Metric, symbol Device:R
- added R69, R70, R74, R75: 348k, Resistor_SMD:R_0805_2012Metric, symbol Device:R
- added R7: 604R, Resistor_SMD:R_0805_2012Metric, symbol Device:R
- added SW5: SW_DPDT_x2, Misc:AYZ0202AGRLC, symbol Misc:AYZ0202AGRLC
- added TP17, TP19, TP21, TP22, TP24: TestPoint_Alt, TestPoint:TestPoint_THTPad_1.0x1.0mm_Drill0.5mm, symbol Connector:TestPoint_Alt
- added U14: ~, Package_SO:SOP-16_3.9x9.9mm_P1.27mm, symbol Library:SP720
- added U16: KP234, Misc:KP234, symbol Misc:KP234
- added U17: LMV324LIDT, Package_SO:SOIC-14_3.9x8.7mm_P1.27mm, symbol Amplifier_Operational:LMV324
- added U18: SP720, Package_SO:SOIC-16_3.9x9.9mm_P1.27mm, symbol IC_Automotive:SP720
- C45: value 100nF -> 0.22uF; footprint Capacitor_SMD:C_0805_2012Metric -> Capacitor_SMD:C_0603_1608Metric; LCSC C49678 -> (none); now in the parts list
- D31, D32, D35: now in the parts list
- R82: value 100k 1/10W +-1% -> 470R; LCSC C217840 -> (none)
Connections:
- net +12VA is gone; now on net E1: R82.2
- net +3V3: now also C64.2, R16.1, R45.2, R47.2, R48.2, U14.16 (V+), U18.16 (V+); no longer D31.1 (K)
- net +5C: now also D29.1 (K), D31.1 (K), D35.1 (K), D37.1 (K), D41.1 (K), R12.2, R14.2, R6.2, R76.2, R78.2, R8.2; no longer D26.1 (K)
- net B1: now also C18.1, R6.1, R9.2
- net C1: now also C26.1, R14.1, R60.2
- net CH2: now also D31.2 (A), D32.1 (K), C21.1, R9.1, TP17.1; no longer C38.1, D21.2 (A), D23.1 (K), R42.1, TP12.1
- net CH3: now also C58.1, D41.2 (A), D42.1 (K), R60.1, TP24.1; no longer C44.1, D22.2 (A), D24.1 (K), R43.1, TP13.1
- net CH4: now also C38.1, D21.2 (A), D23.1 (K), R42.1, TP12.1; no longer D26.2 (A), D29.1 (K), TP14.1
- net CH5: now also C44.1, D22.2 (A), D24.1 (K), D25.2 (A), D26.1 (K), D28.1 (K), D29.2 (A), R43.1, R82.1, TP13.1, TP14.1, C67.1, C69.1, C71.1, R77.1, R79.1, TP19.1
- net CH6: now also C49.1, D35.2 (A), R56.1, TP18.1, C23.1, D36.1 (K), R11.1, TP21.1
- net CH7: now also C45.1, U2.4 (CH7), D37.2 (A), D38.1 (K), R15.1, TP22.1; no longer D25.2 (A), D28.1 (K)
- net D1: now also C20.1, R11.2, R8.1
- net E1: now also C24.1, C66.1, C68.1, C70.1, R12.1, R15.2, R76.1, R77.2, R78.1, R79.2
- net GND: now also C19.2, C22.2, C25.2, C40.2, C43.2, C46.2, C48.1, C50.2, C51.2, C59.1, C60.1, C61.2, C62.2, C63.2, C64.1, C65.2, J7.A2, J7.B2, R69.1, R7.1, R70.1, R74.1, R75.1, U14.8 (GND), U16.6 (GND), U16.8 (NC), U17.11 (V-), U18.8 (GND)
- net GNDA: now also D26.2 (A), D32.2 (A), C18.2, C20.2, C21.2, C23.2, C24.2, C26.2, C58.2, C66.2, C67.2, C68.2, C69.2, C70.2, C71.2, D36.2 (A), D38.2 (A), D42.2 (A); no longer D29.2 (A), D35.2 (A)
- net MUX_3v3: no longer D32.2 (A)
- removed net OV_DET: C45.1, D31.2 (A), D35.1 (K)
- new net: C22.1, R10.1, R44.2, R7.2
- new net: R73.1, R75.2, U17.12 (+)
- new net: R72.1, R74.2, U17.5 (+)
- new net: R67.1, R69.2, U17.3 (+)
- new net: R66.1, U16.7 (Vout)
- new net: R68.1, R70.2, U17.10 (+)
- new net: J7.A1, J7.B1, SW5.3 (NO_1), SW5.6 (NO_2)
- new net 12V-SW: R10.2
- new net ADC-Clamp-1: U18.1 (I1)
- new net ADC-Clamp-10: U18.11 (I10)
- new net ADC-Clamp-11: C61.1, R62.1, U18.12 (I11)
- new net ADC-Clamp-12: C62.1, R63.1, U18.13 (I12)
- new net ADC-Clamp-13: U17.8, U17.9 (-), U18.14 (I13)
- new net ADC-Clamp-14: U17.13 (-), U17.14, U18.15 (I14)
- new net ADC-Clamp-2: U18.2 (I2)
- new net ADC-Clamp-3: U18.3 (I3)
- new net ADC-Clamp-4: U18.4 (I4)
- new net ADC-Clamp-5: C25.1, R16.2, U18.5 (I5)
- new net ADC-Clamp-6: C46.1, R45.1, U18.6 (I6)
- new net ADC-Clamp-7: C43.1, R44.1, U18.7 (I7)
- new net ADC-Clamp-8: U18.9 (I8)
- new net ADC-Clamp-9: U18.10 (I9)
- new net BARO-5V: C60.2, R66.2, R67.2
- new net CLT_Sensor: C51.1, R48.1, R63.2
- new net IAT_Sensor: C50.1, R47.1, R62.2
- new net MAP-5V: R72.2, SW5.2 (C_1), SW5.5 (C_2)
- new net MAP_External: SW5.1 (NC_1), SW5.4 (NC_2)
- new net MCU-A0: U17.1, U17.2 (-)
- new net MCU-A1: U17.6 (-), U17.7
- new net O2-5V: C40.1, R13.1, R68.2
- new net O2_Sensor: C19.1, R13.2
- new net TPS-5V: C65.1, R71.1, R73.2
- new net TPS_Sensor: C63.1, R71.2
- new net VDDA: C48.2, C59.2, J7.A3, J7.B3, U16.5 (Vcc), U17.4 (V+)
Other:
- note added: "1"
- note added: "5v to 3.3v Opamp"
- note added: "6"
- note added: "7"
- note added: "8"
- note added: "AUX ANALOG"
- note added: "Air Temp"
- note added: "Baro Sensor"
- note added: "Battery reference voltage"
- note added: "Clutch Input"
- note added: "Coolant Temp"
- note added: "Coolant Temperature Sensor"
- note added: "Flex Sensor Input"
- note added: "Inlet Air Temperature Sensor"
- note added: "MAP Sensor"
- note added: "MUX"
- note added: "O2 Sensor"
- note added: "O2 Sensor (narrow or external Wideband)"
- note added: "TPS"
- note added: "Throttle Position Sensor"
- note removed: "3"
- note removed: "5v ADC Vref"
- note removed: "ADC"
- note removed: "OverVoltage detection "made in La Matanza""
- note removed: "TODO: VBAT"
- moved on the sheet: C1, C32, C34, C35, C37, C38, C39, C4, C44, C49, D15, D16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

Commit message: changes on sensors sch
Parts:
- removed C19, C22, C50, C51, C60, C63: 0.1uF, Capacitor_SMD:C_0805_2012Metric, symbol Device:C
- removed C25, C46: 270nF, Capacitor_SMD:C_0805_2012Metric, symbol Device:C
- removed C40, C43, C61, C62, C65: 0.22uF, Capacitor_SMD:C_0805_2012Metric, symbol Device:C
- removed C48: 0.01uF, Capacitor_SMD:C_0805_2012Metric, symbol Device:C
- removed C58: 0.22uF, Capacitor_SMD:C_0603_1608Metric, symbol Device:C_Small
- removed C59: 1uF, Capacitor_SMD:C_0805_2012Metric, symbol Device:C
- removed C64: 100uF, Capacitor_SMD:C_1206_3216Metric, symbol Device:C
- removed D15, D16, D17, D18, D19, D20, D21, D22, D23, D24, D25, D26, D27, D28, D29, D30, D31, D32, D35, D36, D37, D38, D41, D42: K26, Diode_SMD:D_SOD-323, symbol Diode:BAS316
- removed J7: EBC05DRXN, Misc:EBC05DRXN, symbol Misc:EBC05DRXN
- removed R45: 1k, Resistor_SMD:R_0805_2012Metric, symbol Device:R
- removed R55: 200R, Resistor_SMD:R_0603_1608Metric, symbol Device:R_Small
- removed R57: 1k5, Resistor_SMD:R_0603_1608Metric, symbol Device:R_Small
- removed R61: 3k3, Resistor_SMD:R_0603_1608Metric, symbol Device:R_Small
- removed R71: 470R, Resistor_SMD:R_0805_2012Metric, symbol Device:R
- removed R72, R73: 180k, Resistor_SMD:R_0805_2012Metric, symbol Device:R
- removed R74, R75: 348k, Resistor_SMD:R_0805_2012Metric, symbol Device:R
- removed SW5: SW_DPDT_x2, Misc:AYZ0202AGRLC, symbol Misc:AYZ0202AGRLC
- removed TP16, TP18: TestPoint, TestPoint:TestPoint_Pad_2.0x2.0mm, symbol Connector:TestPoint
- removed TP22, TP24: TestPoint_Alt, TestPoint:TestPoint_THTPad_1.0x1.0mm_Drill0.5mm, symbol Connector:TestPoint_Alt
- removed U11: LMV324, symbol Amplifier_Operational:LMV324
- removed U12, U9: OPA340NA, Package_TO_SOT_SMD:SOT-23-5, symbol Amplifier_Operational:OPA340NA
- removed U14: ~, Package_SO:SOP-16_3.9x9.9mm_P1.27mm, symbol Library:SP720
- removed U16: KP234, Misc:KP234, symbol Misc:KP234
- removed U17: LMV324LIDT, Package_SO:SOIC-14_3.9x8.7mm_P1.27mm, symbol Amplifier_Operational:LMV324
- removed U18: SP720, Package_SO:SOIC-16_3.9x9.9mm_P1.27mm, symbol IC_Automotive:SP720
- added C25, C30: 100nF, Capacitor_SMD:C_0805_2012Metric, symbol Device:C_Small
- added C27, C28: 47p, Capacitor_SMD:C_0402_1005Metric, symbol Device:C
- added C29, C46, C50: 0.22uF, Capacitor_SMD:C_0603_1608Metric, symbol Device:C_Small
- added J9: Conn_02x06_Top_Bottom, mx120:mx120g-12, symbol Connector_Generic:Conn_02x06_Top_Bottom
- added R28: 3.88k, Resistor_SMD:R_0603_1608Metric_Pad1.05x0.95mm_HandSolder, symbol Device:R
- added R45, R84: 470R, Resistor_SMD:R_0603_1608Metric, symbol Device:R_Small
- added R55, R57: 180k, Resistor_SMD:R_0805_2012Metric, symbol Device:R
- added R61: 348k, Resistor_SMD:R_0805_2012Metric, symbol Device:R
- added TP16, TP18, TP20, TP23, TP25: TestPoint_Alt, TestPoint:TestPoint_THTPad_1.0x1.0mm_Drill0.5mm, symbol Connector:TestPoint_Alt
- added U19: f042_wideband_module, Library:rusEFI_WBO, symbol wideband_module:f042_wideband_module
- added U25: TJA1051T-3, Package_SO:SOP-8_3.9x4.9mm_P1.27mm, symbol Interface_CAN_LIN:TJA1051T-3
- added U26: ~, Package_SO:SOP-16_3.9x9.9mm_P1.27mm, symbol Library:SP720
- added U9: LMV324, Package_SO:TSSOP-14_4.4x5mm_P0.65mm, symbol Amplifier_Operational:LMV324
- C20, C26: value 100nF -> 0.22uF; footprint Capacitor_SMD:C_0805_2012Metric -> Capacitor_SMD:C_0603_1608Metric; LCSC C49678 -> (none)
- C21, C45: value 0.22uF -> 100nF; footprint Capacitor_SMD:C_0603_1608Metric -> Capacitor_SMD:C_0805_2012Metric; LCSC (none) -> C49678
- R10: value 3.88k -> 180k; footprint Resistor_SMD:R_0603_1608Metric_Pad1.05x0.95mm_HandSolder -> Resistor_SMD:R_0805_2012Metric; Digikey Part Number YAG4550CT-ND -> 311-180KCRCT-ND; Manufacturer_Part_Number RT0603BRD073K88L -> RC0805FR-07180KL; Tolerance 1% -> (none); URL https://www.digikey.com/product-detail/en/yageo/RT0603BRD07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 -> https://www.digikey.com.au/product-detail/en/yageo/RC0805FR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
- R13, R62: value 470R -> 180k; Digikey Part Number P470CCT-ND -> 311-180KCRCT-ND; Manufacturer_Name Panasonic -> Yageo; Manufacturer_Part_Number ERJ-6ENF4700V -> RC0805FR-07180KL; URL https://www.digikey.com/product-detail/en/panasonic-electro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 -> https://www.digikey.com.au/product-detail/en/yageo/RC0805FR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
- R14, R37, R40, R8: value 2.49k +-1% -> 470R
- R15, R39, R43, R9: value 470R -> 2.49k +-1%
- R16: value 2.4k -> 604R; Digikey Part Number 311-2.40KCRCT-ND -> 311-604CRCT-ND; Manufacturer_Part_Number RC0805FR-072K4L -> RC0805FR-07604RL; Tolerance (none) -> 1%; URL https://www.digikey.com/product-detail/en/yageo/RC0805FR-072K4L/311-2.40KCRCT-ND/730637 -> https://www.digikey.com/product-detail/en/yageo/RC0805FR-07604RL/311-604CRCT-ND/731022
- R44, R63: value 470R -> 348k; Digikey Part Number P470CCT-ND -> P348KCDKR-ND; Manufacturer_Part_Number ERJ-6ENF4700V -> ERJ-6ENF3483V; URL https://www.digikey.com/product-detail/en/panasonic-electro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 -> https://www.digikey.com.au/product-detail/en/panasonic-elec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
- R46: value 0 -> 2.49k +-1%
- R47: value 2.49k -> 180k; Digikey Part Number YAG1854CT-ND -> 311-180KCRCT-ND; Manufacturer_Part_Number RT0805BRD072K49L -> RC0805FR-07180KL; Tolerance 0.1% -> (none); URL https://www.digikey.com/product-detail/en/yageo/RT0805BRD07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 -> https://www.digikey.com.au/product-detail/en/yageo/RC0805FR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
- R48: value 2.49k -> 348k; Digikey Part Number YAG1854CT-ND -> P348KCDKR-ND; Manufacturer_Name Yageo -> Panasonic; Manufacturer_Part_Number RT0805BRD072K49L -> ERJ-6ENF3483V; Tolerance 0.1% -> (none); URL https://www.digikey.com/product-detail/en/yageo/RT0805BRD07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 -> https://www.digikey.com.au/product-detail/en/panasonic-elec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
- R66: value 0 -> 348k; Digikey Part Number P0.0ACT-ND -> P348KCDKR-ND; Manufacturer_Part_Number ERJ-6GEY0R00V -> ERJ-6ENF3483V; URL https://www.digikey.com.au/product-detail/en/panasonic-electronic-components/ERJ-6GEY0R00V/P0-0ACT-ND/82955 -> https://www.digikey.com.au/product-detail/en/panasonic-electronic-components/ERJ-6ENF3483V/P348KCDKR-ND/576673
- R7: value 604R -> 348k; Digikey Part Number 311-604CRCT-ND -> P348KCDKR-ND; Manufacturer_Name Yageo -> Panasonic; Manufacturer_Part_Number RC0805FR-07604RL -> ERJ-6ENF3483V; Tolerance 1% -> (none); URL https://www.digikey.com/product-detail/en/yageo/RC0805FR-07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 -> https://www.digikey.com.au/product-detail/en/panasonic-elec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
- U10: footprint (none) -> Package_SO:TSSOP-14_4.4x5mm_P0.65mm
Connections:
- net ADC-Clamp-12 is gone; now on an unnamed net: R63.1
- net +3V3: now also U10.4 (V+), U8.6 (VDDIO), U8.8 (VDD), U26.16 (V+), U9.4 (V+); no longer R16.1, R47.2, R48.2
- net +5C: now also R15.2, R39.2, R43.2, R46.2, R9.2, U19.1 (5V), U25.3 (VCC); no longer R14.2, R37.2, R40.2, R8.2
- net B1: now also C21.1, C24.1, C34.1, C37.1, C39.1, C45.1, R11.2, R12.1, R14.2, R15.1, R37.2, R39.1, R40.2, R41.1, R42.2, R43.1, R60.2, R8.2, R9.1; no longer R9.2
- net CH0: no longer C4.1, R38.1, TP10.1
- net CH1: no longer C35.1, R39.1, TP11.1
- net CH2: no longer C21.1, R9.1, TP17.1
- net CH3: no longer R60.1
- net CH4: no longer C38.1, R42.1, TP12.1
- net CH5: no longer C44.1, C67.1, C69.1, C71.1, R43.1, R77.1, R79.1, R82.1, TP13.1, TP14.1, TP15.1, TP19.1
- net CH6: no longer C23.1, C49.1, R11.1, R56.1, TP21.1
- net CH7: no longer C45.1, R15.1
- net E1: now also R46.1, C30.1, R84.2; no longer C24.1, C39.1, R12.1, R15.2, R41.1, R43.2
- net GND: now also C18.2, C20.2, C21.2, C23.2, C24.2, C26.2, C32.2, C34.2, C35.2, C37.2, C38.2, C39.2, C4.2, C44.2, C45.2, C66.2, C67.2, C68.2, C69.2, C70.2, C71.2, R16.1, R44.2, R48.2, R63.2, R66.2, R69.2, R7.2, R70.2, U10.11 (V-), U8.1 (GND), U8.7 (GND), C25.2, C27.1, C28.2, C29.2, C30.2, C46.2, C50.2, J9.1 (Pin_1), R61.2, U19.10 (HEAT_GND2), U19.2 (GND), U19.9 (HEAT_GND), U25.2 (GND), U25.8 (S), U26.8 (GND), U9.11 (V-); no longer R46.2, R69.1, R7.1, R70.1
- net mux_out: now also R57.2
- net at U10.5 (+): now also R67.1, R69.1
- net at U10.6 (-): now also U10.7
- net at R66.1: now also U10.12 (+), R57.1
- net BARO_CS: now reaches U8.2 (CSB)
- net SPI2_MOSI: now reaches U8.3 (SDI)
- net SPI2_SCK: now reaches U8.4 (SCK)
- net SPI2_MISO: now reaches U8.5 (SDO)
- net at U10.1: now also U10.2 (-)
- net at U10.3 (+): now also R55.1, R61.1
- net at R68.1: now also R70.1, U10.10 (+); no longer R70.2
- net at U10.8: now also U10.9 (-)
- net at U10.13 (-): now also U10.14
- net 12V-SW renamed CH_TPS
- net CH_TPS: now also C71.1, R82.1, TP19.1, U26.12 (I11)
- net ADC-Clamp-11: no longer names the net of R62.1
- net ADC-Clamp-11: now also U9.12 (+)
- net ADC-Clamp-5: no longer names the net of R16.2
- net ADC-Clamp-5: now also C25.1, R28.1, R45.2
- net ADC-Clamp-7: no longer names the net of R44.1
- net ADC-Clamp-7: now also R13.1, U9.10 (+)
- net BARO-5V renamed CH_VBATT
- net CH_VBATT: now also R62.2, C29.1, R45.1, TP20.1, U26.13 (I12); no longer R66.2
- removed net C1: C26.1, C34.1, R14.1, R37.1, R39.2, R60.2
- net CLT_Sensor: no longer names the net of R48.1
- net CLT_Sensor: now also R47.1, U9.3 (+); no longer R63.2
- removed net D1: C20.1, C37.1, R11.2, R40.1, R42.2, R8.1
- removed net GNDA: C18.2, C20.2, C21.2, C23.2, C24.2, C26.2, C32.2, C34.2, C35.2, C37.2, C38.2, C39.2, C4.2, C44.2, C45.2, C66.2, C67.2, C68.2, C69.2, C70.2, C71.2, R46.1
- removed net IAT_Sensor: R47.1, R62.2
- net O2-5V: no longer names the net of R68.2
- net O2-5V: no longer R13.1
- net O2_Sensor renamed CH_MAP
- net CH_MAP: now also C46.1, R84.1, TP23.1, U26.11 (I10)
- new net: R10.1, R7.1, U9.5 (+)
- new net: U9.6 (-), U9.7
- new net: U9.13 (-), U9.14
- new net: U9.1, U9.2 (-)
- new net: U9.8, U9.9 (-)
- new net 12V_RAW: J9.6 (Pin_6)
- new net AUX_CH1: C4.1, R38.1, TP10.1, U26.1 (I1)
- new net AUX_CH2: C20.1, R8.1, TP11.1, U26.2 (I2)
- new net AUX_CH3: C23.1, R11.1, TP12.1, U26.3 (I3)
- new net AUX_CH4: C26.1, R14.1, TP13.1, U26.4 (I4)
- new net AUX_CH5: C35.1, R37.1, TP16.1, U26.5 (I5)
- new net AUX_CH6: C38.1, R40.1, TP17.1, U26.6 (I6)
- new net AUX_CH7: C44.1, R42.1, TP18.1, U26.7 (I7)
- new net AUX_CH8: C50.1, R60.1, TP21.1, U26.9 (I8)
- new net Boot0: U19.8 (Boot0)
- new net CAN+: C27.2, U25.7 (CANH)
- new net CAN-: C28.1, U25.6 (CANL)
- new net CAN_H: J9.11 (Pin_11)
- new net CAN_L: J9.12 (Pin_12)
- new net CAN_RX: U19.5 (CAN_RX), U25.4 (RXD)
- new net CAN_TX: U19.6 (CAN_TX), U25.1 (TXD)
- new net CH_CLT: C69.1, R79.1, TP15.1, U26.14 (I13)
- new net CH_IAT: C67.1, R47.2, R77.1, TP14.1, U26.15 (I14)
- new net CH_O2: C49.1, R55.2, R56.1, TP25.1, U26.10 (I9)
- new net LSU_Heater+: J9.4 (Pin_4), U19.7 (VBatt_Sense)
- new net LSU_Heater-: J9.3 (Pin_3), U19.11 (HEATER-), U19.12 (HEATER-)
- new net LSU_Ip: J9.2 (Pin_2), U19.13 (LSU_ip)
- new net LSU_Rtrim: J9.9 (Pin_9), U19.15 (LSU_rtrim)
- new net LSU_Un: J9.10 (Pin_10), U19.16 (LSU_un)
- new net LSU_Vm: J9.8 (Pin_8), U19.14 (LSU_vm)
- no-connect marks 0 -> 2
Other:
- note added: "MAP"
- note added: "VBATT"
- note added: "black"
- note added: "green"
- note added: "grey"
- note added: "red"
- note added: "rusEFI Wideband"
- note added: "white"
- note added: "yellow"
- note removed: "5v to 3.3v Opamp"
- note removed: "Baro Sensor"
- note removed: "Battery reference voltage"
- note removed: "Clutch Input"
- note removed: "Coolant Temperature Sensor"
- note removed: "Flex Sensor Input"
- note removed: "Inlet Air Temperature Sensor"
- note removed: "MAP Sensor"
- note removed: "O2 Sensor"
- note removed: "Throttle Position Sensor"
- company: Churrosoft -> Churrosoft®
- title: uEFI -> OpenEFI
- moved on the sheet: C32, C4, C66, C67, C68, C69, C70, C71, R36, R38, R76, R77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
