File: OpenEFI_rev4/pwm_relays.kicad_sch (KiCad schematic)
At the start: 16 parts, among them U20 TPL7407LAPWR, U22 TPL7407LAPWR

Commit message: wip PMIC on rev4 board
Parts:
- removed F1, F10, F11, F12, F13, F14, F2, F3, F4, F5, F6, F7, F8, F9: 750mA, Fuse:Fuse_0805_2012Metric, symbol Device:Polyfuse_Small
Connections:
- net CHECK_ENGINE is gone; now on net E3: U20.11 (OUT6)
- net MIL_OUT is gone; now on net D3: U20.10 (OUT7)
- net R3_OUT is gone; now on net F3: U22.10 (OUT7)
- net B4: now also U20.12 (OUT5), U20.13 (OUT4)
- net C4: now also U20.14 (OUT3), U20.15 (OUT2), U20.16 (OUT1)
- net D4: now also U22.11 (OUT6), U22.12 (OUT5)
- net G3: now also U22.13 (OUT4), U22.14 (OUT3)
- net H3: now also U22.15 (OUT2), U22.16 (OUT1)

Commit message: changes on sensors sch
Other:
- company: Churrosoft -> Churrosoft®
- title: uEFI -> OpenEFI
Changed lines of the file:
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@@
   (paper "A4")
   (title_block
-    (title "uEFI")
-    (date "%%date%%")
-    (rev "%%version%%")
-    (company "Churrosoft")
-    (comment 1 "MIT Licence")
+    (title "OpenEFI")
+    (date "2023-10-13")
+    (rev "4.0")
+    (company "Churrosoft®")
+    (comment 1 "CERN-OHL-S Licence")
   )
   (junction (at 149.86 125.095) (diameter 0) (color 0 0 0 0)
