File: OpenEFI_rev4/pwm_relays.kicad_sch (KiCad schematic)
At the start: 2 parts, among them U20 TPL7407LAPWR, U22 TPL7407LAPWR

Commit message: fix board errors
Other:
- note removed: "CONNECTOR BIND"
- moved on the sheet: U20
