File: OpenEFI_rev4/OpenEFI_rev4.kicad_pcb (KiCad board)
At the start: 4 copper layers, 164 x 118 mm, 369 parts, among them J1 USB_B, J2 Tag connect, J4 Conn_02x08_Odd_Even, J5 Conn_01x03, J6 1241434-1, J8 Micro_SD_Card_Det1, Q1 Q_DUAL_NMOS_S1G1D2S2G2D1, Q10 IRF540N, Q11 SS8050, Q12 AO3400A, Q13 AO3400A, Q14 AO3400A, Q15 AO3400A, Q16 AO3400A, Q17 AO3400A, Q18 AO3400A, Q5 SS8050, Q6 IRLZ44N, Q7 IRLZ44N, Q8 SS8050, Q9 SS8050, SW1 SW_Push, SW2 SW_SPDT, SW3 SW_SPDT, U12 OPA340NA, U15 TJA1042T3118, U17 LMV324LIDT, U18 SP720, U19 TC4424A, U2 74HC4851, U20 TPL7407LAPWR, U21 TC4424A, U22 TPL7407LAPWR, U26 TC4424A, U27 TC4424A, U28 MCP2562-E-SN, U29 TC4424A, U3 STM32F407VGTx, U30 TC4424A, U31 TC4424A, U32 TC4424A, U4 MIC2940A-3.3WU, U5 MIC2940A-5.0WT, U6 LT4363IMS, U7 25LCxxx, U8 BMP280, U9 OPA340NA, Y1 25MHz

Commit message: changes on sensors sch
Parts:
- removed C51, C60, C63, C75, C76: 0.1uF, Capacitor_SMD:C_0805_2012Metric
- removed C58: 0.22uF, Capacitor_SMD:C_0603_1608Metric
- removed C59: 1uF, Capacitor_SMD:C_0805_2012Metric
- removed C61, C62, C65: 0.22uF, Capacitor_SMD:C_0805_2012Metric
- removed C64: 100uF, Capacitor_SMD:C_1206_3216Metric
- removed D15, D16, D17, D18, D19, D20, D21, D22, D23, D24, D25, D26, D27, D28, D29, D30, D31, D32, D35, D36, D37, D38, D41, D42: K26, Diode_SMD:D_SOD-323
- removed D33, D34, D39, D40, D44, D45, D46, D55, D56, D57, D58, D59, D60, D61, D62: LED, LED_SMD:LED_0805_2012Metric
- removed D48, D49, D50, D51, D52, D53, D54: D, Diode_SMD:D_SOD-323
- removed H1, H2, H3, H4, H9: MountingHole, MountingHole:MountingHole_2.2mm_M2_Pad_Via
- removed H5, H6, H7, H8: MountingHole, TestPoint:TestPoint_Pad_D1.0mm
- removed J5: Conn_01x03, Connector_PinHeader_2.54mm:PinHeader_1x03_P2.54mm_Vertical
- removed R100, R85, R86, R88, R89, R90, R93, R94, R95, R96, R97, R98, R99: 1k, Resistor_SMD:R_0805_2012Metric
- removed R130, R91, R92: 10k, Resistor_SMD:R_0805_2012Metric
- removed R28: 120R, Resistor_SMD:R_1206_3216Metric
- removed R71: 470R, Resistor_SMD:R_0805_2012Metric
- removed R72, R73: 180k, Resistor_SMD:R_0805_2012Metric
- removed R74, R75: 348k, Resistor_SMD:R_0805_2012Metric
- removed TP22, TP24: TestPoint_Alt, TestPoint:TestPoint_THTPad_1.0x1.0mm_Drill0.5mm
- removed U14: ~, Package_SO:SOP-16_3.9x9.9mm_P1.27mm
- removed U17: LMV324LIDT, Package_SO:SOIC-14_3.9x8.7mm_P1.27mm
- removed U18: SP720, Package_SO:SOIC-16_3.9x9.9mm_P1.27mm
- removed U27, U31, U32: TC4424A, Package_SO:SOIC-8_3.9x4.9mm_P1.27mm
- removed U28: MCP2562-E-SN, Package_SO:SOIC-8_3.9x4.9mm_P1.27mm
- added C27: 47p, Capacitor_SMD:C_0402_1005Metric, F.Cu at (202.4, 109.2)
- added C28: 47p, Capacitor_SMD:C_0402_1005Metric, F.Cu at (202.6, 113.3)
- added C29: 0.22uF, Capacitor_SMD:C_0603_1608Metric, F.Cu at (190.5, 142.9)
- added C30: 100nF, Capacitor_SMD:C_0805_2012Metric, F.Cu at (194.8, 149.2)
- added J7: Conn_01x04, Connector_PinHeader_2.54mm:PinHeader_1x04_P2.54mm_Horizontal, F.Cu at (291.9, 129.3)
- added R10: 180k, Resistor_SMD:R_0805_2012Metric, F.Cu at (151.5, 93.1)
- added TP20: TestPoint_Alt, TestPoint:TestPoint_THTPad_1.0x1.0mm_Drill0.5mm, F.Cu at (184.0, 77.5)
- added TP23: TestPoint_Alt, TestPoint:TestPoint_THTPad_1.0x1.0mm_Drill0.5mm, F.Cu at (184.0, 80.6)
- added TP25: TestPoint_Alt, TestPoint:TestPoint_THTPad_1.0x1.0mm_Drill0.5mm, F.Cu at (184.0, 83.6)
- added U10: LMV324, Package_SO:TSSOP-14_4.4x5mm_P0.65mm, F.Cu at (171.4, 98.5)
- added U24: TC4424A, Package_SO:SOIC-8_3.9x4.9mm_P1.27mm, F.Cu at (149.5, 80.5)
- added U25: TJA1051T-3, Package_SO:SOP-8_3.9x4.9mm_P1.27mm, F.Cu at (182.1, 110.4)
- C19, C22: value 0.1uF -> 47p; footprint Capacitor_SMD:C_0805_2012Metric -> Capacitor_SMD:C_0402_1005Metric
- C20, C26: value 100nF -> 0.22uF; footprint Capacitor_SMD:C_0805_2012Metric -> Capacitor_SMD:C_0603_1608Metric
- C21, C45: value 0.22uF -> 100nF; footprint Capacitor_SMD:C_0603_1608Metric -> Capacitor_SMD:C_0805_2012Metric
- C25: value 270nF -> 100nF
- C40, C43: value 0.22uF -> 1u; footprint Capacitor_SMD:C_0805_2012Metric -> Capacitor_SMD:C_0402_1005Metric
- C46: value 270nF -> 0.22uF; footprint Capacitor_SMD:C_0805_2012Metric -> Capacitor_SMD:C_0603_1608Metric
- C48: value 0.01uF -> 100n; footprint Capacitor_SMD:C_0805_2012Metric -> Capacitor_SMD:C_0402_1005Metric
- C50: value 0.1uF -> 0.22uF; footprint Capacitor_SMD:C_0805_2012Metric -> Capacitor_SMD:C_0603_1608Metric
- D76: footprint Diode_SMD:D_SOD-123 -> Diode_SMD:D_SOD-323_HandSoldering
- J1: footprint Connector_USB:USB_B_OST_USB-B1HSxx_Horizontal -> Connector_USB:USB_Mini-B_Tensility_54-00023_Vertical
- JP6: value Jumper_NO_Small -> SolderJumper_3_Bridged12; footprint Jumper:SolderJumper-2_P1.3mm_Open_Pad1.0x1.5mm -> Jumper:SolderJumper-3_P2.0mm_Open_TrianglePad1.0x1.5mm
- R13, R62: value 470R -> 180k
- R14, R37, R40, R8: value 2.49k +-1% -> 470R
- R15, R39, R43, R9: value 470R -> 2.49k +-1%
- R16: value 2.4k -> 604R
- R44, R63: value 470R -> 348k
- R45, R84: value 1k -> 470R; footprint Resistor_SMD:R_0805_2012Metric -> Resistor_SMD:R_0603_1608Metric
- R46: value 0 -> 2.49k +-1%
- R47: value 2.49k -> 180k
- R48: value 2.49k -> 348k
- R55: value 200R -> 180k; footprint Resistor_SMD:R_0603_1608Metric -> Resistor_SMD:R_0805_2012Metric
- R57: value 1k5 -> 180k; footprint Resistor_SMD:R_0603_1608Metric -> Resistor_SMD:R_0805_2012Metric
- R61: value 3k3 -> 348k; footprint Resistor_SMD:R_0603_1608Metric -> Resistor_SMD:R_0805_2012Metric
- R66: value 0 -> 348k
- R7: value 604R -> 348k
- R83: value 1k -> 10k
- TP16, TP18: value TestPoint -> TestPoint_Alt; footprint TestPoint:TestPoint_Pad_2.0x2.0mm -> TestPoint:TestPoint_THTPad_1.0x1.0mm_Drill0.5mm
- U12: value OPA340NA -> TJA1051T-3; footprint Package_TO_SOT_SMD:SOT-23-5 -> Package_SO:SOP-8_3.9x4.9mm_P1.27mm
- U15: value TJA1042T3118 -> REF3033; footprint Package_SO:HTSOP-8-1EP_3.9x4.9mm_P1.27mm_EP2.4x3.2mm -> Package_TO_SOT_SMD:SOT-23
- U19: value TC4424A -> f042_wideband_module; footprint Package_SO:SOIC-8_3.9x4.9mm_P1.27mm -> Library:rusEFI_WBO
- U26: value TC4424A -> ~; footprint Package_SO:SOIC-8_3.9x4.9mm_P1.27mm -> Package_SO:SOP-16_3.9x9.9mm_P1.27mm
- U9: value OPA340NA -> LMV324; footprint Package_TO_SOT_SMD:SOT-23-5 -> Package_SO:TSSOP-14_4.4x5mm_P0.65mm
- moved J1 239.3 mm to (223.0, 112.9)
- moved TP18 226.6 mm to (310.6, 108.5)
- moved TP16 223.4 mm to (307.6, 114.6)
- moved TP13 219.5 mm to (307.6, 111.6)
- moved R43 217.7 mm to (304.0, 117.7)
- moved R41 215.9 mm to (304.0, 112.7), turned to 0 degrees
- moved C44 213.1 mm to (296.0, 117.7), turned to 0 degrees
- moved TP11 212.8 mm to (307.6, 105.5)
- moved R39 209.9 mm to (304.0, 107.7)
- moved R37 208.6 mm to (304.0, 105.2)
- moved C35 206.6 mm to (296.0, 112.7), turned to 0 degrees
- moved TP12 206.3 mm to (307.6, 108.5)
- moved C39 205.8 mm to (291.8, 120.5)
- moved R42 204.7 mm to (304.0, 115.2)
- moved C37 203.4 mm to (291.8, 117.5)
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Connections:
- C18 pad 2: GNDA -> GND
- C19 pad 1: O2_Sensor -> GND
- C19 pad 2: GND -> CAN+
- C20 pad 1: D1 -> /Sensores/AUX_CH2
- C20 pad 2: GNDA -> GND
- C21 pad 1: /Sensores/CH2 -> B1
- C21 pad 2: GNDA -> GND
- C22 pad 1: Net-(C22-Pad1) -> CAN-
- C23 pad 1: /Sensores/CH6 -> /Sensores/AUX_CH3
- C23 pad 2: GNDA -> GND
- C24 pad 1: E1 -> B1
- C24 pad 2: GNDA -> GND
- C25 pad 1: ADC-Clamp-5 -> Net-(C25-Pad1)
- C26 pad 1: C1 -> /Sensores/AUX_CH4
- C26 pad 2: GNDA -> GND
- C32 pad 2: GNDA -> GND
- C34 pad 1: C1 -> B1
- C34 pad 2: GNDA -> GND
- C35 pad 1: /Sensores/CH1 -> /Sensores/AUX_CH5
- C35 pad 2: GNDA -> GND
- C37 pad 1: D1 -> B1
- C37 pad 2: GNDA -> GND
- C38 pad 1: /Sensores/CH4 -> /Sensores/AUX_CH6
- C38 pad 2: GNDA -> GND
- C39 pad 1: E1 -> B1
- C39 pad 2: GNDA -> GND
- C4 pad 1: /Sensores/CH0 -> /Sensores/AUX_CH1
- C4 pad 2: GNDA -> GND
- C40 pad 1: O2-5V -> +5C
- C43 pad 1: ADC-Clamp-7 -> VDDA
- C44 pad 1: /Sensores/CH5 -> /Sensores/AUX_CH7
- C44 pad 2: GNDA -> GND
- C45 pad 1: /Sensores/CH7 -> B1
- C45 pad 2: GNDA -> GND
- C46 pad 1: ADC-Clamp-6 -> /Sensores/CH_MAP
- C48 pad 1: GND -> VDDA
- C48 pad 2: VDDA -> GND
- C49 pad 1: /Sensores/CH6 -> /Sensores/CH_O2
- C50 pad 1: IAT_Sensor -> /Sensores/AUX_CH8
- C66 pad 2: GNDA -> GND
- C67 pad 1: /Sensores/CH5 -> /Sensores/CH_IAT
- C67 pad 2: GNDA -> GND
- C68 pad 2: GNDA -> GND
- C69 pad 1: /Sensores/CH5 -> /Sensores/CH_CLT
- C69 pad 2: GNDA -> GND
- C70 pad 2: GNDA -> GND
- C71 pad 1: /Sensores/CH5 -> /Sensores/CH_TPS
- C71 pad 2: GNDA -> GND
- D70 pad 1: INJ1 -> INJ5
- D72 pad 1: INJ2 -> INJ6
- D74 pad 1: INJ3 -> INJ7
- D76 pad 1: INJ4 -> INJ8
- D77 pad 2: unconnected-(D77-A-Pad2) -> Net-(D77-A)
- D78 pad 2: unconnected-(D78-A-Pad2) -> Net-(D78-A)
- D79 pad 2: unconnected-(D79-A-Pad2) -> Net-(D79-A)
- D80 pad 2: unconnected-(D80-A-Pad2) -> Net-(D80-A)
- D81 pad 2: unconnected-(D81-A-Pad2) -> Net-(D81-A)
- D82 pad 2: unconnected-(D82-A-Pad2) -> Net-(D82-A)
- D83 pad 2: unconnected-(D83-A-Pad2) -> Net-(D83-A)
- D84 pad 2: unconnected-(D84-A-Pad2) -> Net-(D84-A)
- F1 pad 1: Net-(SW6-NO_1) -> +5C
- F1 pad 2: VDD -> Net-(JP6-A)
- JP6 pad 1: CAN_H -> Net-(JP6-A)
- JP6 pad 2: Net-(JP6-Pad2) -> IGN_V+
- R11 pad 1: /Sensores/CH6 -> /Sensores/AUX_CH3
- R11 pad 2: D1 -> B1
- R12 pad 1: E1 -> B1
- R13 pad 1: O2-5V -> Net-(U9C-+)
- R13 pad 2: O2_Sensor -> /Sensores/CH_MAP
- R14 pad 1: C1 -> /Sensores/AUX_CH4
- R14 pad 2: +5C -> B1
- R15 pad 1: /Sensores/CH7 -> B1
- R15 pad 2: E1 -> +5C
- R16 pad 1: +3V3 -> GND
- R16 pad 2: ADC-Clamp-5 -> Net-(C25-Pad1)
- R37 pad 1: C1 -> /Sensores/AUX_CH5
- R37 pad 2: +5C -> B1
- R38 pad 1: /Sensores/CH0 -> /Sensores/AUX_CH1
- R39 pad 1: /Sensores/CH1 -> B1
- R39 pad 2: C1 -> +5C
- R40 pad 1: D1 -> /Sensores/AUX_CH6
- R40 pad 2: +5C -> B1
- R41 pad 1: E1 -> B1
- R42 pad 1: /Sensores/CH4 -> /Sensores/AUX_CH7
- R42 pad 2: D1 -> B1
- R43 pad 1: /Sensores/CH5 -> B1
- R43 pad 2: E1 -> +5C
- R44 pad 1: ADC-Clamp-7 -> Net-(U9C-+)
- R44 pad 2: Net-(C22-Pad1) -> GND
- R45 pad 1: ADC-Clamp-6 -> /Sensores/CH_VBATT
- R45 pad 2: +3V3 -> Net-(C25-Pad1)
- R46 pad 1: GNDA -> E1
- R46 pad 2: GND -> +5C
- R47 pad 1: IAT_Sensor -> Net-(U9A-+)
- R47 pad 2: +3V3 -> /Sensores/CH_IAT
- R48 pad 1: CLT_Sensor -> Net-(U9A-+)
- R48 pad 2: +3V3 -> GND
- R55 pad 1: /Sensores/MUX_3v3 -> Net-(U10A-+)
- R55 pad 2: Net-(R55-Pad2) -> /Sensores/CH_O2
- R56 pad 1: /Sensores/CH6 -> /Sensores/CH_O2
- R57 pad 1: Net-(R55-Pad2) -> Net-(U10D-+)
- R57 pad 2: Net-(U9--) -> /Sensores/mux_out
- R60 pad 1: /Sensores/CH3 -> /Sensores/AUX_CH8
- R60 pad 2: C1 -> B1
- R61 pad 1: GNDA -> Net-(U10A-+)
- R61 pad 2: /Sensores/MUX_3v3 -> GND
- R62 pad 1: ADC-Clamp-11 -> Net-(U9D-+)
- R62 pad 2: IAT_Sensor -> /Sensores/CH_VBATT
- R63 pad 1: ADC-Clamp-12 -> Net-(U9D-+)
- R63 pad 2: CLT_Sensor -> GND
- R66 pad 1: Net-(U16-Vout) -> Net-(U10D-+)
- R66 pad 2: BARO-5V -> GND
- R67 pad 1: Net-(U17A-+) -> Net-(U10B-+)
- R67 pad 2: BARO-5V -> /Sensores/CH_VBATT
- R68 pad 1: Net-(U17C-+) -> Net-(U10C-+)
- R68 pad 2: O2-5V -> unconnected-(R68-Pad2)
- R69 pad 1: GND -> Net-(U10B-+)
- R69 pad 2: Net-(U17A-+) -> GND
- R7 pad 1: GND -> Net-(U9B-+)
- R7 pad 2: Net-(C22-Pad1) -> GND
- R70 pad 1: GND -> Net-(U10C-+)
- R70 pad 2: Net-(U17C-+) -> GND
- R77 pad 1: /Sensores/CH5 -> /Sensores/CH_IAT
- R79 pad 1: /Sensores/CH5 -> /Sensores/CH_CLT
- R8 pad 1: D1 -> /Sensores/AUX_CH2
- R8 pad 2: +5C -> B1
- R82 pad 1: /Sensores/CH5 -> /Sensores/CH_TPS
- R83 pad 1: Net-(D33-A) -> GND
- R83 pad 2: IGN1 -> /PMIC/PMIC1_ENABLE
- R84 pad 1: Net-(D34-A) -> /Sensores/CH_MAP
- R84 pad 2: IGN2 -> E1
- R9 pad 1: /Sensores/CH2 -> B1
- R9 pad 2: B1 -> +5C
- RN3 pad 1: unconnected-(RN3-R1.1-Pad1) -> Net-(D77-A)
- RN3 pad 2: unconnected-(RN3-R2.1-Pad2) -> Net-(D78-A)
- RN3 pad 3: unconnected-(RN3-R3.1-Pad3) -> Net-(D79-A)
- RN3 pad 4: unconnected-(RN3-R4.1-Pad4) -> Net-(D80-A)
- RN3 pad 5: unconnected-(RN3-R4.2-Pad5) -> IGN3
- RN3 pad 6: unconnected-(RN3-R3.2-Pad6) -> IGN4
- RN3 pad 7: unconnected-(RN3-R2.2-Pad7) -> IGN2
- RN3 pad 8: unconnected-(RN3-R1.2-Pad8) -> IGN1
- RN4 pad 1: unconnected-(RN4-R1.1-Pad1) -> Net-(D81-A)
- RN4 pad 2: unconnected-(RN4-R2.1-Pad2) -> Net-(D82-A)
- RN4 pad 3: unconnected-(RN4-R3.1-Pad3) -> Net-(D83-A)
- RN4 pad 4: unconnected-(RN4-R4.1-Pad4) -> Net-(D84-A)
- RN4 pad 5: unconnected-(RN4-R4.2-Pad5) -> IGN8
- RN4 pad 6: unconnected-(RN4-R3.2-Pad6) -> IGN7
- RN4 pad 7: unconnected-(RN4-R2.2-Pad7) -> IGN6
- RN4 pad 8: unconnected-(RN4-R1.2-Pad8) -> IGN5
- TP10 pad 1: /Sensores/CH0 -> /Sensores/AUX_CH1
- TP11 pad 1: /Sensores/CH1 -> /Sensores/AUX_CH2
- TP12 pad 1: /Sensores/CH4 -> /Sensores/AUX_CH3
- TP13 pad 1: /Sensores/CH5 -> /Sensores/AUX_CH4
- TP14 pad 1: /Sensores/CH5 -> /Sensores/CH_IAT
- TP15 pad 1: /Sensores/CH5 -> /Sensores/CH_CLT
- TP16 pad 1: /MUX_OUT -> /Sensores/AUX_CH5
- TP17 pad 1: /Sensores/CH2 -> /Sensores/AUX_CH6
- TP18 pad 1: /Sensores/CH6 -> /Sensores/AUX_CH7
- TP19 pad 1: /Sensores/CH5 -> /Sensores/CH_TPS
- TP21 pad 1: /Sensores/CH6 -> /Sensores/AUX_CH8
- U12 pad 1: /MUX_OUT -> /CAN_TX
- U12 pad 2: GNDA -> GND
- U12 pad 3: /Sensores/MUX_3v3 -> +5C
- U12 pad 4: /MUX_OUT -> /CAN_RX
- U15 pad 1: /CAN1_TX -> +5C
- U15 pad 2: GND -> VDDA
- U15 pad 3: +5C -> GND
- U19 pad 1: unconnected-(U19-NC-Pad1) -> +5C
- U19 pad 2: Net-(U19-IN_A) -> GND
- U19 pad 3: GND -> unconnected-(U19-SEL_1-Pad3)
- U19 pad 4: Net-(U19-IN_B) -> unconnected-(U19-SEL_2-Pad4)
- U19 pad 5: IGN1 -> /Sensores/CAN_RX
- U19 pad 6: IGN_V+ -> /Sensores/CAN_TX
- U19 pad 7: IGN2 -> /Sensores/LSU_Heater+
- U19 pad 8: unconnected-(U19-NC-Pad8) -> /Sensores/Boot0
- U21 pad 2: Net-(U21-IN_A) -> /PMIC/GD0
- U21 pad 4: Net-(U21-IN_B) -> /PMIC/GD1
- U21 pad 5: IGN5 -> IGN2
- U21 pad 7: IGN6 -> IGN1
- U26 pad 1: unconnected-(U26-NC-Pad1) -> /Sensores/AUX_CH1
- U26 pad 2: Net-(U24-GD2) -> /Sensores/AUX_CH2
- U26 pad 3: GND -> /Sensores/AUX_CH3
- U26 pad 4: Net-(U24-GD3) -> /Sensores/AUX_CH4
- U26 pad 5: IGN4 -> /Sensores/AUX_CH5
- U26 pad 6: IGN_V+ -> /Sensores/AUX_CH6
- U26 pad 7: IGN3 -> /Sensores/AUX_CH7
- U26 pad 8: unconnected-(U26-NC-Pad8) -> GND
- U29 pad 3: unconnected-(U29-GND-Pad3) -> GND
- U29 pad 6: unconnected-(U29-VDD-Pad6) -> IGN_V+
- U3 pad 22: +3V3 -> VDDA
- U30 pad 3: unconnected-(U30-GND-Pad3) -> GND
- U30 pad 6: unconnected-(U30-VDD-Pad6) -> IGN_V+
- U8 pad 1: unconnected-(U8-GND-Pad1) -> GND
- U8 pad 2: unconnected-(U8-CSB-Pad2) -> /Sensores/BARO_CS
- U8 pad 3: unconnected-(U8-SDI-Pad3) -> /Sensores/SPI2_MOSI
- U8 pad 4: unconnected-(U8-SCK-Pad4) -> /Sensores/SPI2_SCK
- U8 pad 5: unconnected-(U8-SDO-Pad5) -> /Sensores/SPI2_MISO
- U8 pad 6: unconnected-(U8-VDDIO-Pad6) -> +3V3
- U8 pad 7: unconnected-(U8-GND-Pad7) -> GND
- U8 pad 8: unconnected-(U8-VDD-Pad8) -> +3V3
- U9 pad 1: Net-(U9--) -> Net-(U9A--)
- U9 pad 2: GNDA -> Net-(U9A--)
- U9 pad 3: /Sensores/mux_out -> Net-(U9A-+)
- U9 pad 4: Net-(U9--) -> +3V3
- U9 pad 5: +5C -> Net-(U9B-+)
Routing:
- net Net-(D77-A): track 0.00 -> 20.6 mm
- net Net-(D78-A): track 0.00 -> 18.2 mm
- net Net-(D79-A): track 0.00 -> 15.7 mm
- net Net-(D80-A): track 0.00 -> 13.4 mm
- net Net-(D81-A): track 0.00 -> 10.6 mm
- net Net-(D82-A): track 0.00 -> 8.09 mm
- net Net-(D83-A): track 0.00 -> 5.52 mm
- net Net-(D84-A): track 0.00 -> 3.07 mm

Commit message: wip sensors pinout:
Parts:
- removed D78, D79, D80, D81, D82, D83, D84: LED, LED_SMD:LED_0805_2012Metric
- removed R112, R113, R114, R118, R119: 4.99K 1/2W, Resistor_SMD:R_1210_3225Metric
- removed R84: 470R, Resistor_SMD:R_0603_1608Metric
- removed SW2, SW3: SW_SPDT, Button_Switch_THT:SW_Slide_1P2T_CK_OS102011MS2Q
- added C51: 0.01uF, Capacitor_SMD:C_0805_2012Metric, F.Cu at (123.5, 188.8)
- added D15: SS26, Diode_SMD:D_SMA, F.Cu at (283.6, 153.3)
- added D16: LED, LED_SMD:LED_0805_2012Metric, F.Cu at (138.2, 78.0)
- added D17: LED, LED_SMD:LED_0805_2012Metric, F.Cu at (138.2, 80.2)
- added D18: LED, LED_SMD:LED_0805_2012Metric, F.Cu at (138.2, 82.3)
- added D19: LED, LED_SMD:LED_0805_2012Metric, F.Cu at (138.2, 84.5)
- added D20: LED, LED_SMD:LED_0805_2012Metric, F.Cu at (138.2, 86.7)
- added D21: LED, LED_SMD:LED_0805_2012Metric, F.Cu at (138.2, 88.8)
- added D22: LED, LED_SMD:LED_0805_2012Metric, F.Cu at (138.2, 91.0)
- added JP7: Jumper_2_Open, Jumper:SolderJumper-2_P1.3mm_Bridged2Bar_Pad1.0x1.5mm, F.Cu at (234.1, 164.8)
- added JP8: Jumper_3_Bridged12, Jumper:SolderJumper-3_P1.3mm_Bridged12_Pad1.0x1.5mm, F.Cu at (306.0, 161.3)
- added JP9: Jumper_3_Bridged12, Jumper:SolderJumper-3_P1.3mm_Bridged12_Pad1.0x1.5mm, F.Cu at (306.0, 165.1)
- added Q2: AO3400A, Package_TO_SOT_SMD:SOT-23, F.Cu at (289.3, 166.7)
- added Q3: AO3400A, Package_TO_SOT_SMD:SOT-23, F.Cu at (114.8, 187.9)
- added Q4: AO3400A, Package_TO_SOT_SMD:SOT-23, F.Cu at (114.8, 192.4)
- added R28: 3.88k, Resistor_SMD:R_0603_1608Metric, F.Cu at (331.0, 162.6)
- added R71: 10K 1/2W, Resistor_SMD:R_1210_3225Metric, F.Cu at (300.4, 161.6)
- added R72: 10K 1/2W, Resistor_SMD:R_1210_3225Metric, F.Cu at (300.4, 165.8)
- added R73: 10R 1/10W, Resistor_SMD:R_0603_1608Metric, F.Cu at (299.6, 174.1)
- added R74: 2.49k +-1%, Resistor_SMD:R_0603_1608Metric, F.Cu at (316.7, 144.8)
- added R75: 470R, Resistor_SMD:R_0603_1608Metric, F.Cu at (337.0, 147.4)
- added SW4: SW_DIP_x02, Button_Switch_SMD:SW_DIP_SPSTx02_Slide_6.7x6.64mm_W8.61mm_P2.54mm_LowProfile, F.Cu at (193.5, 82.2)
- added U1: MCZ33810EK, Library:SOP65P1030X245-33N, F.Cu at (154.6, 78.4)
- added U11: SRV05-4, Package_TO_SOT_SMD:SOT-23-6, F.Cu at (284.3, 166.7)
- added U13: MCZ33810EK, Library:SOP65P1030X245-33N, F.Cu at (157.5, 94.0)
- added U23: PaP_Driver_v1, Library:MODULE_A4988_STEPPER_MOTOR_DRIVER_CARRIER, F.Cu at (215.1, 85.4)
- added U36: MAX9926UAEE+, Package_SO:QSOP-16_3.9x4.9mm_P0.635mm, F.Cu at (201.8, 194.1)
- BT1: footprint Battery:BatteryHolder_Keystone_103_1x20mm -> Connector_JST:JST_EH_B2B-EH-A_1x02_P2.50mm_Vertical
- C19, C22: value 47p -> 0.01uF; footprint Capacitor_SMD:C_0402_1005Metric -> Capacitor_SMD:C_0805_2012Metric
- D1, D10, D12, D13, D5, D6, D7, D8, D9: footprint LED_SMD:LED_0603_1608Metric -> LED_SMD:LED_0805_2012Metric
- J4: footprint Connector_PinHeader_1.27mm:PinHeader_2x08_P1.27mm_Vertical -> Connector_PinHeader_2.54mm:PinHeader_2x08_P2.54mm_Vertical
- J7: footprint Connector_PinHeader_2.54mm:PinHeader_1x04_P2.54mm_Horizontal -> Connector_PinHeader_2.54mm:PinHeader_1x04_P2.54mm_Vertical
- Q1: value Q_DUAL_NMOS_S1G1D2S2G2D1 -> AO3400A; footprint Package_TO_SOT_SMD:SOT-363_SC-70-6 -> Package_TO_SOT_SMD:SOT-23
- R116, R117: value 4.99K 1/2W -> 10K 1/2W
- R17: value 10K 1/10W -> 10k; footprint Resistor_SMD:R_0603_1608Metric -> Resistor_SMD:R_0805_2012Metric
- R18: value 10R 1/10W -> 10k; footprint Resistor_SMD:R_0603_1608Metric -> Resistor_SMD:R_0805_2012Metric
- R49, R50, R51, R52, R53, R58: footprint Resistor_SMD:R_0603_1608Metric -> Resistor_SMD:R_0805_2012Metric
- R54: value 10k -> 2.49k +-1%
- R76, R78: value 2.49k +-1% -> 470R
- R79, R82: value 470R -> 1k
- R80: footprint Resistor_SMD:R_0805_2012Metric -> Resistor_SMD:R_0603_1608Metric
- R81: value 4.99K 1/2W -> 1k; footprint Resistor_SMD:R_1210_3225Metric -> Resistor_SMD:R_0603_1608Metric
- U26: value ~ -> SP720ABTG
- moved D47 175.7 mm to (23.1, 186.3)
- moved JP6 175.7 mm to (50.0, 179.9)
- moved TP29 175.7 mm to (37.5, 186.8)
- moved TP30 175.7 mm to (37.5, 189.9)
- moved U25 175.7 mm to (19.5, 177.0)
- moved C27 175.7 mm to (39.8, 175.8)
- moved C28 175.7 mm to (40.1, 179.9)
- moved D11 175.7 mm to (46.8, 186.8)
- moved JP5 175.7 mm to (41.8, 187.1)
- moved R83 175.7 mm to (48.7, 183.4)
- moved TP28 175.7 mm to (34.4, 189.9)
- moved TP9 175.7 mm to (34.4, 186.8)
- moved U2 166.2 mm to (39.3, 159.9)
- moved R82 155.0 mm to (119.3, 190.0)
- moved R79 153.5 mm to (119.3, 182.5)
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Connections:
- C19 pad 2: CAN+ -> MCU-D23
- C22 pad 1: CAN- -> GND
- C22 pad 2: GND -> MCU-D23
- C53 pad 1: Net-(SW2-A) -> Net-(JP8-A)
- C73 pad 1: IGN_V+ -> GND
- C73 pad 2: GND -> IGN_V+
- D5 pad 2: +5C -> +3V3
- D6 pad 2: +3V3 -> +5C
- Q1 pad 1: MCU-D23 -> +3V3
- Q1 pad 2: +3V3 -> AUX_IN2
- Q1 pad 3: (no net) -> MCU-D23
- R11 pad 1: /Sensores/AUX_CH3 -> /Sensores/AUX_CH2
- R116 pad 2: Net-(R116-Pad2) -> /CKP/CMP_sensors/IN2-
- R117 pad 2: Net-(R117-Pad2) -> /CKP/CMP_sensors/IN2+
- R129 pad 2: /PMIC/PMIC1_ENABLE -> /PMIC1_ENABLE
- R14 pad 1: /Sensores/AUX_CH4 -> /Sensores/AUX_CH3
- R17 pad 1: Net-(D2-K) -> Net-(D3-K)
- R17 pad 2: Net-(D3-K) -> Net-(D2-K)
- R18 pad 1: Net-(Q6-G) -> +5C
- R18 pad 2: Net-(Q5-C) -> /Sensores/A
- R24 pad 1: Net-(D7-K) -> Net-(D5-K)
- R3 pad 1: Net-(D1-K) -> Net-(D7-K)
- R37 pad 1: /Sensores/AUX_CH5 -> /Sensores/AUX_CH4
- R4 pad 1: Net-(D5-K) -> Net-(D6-K)
- R40 pad 1: /Sensores/AUX_CH6 -> /Sensores/AUX_CH8
- R45 pad 1: /Sensores/CH_VBATT -> /Sensores/CH_CLT
- R45 pad 2: Net-(C25-Pad1) -> E1
- R49 pad 1: +5C -> /MUX_A
- R49 pad 2: /Sensores/B -> +3V3
- R5 pad 1: Net-(D6-K) -> Net-(D1-K)
- R50 pad 2: /Sensores/C -> /Sensores/B
- R51 pad 1: +5C -> /MUX_B
- R51 pad 2: /Sensores/A -> +3V3
- R52 pad 1: /MUX_B -> +5C
- R52 pad 2: +3V3 -> /Sensores/C
- R54 pad 1: /MUX_A -> E1
- R54 pad 2: +3V3 -> +5C
- R56 pad 1: /Sensores/CH_O2 -> /Sensores/CH_VBATT
- R56 pad 2: K1 -> Net-(C25-Pad1)
- R60 pad 1: /Sensores/AUX_CH8 -> /Sensores/AUX_CH6
- R76 pad 1: E1 -> /Sensores/CH_TPS
- R76 pad 2: +5C -> E1
- R77 pad 1: /Sensores/CH_IAT -> /Sensores/CH_MAP
- R78 pad 1: E1 -> /Sensores/CH_O2
- R78 pad 2: +5C -> K1
- R79 pad 1: /Sensores/CH_CLT -> MCU-D23
- R79 pad 2: E1 -> +3V3
- R8 pad 1: /Sensores/AUX_CH2 -> /Sensores/AUX_CH5
- R81 pad 1: Net-(SW2-A) -> MCU-D23
- R81 pad 2: Net-(R113-Pad1) -> +3V3
- R82 pad 1: /Sensores/CH_TPS -> MCU-D23
- R82 pad 2: E1 -> +3V3
- R83 pad 2: /PMIC/PMIC1_ENABLE -> /PMIC1_ENABLE
- U3 pad 51: /PMIC_ENABLE -> /PMIC1_ENABLE
- U3 pad 52: /PMIC_SPARK -> /PMIC2_ENABLE
- U3 pad 57: /INY3 -> /ECN1
- U3 pad 58: /INY4 -> /ECN2
- U3 pad 59: /ECN1 -> unconnected-(U3-PD12-Pad59)
- U3 pad 60: /ECN2 -> unconnected-(U3-PD13-Pad60)
- U3 pad 61: /ECN3 -> unconnected-(U3-PD14-Pad61)
- U3 pad 62: /ECN4 -> unconnected-(U3-PD15-Pad62)
- U3 pad 78: /PMIC_NOMI -> /PMIC1_CS
- U3 pad 79: /PMIC_MAXI -> /PMIC2_CS
Other:
- board text added: "POWA"
- board text added: "locked"
- board text removed: "1"
- board text removed: "8"
- board text removed: "Encendido"
- board text removed: "Inyección"
