File: OpenEFI_rev4/Drivers.kicad_sch (KiCad schematic)
At the start: 28 parts, among them Q1 ISL9V5045S3ST, Q2 ISL9V5045S3ST, Q3 ISL9V5045S3ST, Q4 ISL9V5045S3ST

Commit message: WIP Analog frontend
Parts:
- R10: LCSC C23040 -> C17501
- R13: LCSC C192548 -> C17501
Changed lines of the file:
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@@
       (effects (font (size 1.27 1.27)) hide)
     )
-    (property "LCSC" "C192548" (at 66.04 64.77 0)
+    (property "LCSC" "C17501" (at 66.04 64.77 0)
       (effects (font (size 1.27 1.27)) hide)
     )
@@
       (effects (font (size 1.27 1.27)) hide)
     )
-    (property "LCSC" "C23040" (at 58.42 85.09 90)
-      (effects (font (size 1.27 1.27)) hide)
-    )
+    (property "LCSC" "C17501" (at 58.42 85.09 90)
+      (effects (font (size 1.27 1.27)) hide)
+    )
