File: OpenEFI_rev4/PMIC.kicad_sch (KiCad schematic)
At the start: 40 parts, among them U1 MCZ33810EK, U21 TC4424A, U24 TC4424A, U29 TC4424A, U30 TC4424A

Commit message: update footprints
Parts:
- D47, D64, D66, D68, D70, D72, D74: LCSC C5277952 -> C2128
- D76: LCSC C7473300 -> C2128
- JP6: now left out of the parts list
