File: OpenEFI_rev4/untitled.kicad_sch (KiCad schematic)
At the start: 32 parts, among them Q12 AO3400A, SW4 SW_DIP_x02, U36 MAX9926UAEE+

Commit message: WIP relay driver
Changed lines of the file:
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@@
+    )
+  )
+  (global_label "CKP+" (shape input) (at 162.56 160.02 180)
+    (effects (font (size 1.27 1.27)) (justify right))
+    (property "Intersheetrefs" "${INTERSHEET_REFS}" (at 154.7645 159.9406 0)
+      (effects (font (size 1.27 1.27)) (justify right) hide)
     )
   )

Commit message: Rev4 WIP LCSC assigments
Parts:
- R121, R122: LCSC (none) -> C25804
Changed lines of the file:
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@@
+      (effects (font (size 1.27 1.27)) hide)
+    )
+    (property "LCSC" "C25804" (at 184.3787 77.5906 0)
       (effects (font (size 1.27 1.27)) hide)
     )
@@
       (effects (font (size 1.27 1.27)) hide)
     )
+    (property "LCSC" "C25804" (at 195.8087 80.1306 0)
+      (effects (font (size 1.27 1.27)) hide)
+    )
