File: OpenEFI_rev4/OpenEFI_rev4.kicad_sch (KiCad schematic)
At the start: 103 parts, among them J1 USB_B, J2 Tag connect, J3 104031-0811, J4 Conn_02x08_Odd_Even, Q1 AO3400A, Q11 SS8050, Q12 AO3400A, Q19 AO3400A, Q2 AO3400A, Q3 AO3400A, Q4 AO3400A, Q8 SS8050, Q9 SS8050, SW1 SW_Push, U11 SRV05-4, U15 REF3033, U23 PaP_Driver_v1, U25 TJA1051T-3, U3 STM32F407VGTx, U7 25LCxxx, Y1 25MHz, Y3 32.768kHz

Commit message: Rev4 WIP LCSC assigments
Parts:
- C16: LCSC 0805 -> C1779
- C7, C8: LCSC C49217 -> C377773
- D77: LCSC C965812 -> C965814
- D77: LCSC C965817 -> C965814
- D77: LCSC C965816 -> C965814
- D77: LCSC C965813 -> C965814
- R1: LCSC (none) -> C144469
- R2: LCSC (none) -> C25804
- R35: LCSC --- -> C25803
- U11: LCSC (none) -> C85364
- U3: LCSC (none) -> C12345
- U7: LCSC (none) -> C188247
- Y1: LCSC (none) -> C9006
Changed lines of the file:
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@@
       (effects (font (size 1.27 1.27)) hide)
     )
+    (property "LCSC" "C9006" (at 34.29 27.94 0)
+      (effects (font (size 1.27 1.27)) hide)
+    )
     (pin "1")
     (pin "2")
@@
       (effects (font (size 1.27 1.27)) hide)
     )
-    (property "LCSC" "0805" (at 46.99 150.495 0)
+    (property "LCSC" "C1779" (at 46.99 150.495 0)
       (effects (font (size 1.27 1.27)) hide)
     )
@@
       (effects (font (size 1.27 1.27)) hide)
     )
+    (property "LCSC" "C12345" (at 167.64 215.9 0)
+      (effects (font (size 1.27 1.27)) hide)
+    )
     (pin "1")
     (pin "10")
@@
       (effects (font (size 1.27 1.27)) hide)
     )
-    (property "LCSC" "C49217" (at 135.89 119.38 90)
+    (property "LCSC" "C377773" (at 135.89 119.38 90)
       (effects (font (size 1.27 1.27)) hide)
     )
@@
       (effects (font (size 1.27 1.27)) hide)
     )
-    (property "LCSC" "C49217" (at 135.89 115.57 90)
+    (property "LCSC" "C377773" (at 135.89 115.57 90)
       (effects (font (size 1.27 1.27)) hide)
     )
@@
       (effects (font (size 1.27 1.27)) hide)
     )
+    (property "LCSC" "C25804" (at 138.43 110.49 0)
+      (effects (font (size 1.27 1.27)) hide)
+    )
     (pin "1")
     (pin "2")
@@
       (effects (font (size 1.27 1.27)) hide)
     )
-    (property "LCSC" "C965812" (at 384.81 157.48 0)
+    (property "LCSC" "C965814" (at 384.81 157.48 0)
       (effects (font (size 0.889 0.889)) hide)
     )
@@
       (effects (font (size 1.27 1.27)) hide)
     )
+    (property "LCSC" "C188247" (at 26.67 168.2558 0)
+      (effects (font (size 1.27 1.27)) hide)
+    )
     (pin "1")
     (pin "2")
@@
       (effects (font (size 1.27 1.27)) hide)
     )
+    (property "LCSC" "C85364" (at 250.0061 245.745 0)
+      (effects (font (size 1.27 1.27)) hide)
+    )
     (pin "1")
     (pin "2")
@@
       (effects (font (size 1.27 1.27)) hide)
     )
-    (property "LCSC" "C965817" (at 396.24 157.48 0)
+    (property "LCSC" "C965814" (at 396.24 157.48 0)
       (effects (font (size 0.889 0.889)) hide)
     )
@@
       (effects (font (size 1.27 1.27)) hide)
     )
-    (property "LCSC" "C965816" (at 372.11 157.48 0)
+    (property "LCSC" "C965814" (at 372.11 157.48 0)
       (effects (font (size 0.889 0.889)) hide)
     )
@@
       (effects (font (size 1.27 1.27)) hide)
     )
-    (property "LCSC" "C965813" (at 344.17 154.94 0)
+    (property "LCSC" "C965814" (at 344.17 154.94 0)
       (effects (font (size 0.889 0.889)) hide)
     )
@@
       (effects (font (size 1.27 1.27)) hide)
     )
+    (property "LCSC" "C144469" (at 72.39 246.38 0)
+      (effects (font (size 1.27 1.27)) hide)
+    )
     (pin "1")
     (pin "2")
@@
       (effects (font (size 1.27 1.27)) hide)
     )
-    (property "LCSC" "C965813" (at 356.87 154.94 0)
+    (property "LCSC" "C965814" (at 356.87 154.94 0)
       (effects (font (size 0.889 0.889)) hide)
     )
@@
       (effects (font (size 1.27 1.27)) hide)
     )
-    (property "LCSC" "C965813" (at 374.015 201.93 0)
+    (property "LCSC" "C965814" (at 374.015 201.93 0)
       (effects (font (size 0.889 0.889)) hide)
     )
@@
       (effects (font (size 1.27 1.27)) hide)
     )
-    (property "LCSC" "C965817" (at 323.85 158.75 0)
+    (property "LCSC" "C965814" (at 323.85 158.75 0)
       (effects (font (size 0.889 0.889)) hide)
     )
@@
       (effects (font (size 1.27 1.27)) hide)
     )
-    (property "LCSC" "C965813" (at 386.715 201.93 0)
+    (property "LCSC" "C965814" (at 386.715 201.93 0)
       (effects (font (size 0.889 0.889)) hide)
     )
@@
       (effects (font (size 1.27 1.27)) hide)
     )
-    (property "LCSC" "---" (at 25.908 87.884 90)
+    (property "LCSC" "C25803" (at 25.908 87.884 90)
       (effects (font (size 1.27 1.27)) hide)
     )

Commit message: update 32khz crystal
Parts:
- renumbered D77 to D1, D77 to D10, D77 to D12, D77 to D13, D24 to D14, D77 to D5, D77 to D6, D77 to D7, D77 to D8, D77 to D9, JP11 to JP5, TP23 to TP38, U25 to U12
Connections:
- net ADC_CS: no longer names the net of U3.15 (PC0)
- net PMIC_CS: no longer names the net of U3.77 (PA15)
- no-connect marks 2 -> 4
Other:
- note added: "Electro 1"
- note added: "Electro 2"
